Commit message: Fix collision models

File: turtlebot_arm_description/urdf/arm.urdf (robot description, URDF)
Before this commit: robot turtlebot_arm, 3 links, 2 joints
Links:
- added link arm_base_link
- added link base_footprint, mass 0.0001; collision box size=0.001 0.001 0.001; visual box size=0.001 0.001 0.001
- added link base_link, mass 1; collision cylinder length=0.0611632 radius=0.16495; visual mesh filename=package://turtlebot_description/meshes/create_body.dae
- added link bioloid_F10_3_link, mass 0.00001; collision box size=0.025 0.038 0.004; visual mesh filename=package://turtlebot_arm_description/meshes/F10.stl scale=0.001 0.001 0.001
- added link bioloid_F10_4_link, mass 0.00001; collision box size=0.025 0.038 0.004; visual mesh filename=package://turtlebot_arm_description/meshes/F10.stl scale=0.001 0.001 0.001
- added link bioloid_F10_5_link, mass 0.00001; collision box size=0.025 0.038 0.004; visual mesh filename=package://turtlebot_arm_description/meshes/F10.stl scale=0.001 0.001 0.001
- added link bioloid_F2_0_link, mass 0.00001; collision box size=0.025 0.0485 0.0375; visual mesh filename=package://turtlebot_arm_description/meshes/F2.stl scale=0.001 0.001 0.001
- added link bioloid_F2_1_link, mass 0.00001; collision box size=0.025 0.0485 0.0375; visual mesh filename=package://turtlebot_arm_description/meshes/F2.stl scale=0.001 0.001 0.001
- added link bioloid_F3_0_link, mass 0.00001; collision box size=0.025 0.038 0.009; visual mesh filename=package://turtlebot_arm_description/meshes/F3.stl scale=0.001 0.001 0.001
- added link bioloid_F3_1_link, mass 0.00001; collision box size=0.025 0.038 0.009; visual mesh filename=package://turtlebot_arm_description/meshes/F3.stl scale=0.001 0.001 0.001
- added link bioloid_F3_2_link, mass 0.00001; collision box size=0.025 0.038 0.009; visual mesh filename=package://turtlebot_arm_description/meshes/F3.stl scale=0.001 0.001 0.001
- added link bioloid_F3_3_link, mass 0.00001; collision box size=0.025 0.038 0.009; visual mesh filename=package://turtlebot_arm_description/meshes/F3.stl scale=0.001 0.001 0.001
- added link bioloid_F3_4_link, mass 0.00001; collision box size=0.025 0.038 0.009; visual mesh filename=package://turtlebot_arm_description/meshes/F3.stl scale=0.001 0.001 0.001
- added link bioloid_F4_0_link, mass 0.00001; collision box size=0.028 0.0485 0.065; visual mesh filename=package://turtlebot_arm_description/meshes/F4.stl scale=0.001 0.001 0.001
- added link bioloid_F4_1_link, mass 0.00001; collision box size=0.028 0.0485 0.065; visual mesh filename=package://turtlebot_arm_description/meshes/F4.stl scale=0.001 0.001 0.001
- added link dynamixel_AX12_0_link, mass 0.00001; collision box size=0.025 0.038 0.04762; visual mesh filename=package://turtlebot_arm_description/meshes/ax12_box.stl scale=0.001 0.001 0.001
- added link dynamixel_AX12_1_link, mass 0.00001; collision box size=0.025 0.038 0.04762; visual mesh filename=package://turtlebot_arm_description/meshes/ax12_box.stl scale=0.001 0.001 0.001
- added link dynamixel_AX12_2_link, mass 0.00001; collision box size=0.025 0.038 0.04762; visual mesh filename=package://turtlebot_arm_description/meshes/ax12_box.stl scale=0.001 0.001 0.001
- added link dynamixel_AX12_3_link, mass 0.00001; collision box size=0.025 0.038 0.04762; visual mesh filename=package://turtlebot_arm_description/meshes/ax12_box.stl scale=0.001 0.001 0.001
- added link dynamixel_AX12_4_link, mass 0.00001; collision box size=0.025 0.038 0.04762; visual mesh filename=package://turtlebot_arm_description/meshes/ax12_box.stl scale=0.001 0.001 0.001
- added link finger_0_link, mass 0.00001; collision box size=0.0783 0.03801 0.0193; visual mesh filename=package://turtlebot_arm_description/meshes/finger.stl scale=0.001 0.001 0.001
- added link finger_1_link, mass 0.00001; collision box size=0.0783 0.03801 0.0193; visual mesh filename=package://turtlebot_arm_description/meshes/finger.stl scale=0.001 0.001 0.001
- added link front_wheel_link, mass 0.01; collision sphere radius=0.018; visual sphere radius=0.018
- added link gripper_link
- added link gyro_link, mass 0.000001; visual box size=0.02 0.035 0.002
- added link kinect_depth_frame, mass 0.000001
- added link kinect_depth_optical_frame, mass 0.000001
- added link kinect_link, mass 0.00001; collision box size=0.0730 .2760 0.0720; visual mesh filename=package://turtlebot_description/meshes/kinect.dae
- added link kinect_rgb_frame, mass 0.000001
- added link kinect_rgb_optical_frame, mass 0.000001
- added link laser, mass 0.000001; visual box size=0.02 0.035 0.002
- added link left_cliff_sensor_link, mass 0.01
- added link left_wheel_link, mass 0.01; collision cylinder length=0.023 radius=0.033; visual cylinder length=0.023 radius=0.033
- added link leftfront_cliff_sensor_link, mass 0.01
- added link plate_0_link, mass 0.01; collision box size=0.233502 0.314845 0.006401; visual mesh filename=package://turtlebot_description/meshes/plate_0_logo.dae
- added link plate_1_link, mass 0.1; collision box size=0.314856 0.314856 0.006401; visual mesh filename=package://turtlebot_description/meshes/plate_1_logo.dae
- added link plate_2_link, mass 0.01; collision box size=0.314856 0.314856 0.006401; visual mesh filename=package://turtlebot_description/meshes/plate_1_logo.dae
- added link plate_3_link, mass 0.01; collision box size=0.288 0.315 0.006401; visual mesh filename=package://turtlebot_description/meshes/plate_2_logo.dae
- added link rear_wheel_link, mass 0.001; collision sphere radius=0.018; visual sphere radius=0.018
- added link right_cliff_sensor_link, mass 0.01
- added link right_wheel_link, mass 0.01; collision cylinder length=0.023 radius=0.033; visual cylinder length=0.023 radius=0.033
- added link rightfront_cliff_sensor_link, mass 0.01
- added link spacer_0_link, mass 0.00001; collision cylinder length=0.003175 radius=.0127; visual mesh filename=package://turtlebot_description/meshes/68-02403-125_Spacer.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 scale=0.001 0.001 0.001
- added link spacer_1_link, mass 0.00001; collision cylinder length=0.003175 radius=.0127; visual mesh filename=package://turtlebot_description/meshes/68-02403-125_Spacer.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 scale=0.001 0.001 0.001
- added link spacer_2_link, mass 0.00001; collision cylinder length=0.003175 radius=.0127; visual mesh filename=package://turtlebot_description/meshes/68-02403-125_Spacer.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 scale=0.001 0.001 0.001
- added link spacer_3_link, mass 0.00001; collision cylinder length=0.003175 radius=.0127; visual mesh filename=package://turtlebot_description/meshes/68-02403-125_Spacer.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 scale=0.001 0.001 0.001
- added link standoff_2in_0_link, mass 0.00001; collision cylinder length=0.0635 radius=0.0381; visual mesh filename=package://turtlebot_description/meshes/68-04552-2000-RA_Tur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 scale=0.001 0.001 0.001
- added link standoff_2in_1_link, mass 0.00001; collision cylinder length=0.0635 radius=0.0381; visual mesh filename=package://turtlebot_description/meshes/68-04552-2000-RA_Tur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 scale=0.001 0.001 0.001
- added link standoff_2in_2_link, mass 0.00001; collision cylinder length=0.0635 radius=0.0381; visual mesh filename=package://turtlebot_description/meshes/68-04552-2000-RA_Tur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 scale=0.001 0.001 0.001
- added link standoff_2in_3_link, mass 0.00001; collision cylinder length=0.0635 radius=0.0381; visual mesh filename=package://turtlebot_description/meshes/68-04552-2000-RA_Tur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 scale=0.001 0.001 0.001
- added link standoff_2in_4_link, mass 0.00001; collision cylinder length=0.0635 radius=0.0381; visual mesh filename=package://turtlebot_description/meshes/68-04552-2000-RA_Tur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 scale=0.001 0.001 0.001
- added link standoff_2in_5_link, mass 0.00001; collision cylinder length=0.0635 radius=0.0381; visual mesh filename=package://turtlebot_description/meshes/68-04552-2000-RA_Tur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 scale=0.001 0.001 0.001
- added link standoff_2in_6_link, mass 0.00001; collision cylinder length=0.0635 radius=0.0381; visual mesh filename=package://turtlebot_description/meshes/68-04552-2000-RA_Tur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 scale=0.001 0.001 0.001
- added link standoff_2in_7_link, mass 0.00001; collision cylinder length=0.0635 radius=0.0381; visual mesh filename=package://turtlebot_description/meshes/68-04552-2000-RA_Tur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 scale=0.001 0.001 0.001
- added link standoff_8in_0_link, mass 0.00001; collision cylinder length=0.2032 radius=0.011113; visual mesh filename=package://turtlebot_description/meshes/68-02421-8000-RA_Tur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 scale=0.001 0.001 0.001
- added link standoff_8in_1_link, mass 0.00001; collision cylinder length=0.2032 radius=0.011113; visual mesh filename=package://turtlebot_description/meshes/68-02421-8000-RA_Tur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 scale=0.001 0.001 0.001
- added link standoff_8in_2_link, mass 0.00001; collision cylinder length=0.2032 radius=0.011113; visual mesh filename=package://turtlebot_description/meshes/68-02421-8000-RA_Tur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 scale=0.001 0.001 0.001
- added link standoff_8in_3_link, mass 0.00001; collision cylinder length=0.2032 radius=0.011113; visual mesh filename=package://turtlebot_description/meshes/68-02421-8000-RA_Tur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 scale=0.001 0.001 0.001
- added link standoff_kinect_0_link, mass 0.00001; collision cylinder length=0.008585 radius=0.001111; visual mesh filename=package://turtlebot_description/meshes/68-04556-RA_Kinect_S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 scale=0.001 0.001 0.001
- added link standoff_kinect_1_link, mass 0.00001; collision cylinder length=0.008585 radius=0.001111; visual mesh filename=package://turtlebot_description/meshes/68-04556-RA_Kinect_S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 scale=0.001 0.001 0.001
- added link wall_sensor_link, mass 0.01
- link bioloid_F10_0_link: geometry collision box size=0.025 0.038 0.004; visual mesh filename=package://turtlebot_arm_description/meshes/F10.stl scale=0.001 0.001 0.001
- link bioloid_F10_1_link: geometry collision box size=0.025 0.038 0.004; visual mesh filename=package://turtlebot_arm_description/meshes/F10.stl scale=0.001 0.001 0.001
- link bioloid_F10_2_link: geometry collision box size=0.025 0.038 0.004; visual mesh filename=package://turtlebot_arm_description/meshes/F10.stl scale=0.001 0.001 0.001
Joints:
- added joint arm_base_joint: type fixed, parent plate_3_link, child arm_base_link, origin xyz=0.1143 0 0.0508
- added joint base_footprint_joint: type fixed, parent base_footprint, child base_link, origin xyz=0 0 0.017 rpy=0 0 0
- added joint base_kinect_joint: type fixed, parent plate_2_link, child kinect_link, origin xyz=-0.0844382 0 0.1047496 rpy=0 0 0
- added joint base_left_cliff_sensor_joint: type fixed, parent base_link, child left_cliff_sensor_link, origin xyz=0.07 0.14 0.01 rpy=0 1.57079 0
- added joint base_leftfront_cliff_sensor_joint: type fixed, parent base_link, child leftfront_cliff_sensor_link, origin xyz=0.15 0.04 0.01 rpy=0 1.57079 0
- added joint base_right_cliff_sensor_joint: type fixed, parent base_link, child right_cliff_sensor_link, origin xyz=0.07 -0.14 0.01 rpy=0 1.57079 0
- added joint base_rightfront_cliff_sensor_joint: type fixed, parent base_link, child rightfront_cliff_sensor_link, origin xyz=0.15 -0.04 0.01 rpy=0 1.57079 0
- added joint base_wall_sensor_joint: type fixed, parent base_link, child wall_sensor_link, origin xyz=0.09 -0.120 0.042 rpy=0 0 -1.0
- added joint bioloid_F10_0_joint: type fixed, parent bioloid_F4_0_link, child bioloid_F10_0_link, origin xyz=0 0 0.0545 rpy=0 0 0
- added joint bioloid_F10_3_joint: type fixed, parent bioloid_F4_1_link, child bioloid_F10_3_link, origin xyz=0 0 0.0545 rpy=0 0 0
- added joint bioloid_F10_4_joint: type fixed, parent bioloid_F10_3_link, child bioloid_F10_4_link, origin xyz=0 0 0.004 rpy=0 0 0
- added joint bioloid_F10_5_joint: type fixed, parent bioloid_F10_4_link, child bioloid_F10_5_link, origin xyz=0 0 0.004 rpy=0 0 0
- added joint bioloid_F3_1_joint: type fixed, parent bioloid_F10_2_link, child bioloid_F3_1_link, origin xyz=0 0 0.002 rpy=0 3.14159 0
- added joint bioloid_F3_2_joint: type fixed, parent bioloid_F10_5_link, child bioloid_F3_2_link, origin xyz=0 0 0.002 rpy=0 3.14159 0
- added joint bioloid_F3_3_joint: type fixed, parent bioloid_F2_0_link, child bioloid_F3_3_link, origin xyz=0.0 -0.016 0.0265 rpy=0 3.14159 1.570795
- added joint bioloid_F3_4_joint: type fixed, parent dynamixel_AX12_4_link, child bioloid_F3_4_link, origin xyz=0 0 -0.0415 rpy=0 3.14159 0
- added joint dynamixel_AX12_0_joint: type fixed, parent arm_base_link, child dynamixel_AX12_0_link, origin xyz=0 0 -0.019 rpy=1.570795 0 1.570795
- added joint dynamixel_AX12_1_joint: type fixed, parent bioloid_F3_0_link, child dynamixel_AX12_1_link, origin xyz=0 0 -0.0415 rpy=0 3.14159 0
- added joint dynamixel_AX12_2_joint: type fixed, parent bioloid_F3_1_link, child dynamixel_AX12_2_link, origin xyz=0 0 -0.0415 rpy=0 3.14159 0
- added joint dynamixel_AX12_3_joint: type fixed, parent bioloid_F3_2_link, child dynamixel_AX12_3_link, origin xyz=0 0 -0.0415 rpy=0 3.14159 0
- added joint dynamixel_AX12_4_joint: type fixed, parent bioloid_F3_3_link, child dynamixel_AX12_4_link, origin xyz=-0.02275 0 -0.019 rpy=3.14159 1.570795 0
- added joint elbow_flex_joint: type revolute, parent dynamixel_AX12_2_link, child bioloid_F4_1_link, origin xyz=0 0 0 rpy=0 0 0, axis 0 1 0, limit lower=-2.0 upper=2.0 effort=30 velocity=1.0
- added joint finger_0_joint: type fixed, parent bioloid_F2_1_link, child finger_0_link, origin xyz=0 0 0.0265 rpy=0 0 0
- added joint finger_1_joint: type fixed, parent bioloid_F3_4_link, child finger_1_link, origin xyz=0 0 0 rpy=0 0 3.14159
- added joint front_castor_joint: type continuous, parent base_link, child front_wheel_link, origin xyz=0.13 0 0.0 rpy=0 0 0, axis 0 1 0
- added joint gripper_joint: type revolute, parent dynamixel_AX12_4_link, child bioloid_F2_1_link, origin xyz=0 0 0 rpy=0 0 0, axis 0 1 0, limit lower=-0.6 upper=0.5 effort=30 velocity=1.0
- added joint gripper_link_joint: type fixed, parent bioloid_F2_0_link, child gripper_link, origin xyz=0 0 .112 rpy=0 -1.570795 0
- added joint gyro_joint: type fixed, parent base_link, child gyro_link, origin xyz=0 0 0.04 rpy=0 0 0
- added joint kinect_depth_joint: type fixed, parent kinect_link, child kinect_depth_frame, origin xyz=0 0.018 0 rpy=0 0 0
- added joint kinect_depth_optical_joint: type fixed, parent kinect_depth_frame, child kinect_depth_optical_frame, origin xyz=0 0 0 rpy=-1.570795 0 -1.570795
- added joint kinect_rgb_joint: type fixed, parent kinect_link, child kinect_rgb_frame, origin xyz=0 -0.005 0 rpy=0 0 0
- added joint kinect_rgb_optical_joint: type fixed, parent kinect_rgb_frame, child kinect_rgb_optical_frame, origin xyz=0 0 0 rpy=-1.570795 0 -1.570795
- added joint laser_joint: type fixed, parent base_link, child laser, origin xyz=-0.065 0 0.075 rpy=0 0 0
- added joint left_wheel_joint: type continuous, parent base_link, child left_wheel_link, origin xyz=0 0.13 0.015 rpy=0 0 0, axis 0 1 0
- added joint plate_0_joint: type fixed, parent base_link, child plate_0_link, origin xyz=-0.04334 0  0.06775704 rpy=0 0 0
- added joint plate_1_joint: type fixed, parent plate_0_link, child plate_1_link, origin xyz=0.04068 0 0.05715 rpy=0 0 0
- added joint plate_2_joint: type fixed, parent plate_1_link, child plate_2_link, origin xyz=0 0 0.0572008 rpy=0 0 0
- added joint plate_3_joint: type fixed, parent plate_2_link, child plate_3_link, origin xyz=-0.01316 0 0.2063496 rpy=0 0 0
- added joint rear_castor_joint: type continuous, parent base_link, child rear_wheel_link, origin xyz=-0.13 0 0.0 rpy=0 0 0, axis 0 1 0
- added joint right_wheel_joint: type continuous, parent base_link, child right_wheel_link, origin xyz=0 -0.13 0.015 rpy=0 0 0, axis 0 1 0
- added joint shoulder_lift_joint: type revolute, parent dynamixel_AX12_1_link, child bioloid_F4_0_link, origin xyz=0 0 0 rpy=0 0 0, axis 0 1 0, limit lower=-2.0 upper=2.0 effort=30 velocity=1.0
- added joint shoulder_pan_joint: type revolute, parent dynamixel_AX12_0_link, child bioloid_F3_0_link, origin xyz=0 0.019 0 rpy=-1.570795 1.570795 3.14159, axis 0 0 1, limit lower=-2.0 upper=2.0 effort=30 velocity=1.0
- added joint spacer_0_joint: type fixed, parent base_link, child spacer_0_link, origin xyz=-0.00254 0.1114679 0.062992 rpy=0 0 0
- added joint spacer_1_joint: type fixed, parent base_link, child spacer_1_link, origin xyz=-0.00254 -0.1114679 0.062992 rpy=0 0 0
- added joint spacer_2_joint: type fixed, parent base_link, child spacer_2_link, origin xyz=-0.07239 -0.1114679 0.062992 rpy=0 0 0
- added joint spacer_3_joint: type fixed, parent base_link, child spacer_3_link, origin xyz=-0.07239 0.1114679 0.062992 rpy=0 0 0
- added joint standoff_2in_0_joint: type fixed, parent base_link, child standoff_2in_0_link, origin xyz=0.0676402 0.1314196 0.0709803 rpy=0 0 0
- added joint standoff_2in_1_joint: type fixed, parent base_link, child standoff_2in_1_link, origin xyz=0.0676402 -0.1314196 0.0709803 rpy=0 0 0
- added joint standoff_2in_2_joint: type fixed, parent base_link, child standoff_2in_2_link, origin xyz=-0.052832 -0.1314196 0.0709803 rpy=0 0 0
- added joint standoff_2in_3_joint: type fixed, parent base_link, child standoff_2in_3_link, origin xyz=-0.052832 0.1314196 0.0709803 rpy=0 0 0
- added joint standoff_2in_4_joint: type fixed, parent standoff_2in_0_link, child standoff_2in_4_link, origin xyz=0 0 0.05715 rpy=0 0 0
- added joint standoff_2in_5_joint: type fixed, parent standoff_2in_1_link, child standoff_2in_5_link, origin xyz=0 0 0.05715 rpy=0 0 0
- added joint standoff_2in_6_joint: type fixed, parent standoff_2in_2_link, child standoff_2in_6_link, origin xyz=0 0 0.05715 rpy=0 0 0
- added joint standoff_2in_7_joint: type fixed, parent standoff_2in_3_link, child standoff_2in_7_link, origin xyz=0 0 0.05715 rpy=0 0 0
- added joint standoff_8in_0_joint: type fixed, parent standoff_2in_4_link, child standoff_8in_0_link, origin xyz=0 0 0.05715 rpy=0 0 0
- added joint standoff_8in_1_joint: type fixed, parent standoff_2in_5_link, child standoff_8in_1_link, origin xyz=0 0 0.05715 rpy=0 0 0
- added joint standoff_8in_2_joint: type fixed, parent standoff_2in_6_link, child standoff_8in_2_link, origin xyz=0 0 0.05715 rpy=0 0 0
- added joint standoff_8in_3_joint: type fixed, parent standoff_2in_7_link, child standoff_8in_3_link, origin xyz=0 0 0.05715 rpy=0 0 0
- added joint standoff_kinect_0_joint: type fixed, parent plate_2_link, child standoff_kinect_0_link, origin xyz=-0.1024382 0.098 0.0032004 rpy=0 0 0
- added joint standoff_kinect_1_joint: type fixed, parent plate_2_link, child standoff_kinect_1_link, origin xyz=-0.1024382 -0.098 0.0032004 rpy=0 0 0
- added joint wrist_flex_joint: type revolute, parent dynamixel_AX12_3_link, child bioloid_F2_0_link, origin xyz=0 0 0 rpy=0 0 0, axis 0 1 0, limit lower=-2.0 upper=2.0 effort=30 velocity=1.0
- joint bioloid_F10_1_joint: origin xyz=0 0.004 0 rpy=0 0 0 -> xyz=0 0 0.004 rpy=0 0 0
- joint bioloid_F10_2_joint: origin xyz=0 0.004 0 rpy=0 0 0 -> xyz=0 0 0.004 rpy=0 0 0

File: turtlebot_arm_description/urdf/arm_hardware.xacro (robot description, xacro)
@@ -60,5 +60,5 @@
       </visual>
       <collision>
-        <origin xyz="0.02645 0.0 0.00655" rpy="0 0 0" />
+        <origin xyz="0.02645 0.0 -0.00655" rpy="0 0 0" />
         <geometry>
           <box size="0.0783 0.03801 0.0193"/>
@@ -118,7 +118,7 @@
       </visual>
       <collision>
-        <origin xyz="0.0 0.0 -0.0045" rpy="0 0 0" />
-        <geometry>
-          <box size="0.025 0.038 0.009"/>
+        <origin xyz="0.0 0.0 -0.01241" rpy="0 0 0" />
+        <geometry>
+          <box size="0.025 0.038 0.04762"/>
         </geometry>
       </collision>
@@ -180,5 +180,5 @@
       </visual>
       <collision>
-        <origin xyz="0.0 0.0 0.0775" rpy="0 0 0" />
+        <origin xyz="0.0 0.0 0.00775" rpy="0 0 0" />
         <geometry>
           <box size="0.025 0.0485 0.0375"/>
