Commit message: close #71

File: turtlebot_arm_description/urdf/arm.urdf (robot description, URDF)
Before this commit: robot turtlebot_arm, 64 links, 63 joints
Links:
- removed link bioloid_F10_0_link
- removed link bioloid_F10_1_link
- removed link bioloid_F10_2_link
- removed link bioloid_F10_3_link
- removed link bioloid_F10_4_link
- removed link bioloid_F10_5_link
- removed link bioloid_F2_0_link
- removed link bioloid_F2_1_link
- removed link bioloid_F3_0_link
- removed link bioloid_F3_1_link
- removed link bioloid_F3_2_link
- removed link bioloid_F3_3_link
- removed link bioloid_F3_4_link
- removed link bioloid_F4_0_link
- removed link bioloid_F4_1_link
- removed link dynamixel_AX12_0_link
- removed link dynamixel_AX12_1_link
- removed link dynamixel_AX12_2_link
- removed link dynamixel_AX12_3_link
- removed link dynamixel_AX12_4_link
- removed link finger_0_link
- removed link finger_1_link
- added link arm_elbow_F10_0_link, mass 0.00001; collision box size=0.025 0.038 0.004; visual mesh filename=package://turtlebot_arm_description/meshes/F10.stl scale=0.001 0.001 0.001
- added link arm_elbow_F10_1_link, mass 0.00001; collision box size=0.025 0.038 0.004; visual mesh filename=package://turtlebot_arm_description/meshes/F10.stl scale=0.001 0.001 0.001
- added link arm_elbow_F10_2_link, mass 0.00001; collision box size=0.025 0.038 0.004; visual mesh filename=package://turtlebot_arm_description/meshes/F10.stl scale=0.001 0.001 0.001
- added link arm_elbow_F3_0_link, mass 0.00001; collision box size=0.025 0.038 0.009; visual mesh filename=package://turtlebot_arm_description/meshes/F3.stl scale=0.001 0.001 0.001
- added link arm_elbow_flex_link, mass 0.00001; collision box size=0.028 0.0485 0.065; visual mesh filename=package://turtlebot_arm_description/meshes/F4.stl scale=0.001 0.001 0.001
- added link arm_elbow_flex_servo_link, mass 0.00001; collision box size=0.025 0.038 0.04762; visual mesh filename=package://turtlebot_arm_description/meshes/ax12_box.stl scale=0.001 0.001 0.001
- added link arm_shoulder_F10_0_link, mass 0.00001; collision box size=0.025 0.038 0.004; visual mesh filename=package://turtlebot_arm_description/meshes/F10.stl scale=0.001 0.001 0.001
- added link arm_shoulder_F10_1_link, mass 0.00001; collision box size=0.025 0.038 0.004; visual mesh filename=package://turtlebot_arm_description/meshes/F10.stl scale=0.001 0.001 0.001
- added link arm_shoulder_F10_2_link, mass 0.00001; collision box size=0.025 0.038 0.004; visual mesh filename=package://turtlebot_arm_description/meshes/F10.stl scale=0.001 0.001 0.001
- added link arm_shoulder_F3_0_link, mass 0.00001; collision box size=0.025 0.038 0.009; visual mesh filename=package://turtlebot_arm_description/meshes/F3.stl scale=0.001 0.001 0.001
- added link arm_shoulder_lift_link, mass 0.00001; collision box size=0.028 0.0485 0.065; visual mesh filename=package://turtlebot_arm_description/meshes/F4.stl scale=0.001 0.001 0.001
- added link arm_shoulder_lift_servo_link, mass 0.00001; collision box size=0.025 0.038 0.04762; visual mesh filename=package://turtlebot_arm_description/meshes/ax12_box.stl scale=0.001 0.001 0.001
- added link arm_shoulder_pan_link, mass 0.00001; collision box size=0.025 0.038 0.009; visual mesh filename=package://turtlebot_arm_description/meshes/F3.stl scale=0.001 0.001 0.001
- added link arm_shoulder_pan_servo_link, mass 0.00001; collision box size=0.025 0.038 0.04762; visual mesh filename=package://turtlebot_arm_description/meshes/ax12_box.stl scale=0.001 0.001 0.001
- added link arm_wrist_F3_0_link, mass 0.00001; collision box size=0.025 0.038 0.009; visual mesh filename=package://turtlebot_arm_description/meshes/F3.stl scale=0.001 0.001 0.001
- added link arm_wrist_flex_link, mass 0.00001; collision box size=0.025 0.0485 0.0375; visual mesh filename=package://turtlebot_arm_description/meshes/F2.stl scale=0.001 0.001 0.001
- added link arm_wrist_flex_servo_link, mass 0.00001; collision box size=0.025 0.038 0.04762; visual mesh filename=package://turtlebot_arm_description/meshes/ax12_box.stl scale=0.001 0.001 0.001
- added link gripper_active_finger_link, mass 0.00001; collision box size=0.0783 0.03801 0.0193; visual mesh filename=package://turtlebot_arm_description/meshes/finger.stl scale=0.001 0.001 0.001
- added link gripper_active_link, mass 0.00001; collision box size=0.025 0.0485 0.0375; visual mesh filename=package://turtlebot_arm_description/meshes/F2.stl scale=0.001 0.001 0.001
- added link gripper_servo_link, mass 0.00001; collision box size=0.025 0.038 0.04762; visual mesh filename=package://turtlebot_arm_description/meshes/ax12_box.stl scale=0.001 0.001 0.001
- added link gripper_static_finger_link, mass 0.00001; collision box size=0.0783 0.03801 0.0193; visual mesh filename=package://turtlebot_arm_description/meshes/finger.stl scale=0.001 0.001 0.001
- added link gripper_static_link, mass 0.00001; collision box size=0.025 0.038 0.009; visual mesh filename=package://turtlebot_arm_description/meshes/F3.stl scale=0.001 0.001 0.001
- link base_link: mass 1 -> 2; geometry collision cylinder length=0.0611632 radius=0.016495; visual mesh filename=package://turtlebot_description/meshes/create_body.dae
- link gyro_link: mass 0.000001 -> 0.001
- link kinect_depth_frame: mass 0.000001 -> 0.01
- link kinect_depth_optical_frame: mass 0.000001 -> 0.001
- link kinect_link: mass 0.00001 -> 0.01
- link kinect_rgb_frame: mass 0.000001 -> 0.001
- link kinect_rgb_optical_frame: mass 0.000001 -> 0.001
- link laser: mass 0.000001 -> 0.001
- link rear_wheel_link: geometry collision sphere radius=0.015; visual sphere radius=0.015
- link spacer_0_link: mass 0.00001 -> 0.001
- link spacer_1_link: mass 0.00001 -> 0.001
- link spacer_2_link: mass 0.00001 -> 0.001
- link spacer_3_link: mass 0.00001 -> 0.001
- link standoff_2in_0_link: mass 0.00001 -> 0.001
- link standoff_2in_1_link: mass 0.00001 -> 0.001
- link standoff_2in_2_link: mass 0.00001 -> 0.001
- link standoff_2in_3_link: mass 0.00001 -> 0.001
- link standoff_2in_4_link: mass 0.00001 -> 0.001
- link standoff_2in_5_link: mass 0.00001 -> 0.001
- link standoff_2in_6_link: mass 0.00001 -> 0.001
- link standoff_2in_7_link: mass 0.00001 -> 0.001
- link standoff_8in_0_link: mass 0.00001 -> 0.001
- link standoff_8in_1_link: mass 0.00001 -> 0.001
- link standoff_8in_2_link: mass 0.00001 -> 0.001
- link standoff_8in_3_link: mass 0.00001 -> 0.001
- link standoff_kinect_0_link: mass 0.00001 -> 0.001
- link standoff_kinect_1_link: mass 0.00001 -> 0.001
Joints:
- removed joint bioloid_F10_0_joint
- removed joint bioloid_F10_1_joint
- removed joint bioloid_F10_2_joint
- removed joint bioloid_F10_3_joint
- removed joint bioloid_F10_4_joint
- removed joint bioloid_F10_5_joint
- removed joint bioloid_F3_1_joint
- removed joint bioloid_F3_2_joint
- removed joint bioloid_F3_3_joint
- removed joint bioloid_F3_4_joint
- removed joint dynamixel_AX12_0_joint
- removed joint dynamixel_AX12_1_joint
- removed joint dynamixel_AX12_2_joint
- removed joint dynamixel_AX12_3_joint
- removed joint dynamixel_AX12_4_joint
- removed joint elbow_flex_joint
- removed joint finger_0_joint
- removed joint finger_1_joint
- removed joint shoulder_lift_joint
- removed joint shoulder_pan_joint
- removed joint wrist_flex_joint
- added joint arm_elbow_F10_0_joint: type fixed, parent arm_elbow_flex_link, child arm_elbow_F10_0_link, origin xyz=0 0 0.0545 rpy=0 0 0
- added joint arm_elbow_F10_1_joint: type fixed, parent arm_elbow_F10_0_link, child arm_elbow_F10_1_link, origin xyz=0 0 0.004 rpy=0 0 0
- added joint arm_elbow_F10_2_joint: type fixed, parent arm_elbow_F10_1_link, child arm_elbow_F10_2_link, origin xyz=0 0 0.004 rpy=0 0 0
- added joint arm_elbow_F3_0_joint: type fixed, parent arm_elbow_F10_2_link, child arm_elbow_F3_0_link, origin xyz=0 0 0.002 rpy=0 3.14159 0
- added joint arm_elbow_flex_joint: type revolute, parent arm_elbow_flex_servo_link, child arm_elbow_flex_link, origin xyz=0 0 0 rpy=0 0 0, axis 0 1 0, limit lower=-2.617 upper=2.617 effort=30 velocity=1.571
- added joint arm_elbow_flex_servo_joint: type fixed, parent arm_shoulder_F3_0_link, child arm_elbow_flex_servo_link, origin xyz=0 0 -0.0415 rpy=0 3.14159 0
- added joint arm_shoulder_F10_0_joint: type fixed, parent arm_shoulder_lift_link, child arm_shoulder_F10_0_link, origin xyz=0 0 0.0545 rpy=0 0 0
- added joint arm_shoulder_F10_1_joint: type fixed, parent arm_shoulder_F10_0_link, child arm_shoulder_F10_1_link, origin xyz=0 0 0.004 rpy=0 0 0
- added joint arm_shoulder_F10_2_joint: type fixed, parent arm_shoulder_F10_1_link, child arm_shoulder_F10_2_link, origin xyz=0 0 0.004 rpy=0 0 0
- added joint arm_shoulder_F3_0_joint: type fixed, parent arm_shoulder_F10_2_link, child arm_shoulder_F3_0_link, origin xyz=0 0 0.002 rpy=0 3.14159 0
- added joint arm_shoulder_lift_joint: type revolute, parent arm_shoulder_lift_servo_link, child arm_shoulder_lift_link, origin xyz=0 0 0 rpy=0 0 0, axis 0 1 0, limit lower=-2.617 upper=2.617 effort=30 velocity=1.571
- added joint arm_shoulder_lift_servo_joint: type fixed, parent arm_shoulder_pan_link, child arm_shoulder_lift_servo_link, origin xyz=0 0 -0.0415 rpy=0 3.14159 0
- added joint arm_shoulder_pan_joint: type revolute, parent arm_shoulder_pan_servo_link, child arm_shoulder_pan_link, origin xyz=0 0.019 0 rpy=-1.570795 1.570795 3.14159, axis 0 0 -1, limit lower=-2.617 upper=2.617 effort=30 velocity=0.785
- added joint arm_shoulder_pan_servo_joint: type fixed, parent arm_base_link, child arm_shoulder_pan_servo_link, origin xyz=0 0 0 rpy=1.570795 0 1.570795
- added joint arm_wrist_F3_0_joint: type fixed, parent arm_wrist_flex_link, child arm_wrist_F3_0_link, origin xyz=0 0.016 0.0265 rpy=0 3.14159 -1.570795
- added joint arm_wrist_flex_joint: type revolute, parent arm_wrist_flex_servo_link, child arm_wrist_flex_link, origin xyz=0 0 0 rpy=0 0 0, axis 0 1 0, limit lower=-1.745 upper=1.745 effort=30 velocity=1.571
- added joint arm_wrist_flex_servo_joint: type fixed, parent arm_elbow_F3_0_link, child arm_wrist_flex_servo_link, origin xyz=0 0 -0.0415 rpy=0 3.14159 0
- added joint gripper_active_finger_joint: type fixed, parent gripper_active_link, child gripper_active_finger_link, origin xyz=0 0 0.0265 rpy=0 0 0
- added joint gripper_servo_joint: type fixed, parent arm_wrist_F3_0_link, child gripper_servo_link, origin xyz=-0.02275 0 -0.019 rpy=3.14159 1.570795 0
- added joint gripper_static_finger_joint: type fixed, parent gripper_static_link, child gripper_static_finger_link, origin xyz=0 0 0 rpy=0 0 3.14159
- added joint gripper_static_joint: type fixed, parent gripper_servo_link, child gripper_static_link, origin xyz=0 0 -0.0415 rpy=0 3.14159 0
- joint front_castor_joint: type continuous -> fixed
- joint gripper_joint: child bioloid_F2_1_link -> gripper_active_link; limit lower=-0.6 upper=0.5 effort=30 velocity=1.0 -> lower=-0.060 upper=0.50 effort=30 velocity=0.785; parent dynamixel_AX12_4_link -> gripper_servo_link
- joint gripper_link_joint: parent bioloid_F2_0_link -> arm_wrist_flex_link
- joint rear_castor_joint: type continuous -> fixed

File: turtlebot_arm_description/urdf/arm.xacro (robot description, xacro)
@@ -22,36 +22,106 @@
     <joint name="gripper_link_joint" type="fixed">
       <origin xyz="0 0 .112" rpy="0 -${M_PI/2} 0" />
-      <parent link="bioloid_F2_0_link"/>
+      <parent link="arm_wrist_flex_link"/>
       <child link="gripper_link" />
     </joint>
     <!-- shoulder pan joint -->
-    <dynamixel_AX12_fixed parent="arm_base_link" number="0" x_loc="0" y_loc="0" z_loc="${-AX12_WIDTH/2}" r="${M_PI/2}" p="0" y="${M_PI/2}"/>
-    <bioloid_F3_revolute parent="dynamixel_AX12_0_link" number="0" joint_name="shoulder_pan" x_loc="0" y_loc="${AX12_WIDTH/2}" z_loc="0" r="${-M_PI/2}" p="${M_PI/2}" y="${M_PI}" color="${color}"/>
-    <dynamixel_AX12_fixed parent="bioloid_F3_0_link" number="1" x_loc="0" y_loc="0" z_loc="${-AX12_HEIGHT-F10_HEIGHT+0.001}" r="0" p="${M_PI}" y="0"/>
-    <!--shoulder lift joint -->
-    <bioloid_F4_revolute parent="dynamixel_AX12_1_link" number="0" joint_name="shoulder_lift" x_loc="0" y_loc="0" z_loc="0" color="${color}"/>
-    <bioloid_F10_fixed parent="bioloid_F4_0_link" number="0" x_loc="0" y_loc="0" z_loc="${F4_HEIGHT+F10_HEIGHT/2}" color="${color}"/>
-    <bioloid_F10_fixed parent="bioloid_F10_0_link" number="1" x_loc="0" y_loc="0" z_loc="${F10_HEIGHT}" color="${color}"/>
-    <bioloid_F10_fixed parent="bioloid_F10_1_link" number="2" x_loc="0" y_loc="0" z_loc="${F10_HEIGHT}" color="${color}"/>
-    <bioloid_F3_fixed parent="bioloid_F10_2_link" number="1" x_loc="0" y_loc="0" z_loc="${F10_HEIGHT/2}" r="0" p="${M_PI}" y="0" color="${color}"/>
-    <!--elbow joint -->
-    <dynamixel_AX12_fixed parent="bioloid_F3_1_link" number="2" x_loc="0" y_loc="0" z_loc="${-AX12_HEIGHT-F10_HEIGHT+0.001}" r="0" p="${M_PI}" y="0"/>
-    <bioloid_F4_revolute parent="dynamixel_AX12_2_link" number="1" joint_name="elbow_flex" x_loc="0" y_loc="0" z_loc="0" color="${color}"/>
-    <bioloid_F10_fixed parent="bioloid_F4_1_link" number="3" x_loc="0" y_loc="0" z_loc="${F4_HEIGHT+F10_HEIGHT/2}" color="${color}"/>
-    <bioloid_F10_fixed parent="bioloid_F10_3_link" number="4" x_loc="0" y_loc="0" z_loc="${F10_HEIGHT}" color="${color}"/>
-    <bioloid_F10_fixed parent="bioloid_F10_4_link" number="5" x_loc="0" y_loc="0" z_loc="${F10_HEIGHT}" color="${color}"/>
-    <bioloid_F3_fixed parent="bioloid_F10_5_link" number="2" x_loc="0" y_loc="0" z_loc="${F10_HEIGHT/2}" r="0" p="${M_PI}" y="0" color="${color}"/>
-    <!--wrist joint-->
-    <dynamixel_AX12_fixed parent="bioloid_F3_2_link" number="3" x_loc="0" y_loc="0" z_loc="${-AX12_HEIGHT-F10_HEIGHT+0.001}" r="0" p="${M_PI}" y="0"/>
-    <bioloid_F2_revolute parent="dynamixel_AX12_3_link" number="0" joint_name="wrist_flex" x_loc="0" y_loc="0" z_loc="0" ulimit="2.0" llimit="-2.0" color="${color}"/>
-    <bioloid_F3_fixed parent="bioloid_F2_0_link" number="3" x_loc="0.000" y_loc="0.016" z_loc="${F2_HEIGHT}" r="0" p="${M_PI}" y="${-M_PI/2}" color="${color}"/>
-    <!--gripper joint -->
-    <dynamixel_AX12_fixed parent="bioloid_F3_3_link" number="4" x_loc="-0.02275" y_loc="0" z_loc="${-AX12_WIDTH/2}" r="${M_PI}" p="${M_PI/2}" y="0"/>
-    <!--finger 1-->
-    <bioloid_F2_revolute parent="dynamixel_AX12_4_link" number="1" joint_name="gripper" x_loc="0" y_loc="0" z_loc="0" ulimit="0.50" llimit="-0.60" color="${color}"/>
-    <finger_fixed parent="bioloid_F2_1_link" number="0" x_loc="0" y_loc="0" z_loc="${F2_HEIGHT}" r="0" p="0" y="0" color="${gripper_color}"/>
-    <!--finger 2-->
-    <bioloid_F3_fixed parent="dynamixel_AX12_4_link" number="4" x_loc="0" y_loc="0" z_loc="${-AX12_HEIGHT-F10_HEIGHT+0.001}" r="0" p="${M_PI}" y="0" color="${color}"/>
-    <finger_fixed parent="bioloid_F3_4_link" number="1" x_loc="0" y_loc="0" z_loc="0" r="0" p="0" y="${M_PI}" color="${gripper_color}"/>
+    <dynamixel_AX12_fixed parent="arm_base_link" name="arm_shoulder_pan_servo">
+      <origin xyz="0 0 0" rpy="${M_PI/2} 0 ${M_PI/2}"/>
+    </dynamixel_AX12_fixed>
+    <bioloid_F3_revolute parent="arm_shoulder_pan_servo_link" name="arm_shoulder_pan" color="${color}" vlimit="0.785" llimit="-2.617" ulimit="2.617">
+      <origin xyz="0 ${AX12_WIDTH/2} 0" rpy="${-M_PI/2} ${M_PI/2} ${M_PI}" />
+    </bioloid_F3_revolute>
+    <!-- shoulder lift joint -->
+    <dynamixel_AX12_fixed parent="arm_shoulder_pan_link" name="arm_shoulder_lift_servo">
+      <origin xyz="0 0 ${-AX12_HEIGHT-F10_HEIGHT+0.001}" rpy="0 ${M_PI} 0" />
+    </dynamixel_AX12_fixed>
+    <bioloid_F4_revolute parent="arm_shoulder_lift_servo_link" name="arm_shoulder_lift" color="${color}" vlimit="1.571" llimit="-2.617" ulimit="2.617">
+      <origin xyz="0 0 0" rpy="0 0 0" />
+    </bioloid_F4_revolute>
+    <bioloid_F10_fixed parent="arm_shoulder_lift_link" name="arm_shoulder_F10_0" color="${color}">
+      <origin xyz="0 0 ${F4_HEIGHT+F10_HEIGHT/2}" rpy="0 0 0" />
+    </bioloid_F10_fixed>
+    <bioloid_F10_fixed parent="arm_shoulder_F10_0_link" name="arm_shoulder_F10_1" color="${color}">
+      <origin xyz="0 0 ${F10_HEIGHT}" rpy="0 0 0" />
+    </bioloid_F10_fixed>
+    <bioloid_F10_fixed parent="arm_shoulder_F10_1_link" name="arm_shoulder_F10_2" color="${color}">
+      <origin xyz="0 0 ${F10_HEIGHT}" rpy="0 0 0" />
+    </bioloid_F10_fixed>
+    <bioloid_F3_fixed parent="arm_shoulder_F10_2_link" name="arm_shoulder_F3_0" color="${color}">
+      <origin xyz="0 0 ${F10_HEIGHT/2}" rpy="0 ${M_PI} 0" />
+    </bioloid_F3_fixed>
+    <!-- elbow joint -->
+    <dynamixel_AX12_fixed parent="arm_shoulder_F3_0_link" name="arm_elbow_flex_servo">
+      <origin xyz="0 0 ${-AX12_HEIGHT-F10_HEIGHT+0.001}" rpy="0 ${M_PI} 0"/>
+    </dynamixel_AX12_fixed>
+    <bioloid_F4_revolute parent="arm_elbow_flex_servo_link" name="arm_elbow_flex" color="${color}" vlimit="1.571" llimit="-2.617" ulimit="2.617">
+      <origin xyz="0 0 0" rpy="0 0 0" />
+    </bioloid_F4_revolute>
+    <bioloid_F10_fixed parent="arm_elbow_flex_link" name="arm_elbow_F10_0" color="${color}">
+      <origin xyz="0 0 ${F4_HEIGHT+F10_HEIGHT/2}" rpy="0 0 0" />
+    </bioloid_F10_fixed>
+    <bioloid_F10_fixed parent="arm_elbow_F10_0_link" name="arm_elbow_F10_1" color="${color}">
+      <origin xyz="0 0 ${F10_HEIGHT}" rpy="0 0 0" />
+    </bioloid_F10_fixed>
+    <bioloid_F10_fixed parent="arm_elbow_F10_1_link" name="arm_elbow_F10_2" color="${color}">
+      <origin xyz="0 0 ${F10_HEIGHT}" rpy="0 0 0" />
+    </bioloid_F10_fixed>
+    <bioloid_F3_fixed parent="arm_elbow_F10_2_link" name="arm_elbow_F3_0" color="${color}">
+      <origin xyz="0 0 ${F10_HEIGHT/2}" rpy="0 ${M_PI} 0" />
+    </bioloid_F3_fixed>
+    <!-- wrist joint -->
+    <dynamixel_AX12_fixed parent="arm_elbow_F3_0_link" name="arm_wrist_flex_servo">
+      <origin xyz="0 0 ${-AX12_HEIGHT-F10_HEIGHT+0.001}" rpy="0 ${M_PI} 0"/>
+    </dynamixel_AX12_fixed>
+    <bioloid_F2_revolute parent="arm_wrist_flex_servo_link" name="arm_wrist_flex" color="${color}" vlimit="1.571" llimit="-1.745" ulimit="1.745">
+      <origin xyz="0 0 0" rpy="0 0 0" />
+    </bioloid_F2_revolute>
+    <bioloid_F3_fixed parent="arm_wrist_flex_link" name="arm_wrist_F3_0" color="${color}">
+      <origin xyz="0 0.016 ${F2_HEIGHT}" rpy="0 ${M_PI} ${-M_PI/2}" />
+    </bioloid_F3_fixed>
+    <!-- gripper joint -->
+    <dynamixel_AX12_fixed parent="arm_wrist_F3_0_link" name="gripper_servo">
+      <origin xyz="-0.02275 0 ${-AX12_WIDTH/2}" rpy="${M_PI} ${M_PI/2} 0"/>
+    </dynamixel_AX12_fixed>
+    <!-- finger 1 -->
+    <joint name="gripper_joint" type="revolute">
+      <origin xyz="0 0 0" rpy="0 0 0"/>
+      <axis xyz="0 1 0"/>
+      <limit effort="30" velocity="0.785" lower="-0.060" upper="0.50" />
+      <parent link="gripper_servo_link"/>
+      <child link="gripper_active_link" />
+    </joint>
+    <link name="gripper_active_link">
+      <inertial>
+        <mass value="0.00001" />
+        <origin xyz="0 0 0" />
+        <inertia ixx="1.0" ixy="0.0" ixz="0.0"
+          iyy="1.0" iyz="0.0"
+          izz="1.0" />
+      </inertial>
+      <visual>
+        <origin xyz=" 0 0 0 " rpy="0 0 0" />
+        <geometry>
+          <mesh filename="package://turtlebot_arm_description/meshes/F2.stl" scale="${M_SCALE} ${M_SCALE} ${M_SCALE}"/>
+        </geometry>
+        <material name="${color}"/>
+      </visual>
+      <collision>
+        <origin xyz="0.0 0.0 0.00775" rpy="0 0 0" />
+        <geometry>
+          <box size="0.025 0.0485 0.0375"/>
+        </geometry>
+      </collision>
+    </link>
+    <finger_fixed parent="gripper_active_link" name="gripper_active_finger" color="${gripper_color}">
+      <origin xyz="0 0 ${F2_HEIGHT}" rpy="0 0 0" />
+    </finger_fixed>
+    <!-- finger 2 -->
+    <bioloid_F3_fixed parent="gripper_servo_link" name="gripper_static" color="${color}">
+      <origin xyz="0 0 ${-AX12_HEIGHT-F10_HEIGHT+0.001}" rpy="0 ${M_PI} 0" />
+    </bioloid_F3_fixed>
+    <finger_fixed parent="gripper_static_link" name="gripper_static_finger" color="${gripper_color}">
+      <origin xyz="0 0 0" rpy="0 0 ${M_PI}" />
+    </finger_fixed>
   </macro>
 </robot>
