Commit message: close #71

File: turtlebot_arm_description/urdf/arm_hardware.xacro (robot description, xacro)
@@ -9,11 +9,11 @@
   <property name="AX12_WIDTH" value="0.038"/>
   <property name="F2_HEIGHT" value="0.0265"/>
-  <macro name="bioloid_F10_fixed" params="parent number x_loc y_loc z_loc color">
-    <joint name="bioloid_F10_${number}_joint" type="fixed">
-      <origin xyz="${x_loc} ${y_loc} ${z_loc}" rpy="0 0 0" />
-      <parent link="${parent}"/>
-      <child link="bioloid_F10_${number}_link" />
-    </joint>
-    <link name="bioloid_F10_${number}_link">
+  <macro name="bioloid_F10_fixed" params="parent name color *origin">
+    <joint name="${name}_joint" type="fixed">
+      <insert_block name="origin" />
+      <parent link="${parent}"/>
+      <child link="${name}_link" />
+    </joint>
+    <link name="${name}_link">
       <inertial>
         <mass value="0.00001" />
@@ -38,11 +38,11 @@
     </link>
   </macro>
-  <macro name="finger_fixed" params="parent number x_loc y_loc z_loc r p y color">
-    <joint name="finger_${number}_joint" type="fixed">
-      <origin xyz="${x_loc} ${y_loc} ${z_loc}" rpy="${r} ${p} ${y}" />
-      <parent link="${parent}"/>
-      <child link="finger_${number}_link" />
-    </joint>
-    <link name="finger_${number}_link">
+  <macro name="finger_fixed" params="parent name color *origin">
+    <joint name="${name}_joint" type="fixed">
+      <insert_block name="origin" />
+      <parent link="${parent}"/>
+      <child link="${name}_link" />
+    </joint>
+    <link name="${name}_link">
       <inertial>
         <mass value="0.00001" />
@@ -67,11 +67,11 @@
     </link>
   </macro>
-  <macro name="bioloid_F3_fixed" params="parent number x_loc y_loc z_loc r p y color">
-    <joint name="bioloid_F3_${number}_joint" type="fixed">
-      <origin xyz="${x_loc} ${y_loc} ${z_loc}" rpy="${r} ${p} ${y}" />
-      <parent link="${parent}"/>
-      <child link="bioloid_F3_${number}_link" />
-    </joint>
-    <link name="bioloid_F3_${number}_link">
+  <macro name="bioloid_F3_fixed" params="parent name color *origin">
+    <joint name="${name}_joint" type="fixed">
+      <insert_block name="origin" />
+      <parent link="${parent}"/>
+      <child link="${name}_link" />
+    </joint>
+    <link name="${name}_link">
       <inertial>
         <mass value="0.00001" />
@@ -96,11 +96,11 @@
     </link>
   </macro>
-  <macro name="dynamixel_AX12_fixed" params="parent number x_loc y_loc z_loc r p y">
-    <joint name="dynamixel_AX12_${number}_joint" type="fixed">
-      <origin xyz="${x_loc} ${y_loc} ${z_loc}" rpy="${r} ${p} ${y}" />
-      <parent link="${parent}"/>
-      <child link="dynamixel_AX12_${number}_link" />
-    </joint>
-    <link name="dynamixel_AX12_${number}_link">
+  <macro name="dynamixel_AX12_fixed" params="parent name *origin">
+    <joint name="${name}_joint" type="fixed">
+      <insert_block name="origin" />
+      <parent link="${parent}"/>
+      <child link="${name}_link" />
+    </joint>
+    <link name="${name}_link">
       <inertial>
         <mass value="0.00001" />
@@ -125,13 +125,13 @@
     </link>
   </macro>
-  <macro name="bioloid_F3_revolute" params="parent number joint_name x_loc y_loc z_loc r p y color">
-    <joint name="${joint_name}_joint" type="revolute">
-      <origin xyz="${x_loc} ${y_loc} ${z_loc}" rpy="${r} ${p} ${y}" />
-      <parent link="${parent}"/>
-       <axis xyz="0 0 -1"/>
-      <limit effort="30" velocity="1.0" lower="-2.0" upper="2.0" />
-      <child link="bioloid_F3_${number}_link" />
-    </joint>
-    <link name="bioloid_F3_${number}_link">
+  <macro name="bioloid_F3_revolute" params="parent name color llimit ulimit vlimit *origin">
+    <joint name="${name}_joint" type="revolute">
+      <insert_block name="origin" />
+      <axis xyz="0 0 -1"/>
+      <limit effort="30" velocity="${vlimit}" lower="${llimit}" upper="${ulimit}" />
+      <parent link="${parent}"/>
+      <child link="${name}_link" />
+    </joint>
+    <link name="${name}_link">
       <inertial>
         <mass value="0.00001" />
@@ -156,13 +156,13 @@
     </link>
   </macro>
-  <macro name="bioloid_F2_revolute" params="parent number joint_name x_loc y_loc z_loc ulimit llimit color">
-    <joint name="${joint_name}_joint" type="revolute">
-      <origin xyz="${x_loc} ${y_loc} ${z_loc}" rpy="0 0 0" />
-      <parent link="${parent}"/>
-       <axis xyz="0 1 0"/>
-      <limit effort="30" velocity="1.0" lower="${llimit}" upper="${ulimit}" />
-      <child link="bioloid_F2_${number}_link" />
-    </joint>
-    <link name="bioloid_F2_${number}_link">
+  <macro name="bioloid_F2_revolute" params="parent name color llimit ulimit vlimit *origin">
+    <joint name="${name}_joint" type="revolute">
+      <insert_block name="origin" />
+      <axis xyz="0 1 0"/>
+      <limit effort="30" velocity="${vlimit}" lower="${llimit}" upper="${ulimit}" />
+      <parent link="${parent}"/>
+      <child link="${name}_link" />
+    </joint>
+    <link name="${name}_link">
       <inertial>
         <mass value="0.00001" />
@@ -187,13 +187,13 @@
     </link>
   </macro>
-  <macro name="bioloid_F4_revolute" params="parent number joint_name x_loc y_loc z_loc color">
-    <joint name="${joint_name}_joint" type="revolute">
-      <origin xyz="${x_loc} ${y_loc} ${z_loc}" rpy="0 0 0" />
-      <parent link="${parent}"/>
-       <axis xyz="0 1 0"/>
-      <limit effort="30" velocity="1.0" lower="-2.0" upper="2.0" />
-      <child link="bioloid_F4_${number}_link" />
-    </joint>
-    <link name="bioloid_F4_${number}_link">
+  <macro name="bioloid_F4_revolute" params="parent name color llimit ulimit vlimit *origin">
+    <joint name="${name}_joint" type="revolute">
+      <insert_block name="origin" />
+      <axis xyz="0 1 0"/>
+      <limit effort="30" velocity="${vlimit}" lower="${llimit}" upper="${ulimit}" />
+      <parent link="${parent}"/>
+      <child link="${name}_link" />
+    </joint>
+    <link name="${name}_link">
       <inertial>
         <mass value="0.00001" />

Commit message: catkinize turtlebot_arm_description, tear out the turtlebot

File: turtlebot_arm_description/urdf/arm.urdf (robot description, URDF)
Before this commit: robot turtlebot_arm, 64 links, 63 joints
Links:
- removed link base_footprint
- removed link front_wheel_link
- removed link gyro_link
- removed link kinect_depth_frame
- removed link kinect_depth_optical_frame
- removed link kinect_link
- removed link kinect_rgb_frame
- removed link kinect_rgb_optical_frame
- removed link laser
- removed link left_cliff_sensor_link
- removed link left_wheel_link
- removed link leftfront_cliff_sensor_link
- removed link plate_0_link
- removed link plate_1_link
- removed link plate_2_link
- removed link plate_3_link
- removed link rear_wheel_link
- removed link right_cliff_sensor_link
- removed link right_wheel_link
- removed link rightfront_cliff_sensor_link
- removed link spacer_0_link
- removed link spacer_1_link
- removed link spacer_2_link
- removed link spacer_3_link
- removed link standoff_2in_0_link
- removed link standoff_2in_1_link
- removed link standoff_2in_2_link
- removed link standoff_2in_3_link
- removed link standoff_2in_4_link
- removed link standoff_2in_5_link
- removed link standoff_2in_6_link
- removed link standoff_2in_7_link
- removed link standoff_8in_0_link
- removed link standoff_8in_1_link
- removed link standoff_8in_2_link
- removed link standoff_8in_3_link
- removed link standoff_kinect_0_link
- removed link standoff_kinect_1_link
- removed link wall_sensor_link
- link arm_base_link: geometry collision box size=0.01 0.01 0.01; visual box size=0.01 0.01 0.01
- link base_link: mass 2 -> None; geometry collision box size=0.01 0.01 0.01; visual box size=0.01 0.01 0.01
- link gripper_link: geometry collision box size=0.01 0.01 0.01; visual box size=0.01 0.01 0.01
Joints:
- removed joint base_footprint_joint
- removed joint base_kinect_joint
- removed joint base_left_cliff_sensor_joint
- removed joint base_leftfront_cliff_sensor_joint
- removed joint base_right_cliff_sensor_joint
- removed joint base_rightfront_cliff_sensor_joint
- removed joint base_wall_sensor_joint
- removed joint front_castor_joint
- removed joint gyro_joint
- removed joint kinect_depth_joint
- removed joint kinect_depth_optical_joint
- removed joint kinect_rgb_joint
- removed joint kinect_rgb_optical_joint
- removed joint laser_joint
- removed joint left_wheel_joint
- removed joint plate_0_joint
- removed joint plate_1_joint
- removed joint plate_2_joint
- removed joint plate_3_joint
- removed joint rear_castor_joint
- removed joint right_wheel_joint
- removed joint spacer_0_joint
- removed joint spacer_1_joint
- removed joint spacer_2_joint
- removed joint spacer_3_joint
- removed joint standoff_2in_0_joint
- removed joint standoff_2in_1_joint
- removed joint standoff_2in_2_joint
- removed joint standoff_2in_3_joint
- removed joint standoff_2in_4_joint
- removed joint standoff_2in_5_joint
- removed joint standoff_2in_6_joint
- removed joint standoff_2in_7_joint
- removed joint standoff_8in_0_joint
- removed joint standoff_8in_1_joint
- removed joint standoff_8in_2_joint
- removed joint standoff_8in_3_joint
- removed joint standoff_kinect_0_joint
- removed joint standoff_kinect_1_joint
- joint arm_base_joint: origin xyz=0.1143 0 0.0508 -> xyz=0 0 0; parent plate_3_link -> base_link

File: turtlebot_arm_description/urdf/arm.urdf.xacro (robot description, xacro)
@@ -5,9 +5,24 @@
     xmlns:interface="http://playerstage.sourceforge.net/gazebo/xmlschema/#interface">
     <!-- Included URDF Files -->
-    <include filename="$(find turtlebot_description)/urdf/turtlebot.urdf.xacro" />
+    <!--<include filename="$(find turtlebot_description)/urdf/turtlebot.urdf.xacro" />-->
     <include filename="$(find turtlebot_arm_description)/urdf/arm.xacro" />
-    <turtlebot />
-    <turtlebot_arm parent="plate_3_link" color="white" gripper_color="green">
-      <origin xyz="0.1143 0 0.0508"/>
+    <link name="base_link">
+      <visual>
+        <origin xyz=" 0 0 0 " rpy="0 0 0" />
+        <geometry>
+          <box size="0.01 0.01 0.01"/>
+        </geometry>
+        <material name="black"/>
+      </visual>
+      <collision>
+        <origin xyz="0.0 0.0 0" rpy="0 0 0" />
+        <geometry>
+          <box size="0.01 0.01 0.01"/>
+        </geometry>
+      </collision>
+    </link>
+    <!--<turtlebot />-->
+    <turtlebot_arm parent="base_link" color="white" gripper_color="green">
+      <origin xyz="0 0 0"/>
     </turtlebot_arm>
 </robot>

Commit message: fix frame orientation, export new ikfast solver

File: turtlebot_arm_description/urdf/arm.urdf (robot description, URDF)
Before this commit: robot turtlebot_arm, 25 links, 24 joints
Links:
- link arm_base_link: geometry 
- link base_link: geometry 
- link gripper_link: geometry 
Joints:
- joint gripper_link_joint: axis (none) -> 1 0 0; limit (none) -> lower=-3.14 upper=3.14 effort=30 velocity=1; origin xyz=0 0 .112 rpy=0 -1.570795 0 -> xyz=0 0 .112 rpy=0 -1.57 0; type fixed -> revolute

File: turtlebot_arm_description/urdf/arm.urdf.xacro (robot description, xacro)
@@ -7,20 +7,8 @@
     <!--<include filename="$(find turtlebot_description)/urdf/turtlebot.urdf.xacro" />-->
     <include filename="$(find turtlebot_arm_description)/urdf/arm.xacro" />
-    <link name="base_link">
-      <visual>
-        <origin xyz=" 0 0 0 " rpy="0 0 0" />
-        <geometry>
-          <box size="0.01 0.01 0.01"/>
-        </geometry>
-        <material name="black"/>
-      </visual>
-      <collision>
-        <origin xyz="0.0 0.0 0" rpy="0 0 0" />
-        <geometry>
-          <box size="0.01 0.01 0.01"/>
-        </geometry>
-      </collision>
-    </link>
-    <!--<turtlebot />-->
+    <!-- For now I have removed the turtlebot since this all moved around..
+    <turtlebot />-->
+    <!-- Instead, there is a base_link -->
+    <link name="base_link"/>
     <turtlebot_arm parent="base_link" color="white" gripper_color="green">
       <origin xyz="0 0 0"/>

File: turtlebot_arm_description/urdf/arm.xacro (robot description, xacro)
@@ -18,10 +18,14 @@
       <child link="arm_base_link" />
     </joint>
-    <!-- fake gripper_link joint -->
+    <!-- fake gripper_link joint gives us a free servo!
+         this makes us 5DOF and saves you $44.90
+         that's a lot of coin! -->
     <link name="gripper_link" />
-    <joint name="gripper_link_joint" type="fixed">
-      <origin xyz="0 0 .112" rpy="0 -${M_PI/2} 0" />
+    <joint name="gripper_link_joint" type="revolute">
+      <origin xyz="0 0 .112" rpy="0 -1.57 0" />
       <parent link="arm_wrist_flex_link"/>
       <child link="gripper_link" />
+      <limit effort="30" velocity="1" lower="-3.14" upper="3.14"/>
+      <axis xyz="1 0 0"/>
     </joint>
     <!-- shoulder pan joint -->
