Commit message: adding dependency on turtlebot

File: turtlebot_arm_description/urdf/arm.urdf.xacro (robot description, xacro)
@@ -5,5 +5,7 @@
     xmlns:interface="http://playerstage.sourceforge.net/gazebo/xmlschema/#interface">
     <!-- Included URDF Files -->
+    <include filename="$(find turtlebot_description)/urdf/turtlebot.xacro" />
     <include filename="$(find turtlebot_arm_description)/urdf/arm.xacro" />
+    <turtlebot />
     <turtlebot_arm />
 </robot>

File: turtlebot_arm_description/urdf/arm.xacro (robot description, xacro)
@@ -3,6 +3,6 @@
   <include filename="$(find turtlebot_arm_description)/urdf/arm_hardware.xacro" />
     <macro name="turtlebot_arm">
-      <link name="base_link" />
-      <bioloid_F4_revolute parent="base_link" number="0" x_loc="0" y_loc="0" z_loc="0"/>
+      <!--link name="base_link" /-->
+      <bioloid_F4_revolute parent="base_link" number="0" x_loc="0" y_loc="0" z_loc="0.5"/>
       <bioloid_F10_fixed parent="bioloid_F4_0_link" number="0" x_loc="0" y_loc="0" z_loc="${F4_HEIGHT+F10_HEIGHT/2}"/>
       <bioloid_F10_fixed parent="bioloid_F10_0_link" number="1" x_loc="0" y_loc="0" z_loc="${F10_HEIGHT}"/>

Commit message: Make arm colors parameters

File: turtlebot_arm_description/urdf/arm.urdf.xacro (robot description, xacro)
@@ -8,4 +8,4 @@
     <include filename="$(find turtlebot_arm_description)/urdf/arm.xacro" />
     <turtlebot />
-    <turtlebot_arm />
+    <turtlebot_arm color="white" gripper_color="green"/>
 </robot>

File: turtlebot_arm_description/urdf/arm.xacro (robot description, xacro)
@@ -2,12 +2,21 @@
 <robot>
   <include filename="$(find turtlebot_arm_description)/urdf/arm_hardware.xacro" />
-    <macro name="turtlebot_arm">
-      <!-- fake arm_base_link joint -->
-      <link name="arm_base_link" />
-      <joint name="arm_base_joint" type="fixed">
-        <origin xyz="0 0 0 " rpy="-${M_PI/2} -${M_PI/2} 0" />
-        <parent link="dynamixel_AX12_0_link"/>
-        <child link="arm_base_link" />
-      </joint>
+  <material name="white">
+    <color rgba="0.87 0.90 0.87 1.0"/>
+  </material>
+  <material name="black">
+    <color rgba="0.0 0.0 0.0 1.0"/>
+  </material>
+  <material name="green">
+    <color rgba="0.22 0.32 0.14 1.0"/>
+  </material>
+  <macro name="turtlebot_arm" params="color gripper_color">
+    <!-- fake arm_base_link joint -->
+    <link name="arm_base_link" />
+    <joint name="arm_base_joint" type="fixed">
+      <origin xyz="0 0 0 " rpy="-${M_PI/2} -${M_PI/2} 0" />
+      <parent link="dynamixel_AX12_0_link"/>
+      <child link="arm_base_link" />
+    </joint>
       <!-- fake gripper_link joint -->
       <link name="gripper_link" />
@@ -19,31 +28,31 @@
       <!-- shoulder pan joint -->
       <dynamixel_AX12_fixed parent="plate_3_link" number="0" x_loc="0.1143" y_loc="0" z_loc="${0.0508-AX12_WIDTH/2}" r="${M_PI/2}" p="0" y="${M_PI/2}"/>
-      <bioloid_F3_revolute parent="arm_base_link" number="0" joint_name="shoulder_pan" x_loc="0" y_loc="0" z_loc="${AX12_WIDTH/2}" r="${-M_PI}" p="0" y="${M_PI}" />
+      <bioloid_F3_revolute parent="arm_base_link" number="0" joint_name="shoulder_pan" x_loc="0" y_loc="0" z_loc="${AX12_WIDTH/2}" r="${-M_PI}" p="0" y="${M_PI}" color="${color}"/>
       <dynamixel_AX12_fixed parent="bioloid_F3_0_link" number="1" x_loc="0" y_loc="0" z_loc="${-AX12_HEIGHT-F10_HEIGHT+0.001}" r="0" p="${M_PI}" y="0"/>
       <!--shoulder lift joint -->
-      <bioloid_F4_revolute parent="dynamixel_AX12_1_link" number="0" joint_name="shoulder_lift" x_loc="0" y_loc="0" z_loc="0"/>
-      <bioloid_F10_fixed parent="bioloid_F4_0_link" number="0" x_loc="0" y_loc="0" z_loc="${F4_HEIGHT+F10_HEIGHT/2}"/>
-      <bioloid_F10_fixed parent="bioloid_F10_0_link" number="1" x_loc="0" y_loc="0" z_loc="${F10_HEIGHT}"/>
-      <bioloid_F10_fixed parent="bioloid_F10_1_link" number="2" x_loc="0" y_loc="0" z_loc="${F10_HEIGHT}" />
-      <bioloid_F3_fixed parent="bioloid_F10_2_link" number="1" x_loc="0" y_loc="0" z_loc="${F10_HEIGHT/2}" r="0" p="${M_PI}" y="0" />
+      <bioloid_F4_revolute parent="dynamixel_AX12_1_link" number="0" joint_name="shoulder_lift" x_loc="0" y_loc="0" z_loc="0" color="${color}"/>
+      <bioloid_F10_fixed parent="bioloid_F4_0_link" number="0" x_loc="0" y_loc="0" z_loc="${F4_HEIGHT+F10_HEIGHT/2}" color="${color}"/>
+      <bioloid_F10_fixed parent="bioloid_F10_0_link" number="1" x_loc="0" y_loc="0" z_loc="${F10_HEIGHT}" color="${color}"/>
+      <bioloid_F10_fixed parent="bioloid_F10_1_link" number="2" x_loc="0" y_loc="0" z_loc="${F10_HEIGHT}" color="${color}"/>
+      <bioloid_F3_fixed parent="bioloid_F10_2_link" number="1" x_loc="0" y_loc="0" z_loc="${F10_HEIGHT/2}" r="0" p="${M_PI}" y="0" color="${color}"/>
       <!--elbow joint -->
       <dynamixel_AX12_fixed parent="bioloid_F3_1_link" number="2" x_loc="0" y_loc="0" z_loc="${-AX12_HEIGHT-F10_HEIGHT+0.001}" r="0" p="${M_PI}" y="0"/>
-      <bioloid_F4_revolute parent="dynamixel_AX12_2_link" number="1" joint_name="elbow_flex" x_loc="0" y_loc="0" z_loc="0"/>
-      <bioloid_F10_fixed parent="bioloid_F4_1_link" number="3" x_loc="0" y_loc="0" z_loc="${F4_HEIGHT+F10_HEIGHT/2}"/>
-      <bioloid_F10_fixed parent="bioloid_F10_3_link" number="4" x_loc="0" y_loc="0" z_loc="${F10_HEIGHT}"/>
-      <bioloid_F10_fixed parent="bioloid_F10_4_link" number="5" x_loc="0" y_loc="0" z_loc="${F10_HEIGHT}" />
-      <bioloid_F3_fixed parent="bioloid_F10_5_link" number="2" x_loc="0" y_loc="0" z_loc="${F10_HEIGHT/2}" r="0" p="${M_PI}" y="0" />
+      <bioloid_F4_revolute parent="dynamixel_AX12_2_link" number="1" joint_name="elbow_flex" x_loc="0" y_loc="0" z_loc="0" color="${color}"/>
+      <bioloid_F10_fixed parent="bioloid_F4_1_link" number="3" x_loc="0" y_loc="0" z_loc="${F4_HEIGHT+F10_HEIGHT/2}" color="${color}"/>
+      <bioloid_F10_fixed parent="bioloid_F10_3_link" number="4" x_loc="0" y_loc="0" z_loc="${F10_HEIGHT}" color="${color}"/>
+      <bioloid_F10_fixed parent="bioloid_F10_4_link" number="5" x_loc="0" y_loc="0" z_loc="${F10_HEIGHT}" color="${color}"/>
+      <bioloid_F3_fixed parent="bioloid_F10_5_link" number="2" x_loc="0" y_loc="0" z_loc="${F10_HEIGHT/2}" r="0" p="${M_PI}" y="0" color="${color}"/>
       <!--wrist joint-->
       <dynamixel_AX12_fixed parent="bioloid_F3_2_link" number="3" x_loc="0" y_loc="0" z_loc="${-AX12_HEIGHT-F10_HEIGHT+0.001}" r="0" p="${M_PI}" y="0"/>
-      <bioloid_F2_revolute parent="dynamixel_AX12_3_link" number="0" joint_name="wrist_flex" x_loc="0" y_loc="0" z_loc="0" ulimit="2.0" llimit="-2.0"/>
-      <bioloid_F3_fixed parent="bioloid_F2_0_link" number="3" x_loc="0.000" y_loc="-0.016" z_loc="${F2_HEIGHT}" r="0" p="${M_PI}" y="${M_PI/2}" />
+      <bioloid_F2_revolute parent="dynamixel_AX12_3_link" number="0" joint_name="wrist_flex" x_loc="0" y_loc="0" z_loc="0" ulimit="2.0" llimit="-2.0" color="${color}"/>
+      <bioloid_F3_fixed parent="bioloid_F2_0_link" number="3" x_loc="0.000" y_loc="-0.016" z_loc="${F2_HEIGHT}" r="0" p="${M_PI}" y="${M_PI/2}" color="${color}"/>
       <!--gripper joint -->
       <dynamixel_AX12_fixed parent="bioloid_F3_3_link" number="4" x_loc="-0.02275" y_loc="0" z_loc="${-AX12_WIDTH/2}" r="${M_PI}" p="${M_PI/2}" y="0"/>
       <!--finger 1-->
-      <bioloid_F2_revolute parent="dynamixel_AX12_4_link" number="1" joint_name="gripper" x_loc="0" y_loc="0" z_loc="0" ulimit="0.50" llimit="-0.60"/>
-      <finger_fixed parent="bioloid_F2_1_link" number="0" x_loc="0" y_loc="0" z_loc="${F2_HEIGHT}" r="0" p="0" y="0"/>
+      <bioloid_F2_revolute parent="dynamixel_AX12_4_link" number="1" joint_name="gripper" x_loc="0" y_loc="0" z_loc="0" ulimit="0.50" llimit="-0.60" color="${color}"/>
+      <finger_fixed parent="bioloid_F2_1_link" number="0" x_loc="0" y_loc="0" z_loc="${F2_HEIGHT}" r="0" p="0" y="0" color="${gripper_color}"/>
       <!--finger 2-->
-      <bioloid_F3_fixed parent="dynamixel_AX12_4_link" number="4" x_loc="0" y_loc="0" z_loc="${-AX12_HEIGHT-F10_HEIGHT+0.001}" r="0" p="${M_PI}" y="0" />
-      <finger_fixed parent="bioloid_F3_4_link" number="1" x_loc="0" y_loc="0" z_loc="0" r="0" p="0" y="${M_PI}"/>
+      <bioloid_F3_fixed parent="dynamixel_AX12_4_link" number="4" x_loc="0" y_loc="0" z_loc="${-AX12_HEIGHT-F10_HEIGHT+0.001}" r="0" p="${M_PI}" y="0" color="${color}"/>
+      <finger_fixed parent="bioloid_F3_4_link" number="1" x_loc="0" y_loc="0" z_loc="0" r="0" p="0" y="${M_PI}" color="${gripper_color}"/>
   </macro>
 </robot>

File: turtlebot_arm_description/urdf/arm_hardware.xacro (robot description, xacro)
@@ -9,14 +9,5 @@
   <property name="AX12_WIDTH" value="0.038"/>
   <property name="F2_HEIGHT" value="0.0265"/>
-  <material name="white">
-    <color rgba="0.87 0.90 0.87 1.0"/>
-  </material>
-  <material name="black">
-    <color rgba="0.0 0.0 0.0 1.0"/>
-  </material>
-  <material name="green">
-    <color rgba="0.22 0.32 0.14 1.0"/>
-  </material>
- <macro name="bioloid_F10_fixed" params="parent number x_loc y_loc z_loc">
+  <macro name="bioloid_F10_fixed" params="parent number x_loc y_loc z_loc color">
     <joint name="bioloid_F10_${number}_joint" type="fixed">
       <origin xyz="${x_loc} ${y_loc} ${z_loc}" rpy="0 0 0" />
@@ -37,5 +28,5 @@
           <mesh filename="package://turtlebot_arm_description/meshes/F10.stl" scale="${M_SCALE} ${M_SCALE} ${M_SCALE}"/>
         </geometry>
-        <material name="white"/>
+        <material name="${color}"/>
       </visual>
       <collision>
@@ -47,5 +38,5 @@
     </link>
   </macro>
- <macro name="finger_fixed" params="parent number x_loc y_loc z_loc r p y">
+  <macro name="finger_fixed" params="parent number x_loc y_loc z_loc r p y color">
     <joint name="finger_${number}_joint" type="fixed">
       <origin xyz="${x_loc} ${y_loc} ${z_loc}" rpy="${r} ${p} ${y}" />
@@ -66,5 +57,5 @@
           <mesh filename="package://turtlebot_arm_description/meshes/finger.stl" scale="${M_SCALE} ${M_SCALE} ${M_SCALE}"/>
         </geometry>
-        <material name="green"/>
+        <material name="${color}"/>
       </visual>
       <collision>
@@ -76,5 +67,5 @@
     </link>
   </macro>
- <macro name="bioloid_F3_fixed" params="parent number x_loc y_loc z_loc r p y">
+  <macro name="bioloid_F3_fixed" params="parent number x_loc y_loc z_loc r p y color">
     <joint name="bioloid_F3_${number}_joint" type="fixed">
       <origin xyz="${x_loc} ${y_loc} ${z_loc}" rpy="${r} ${p} ${y}" />
@@ -95,5 +86,5 @@
           <mesh filename="package://turtlebot_arm_description/meshes/F3.stl" scale="${M_SCALE} ${M_SCALE} ${M_SCALE}"/>
         </geometry>
-        <material name="white"/>
+        <material name="${color}"/>
       </visual>
       <collision>
@@ -105,5 +96,5 @@
     </link>
   </macro>
- <macro name="dynamixel_AX12_fixed" params="parent number x_loc y_loc z_loc r p y">
+  <macro name="dynamixel_AX12_fixed" params="parent number x_loc y_loc z_loc r p y">
     <joint name="dynamixel_AX12_${number}_joint" type="fixed">
       <origin xyz="${x_loc} ${y_loc} ${z_loc}" rpy="${r} ${p} ${y}" />
@@ -134,5 +125,5 @@
     </link>
   </macro>
- <macro name="bioloid_F3_revolute" params="parent number joint_name x_loc y_loc z_loc r p y">
+  <macro name="bioloid_F3_revolute" params="parent number joint_name x_loc y_loc z_loc r p y color">
     <joint name="${joint_name}_joint" type="revolute">
       <origin xyz="${x_loc} ${y_loc} ${z_loc}" rpy="${r} ${p} ${y}" />
@@ -155,5 +146,5 @@
           <mesh filename="package://turtlebot_arm_description/meshes/F3.stl" scale="${M_SCALE} ${M_SCALE} ${M_SCALE}"/>
         </geometry>
-        <material name="white"/>
+        <material name="${color}"/>
       </visual>
       <collision>
@@ -165,5 +156,5 @@
     </link>
   </macro>
- <macro name="bioloid_F2_revolute" params="parent number joint_name x_loc y_loc z_loc ulimit llimit">
+  <macro name="bioloid_F2_revolute" params="parent number joint_name x_loc y_loc z_loc ulimit llimit color">
     <joint name="${joint_name}_joint" type="revolute">
       <origin xyz="${x_loc} ${y_loc} ${z_loc}" rpy="0 0 0" />
@@ -186,5 +177,5 @@
           <mesh filename="package://turtlebot_arm_description/meshes/F2.stl" scale="${M_SCALE} ${M_SCALE} ${M_SCALE}"/>
         </geometry>
-        <material name="white"/>
+        <material name="${color}"/>
       </visual>
       <collision>
@@ -196,5 +187,5 @@
     </link>
   </macro>
- <macro name="bioloid_F4_revolute" params="parent number joint_name x_loc y_loc z_loc">
+  <macro name="bioloid_F4_revolute" params="parent number joint_name x_loc y_loc z_loc color">
     <joint name="${joint_name}_joint" type="revolute">
       <origin xyz="${x_loc} ${y_loc} ${z_loc}" rpy="0 0 0" />
@@ -217,5 +208,5 @@
           <mesh filename="package://turtlebot_arm_description/meshes/F4.stl" scale="${M_SCALE} ${M_SCALE} ${M_SCALE}"/>
         </geometry>
-        <material name="white"/>
+        <material name="${color}"/>
       </visual>
       <collision>

Commit message: Make arm reusable

File: turtlebot_arm_description/urdf/arm.urdf.xacro (robot description, xacro)
@@ -8,4 +8,6 @@
     <include filename="$(find turtlebot_arm_description)/urdf/arm.xacro" />
     <turtlebot />
-    <turtlebot_arm color="white" gripper_color="green"/>
+    <turtlebot_arm parent="plate_3_link" color="white" gripper_color="green">
+      <origin xyz="0.1143 0 0.0508"/>
+    </turtlebot_arm>
 </robot>

File: turtlebot_arm_description/urdf/arm.xacro (robot description, xacro)
@@ -11,48 +11,47 @@
     <color rgba="0.22 0.32 0.14 1.0"/>
   </material>
-  <macro name="turtlebot_arm" params="color gripper_color">
-    <!-- fake arm_base_link joint -->
+  <macro name="turtlebot_arm" params="parent color gripper_color *origin">
     <link name="arm_base_link" />
     <joint name="arm_base_joint" type="fixed">
-      <origin xyz="0 0 0 " rpy="-${M_PI/2} -${M_PI/2} 0" />
-      <parent link="dynamixel_AX12_0_link"/>
+      <insert_block name="origin" />
+      <parent link="${parent}"/>
       <child link="arm_base_link" />
     </joint>
-      <!-- fake gripper_link joint -->
-      <link name="gripper_link" />
-      <joint name="gripper_link_joint" type="fixed">
-        <origin xyz="0 0 .112" rpy="0 -${M_PI/2} 0" />
-        <parent link="bioloid_F2_0_link"/>
-        <child link="gripper_link" />
-      </joint>
-      <!-- shoulder pan joint -->
-      <dynamixel_AX12_fixed parent="plate_3_link" number="0" x_loc="0.1143" y_loc="0" z_loc="${0.0508-AX12_WIDTH/2}" r="${M_PI/2}" p="0" y="${M_PI/2}"/>
-      <bioloid_F3_revolute parent="arm_base_link" number="0" joint_name="shoulder_pan" x_loc="0" y_loc="0" z_loc="${AX12_WIDTH/2}" r="${-M_PI}" p="0" y="${M_PI}" color="${color}"/>
-      <dynamixel_AX12_fixed parent="bioloid_F3_0_link" number="1" x_loc="0" y_loc="0" z_loc="${-AX12_HEIGHT-F10_HEIGHT+0.001}" r="0" p="${M_PI}" y="0"/>
-      <!--shoulder lift joint -->
-      <bioloid_F4_revolute parent="dynamixel_AX12_1_link" number="0" joint_name="shoulder_lift" x_loc="0" y_loc="0" z_loc="0" color="${color}"/>
-      <bioloid_F10_fixed parent="bioloid_F4_0_link" number="0" x_loc="0" y_loc="0" z_loc="${F4_HEIGHT+F10_HEIGHT/2}" color="${color}"/>
-      <bioloid_F10_fixed parent="bioloid_F10_0_link" number="1" x_loc="0" y_loc="0" z_loc="${F10_HEIGHT}" color="${color}"/>
-      <bioloid_F10_fixed parent="bioloid_F10_1_link" number="2" x_loc="0" y_loc="0" z_loc="${F10_HEIGHT}" color="${color}"/>
-      <bioloid_F3_fixed parent="bioloid_F10_2_link" number="1" x_loc="0" y_loc="0" z_loc="${F10_HEIGHT/2}" r="0" p="${M_PI}" y="0" color="${color}"/>
-      <!--elbow joint -->
-      <dynamixel_AX12_fixed parent="bioloid_F3_1_link" number="2" x_loc="0" y_loc="0" z_loc="${-AX12_HEIGHT-F10_HEIGHT+0.001}" r="0" p="${M_PI}" y="0"/>
-      <bioloid_F4_revolute parent="dynamixel_AX12_2_link" number="1" joint_name="elbow_flex" x_loc="0" y_loc="0" z_loc="0" color="${color}"/>
-      <bioloid_F10_fixed parent="bioloid_F4_1_link" number="3" x_loc="0" y_loc="0" z_loc="${F4_HEIGHT+F10_HEIGHT/2}" color="${color}"/>
-      <bioloid_F10_fixed parent="bioloid_F10_3_link" number="4" x_loc="0" y_loc="0" z_loc="${F10_HEIGHT}" color="${color}"/>
-      <bioloid_F10_fixed parent="bioloid_F10_4_link" number="5" x_loc="0" y_loc="0" z_loc="${F10_HEIGHT}" color="${color}"/>
-      <bioloid_F3_fixed parent="bioloid_F10_5_link" number="2" x_loc="0" y_loc="0" z_loc="${F10_HEIGHT/2}" r="0" p="${M_PI}" y="0" color="${color}"/>
-      <!--wrist joint-->
-      <dynamixel_AX12_fixed parent="bioloid_F3_2_link" number="3" x_loc="0" y_loc="0" z_loc="${-AX12_HEIGHT-F10_HEIGHT+0.001}" r="0" p="${M_PI}" y="0"/>
-      <bioloid_F2_revolute parent="dynamixel_AX12_3_link" number="0" joint_name="wrist_flex" x_loc="0" y_loc="0" z_loc="0" ulimit="2.0" llimit="-2.0" color="${color}"/>
-      <bioloid_F3_fixed parent="bioloid_F2_0_link" number="3" x_loc="0.000" y_loc="-0.016" z_loc="${F2_HEIGHT}" r="0" p="${M_PI}" y="${M_PI/2}" color="${color}"/>
-      <!--gripper joint -->
-      <dynamixel_AX12_fixed parent="bioloid_F3_3_link" number="4" x_loc="-0.02275" y_loc="0" z_loc="${-AX12_WIDTH/2}" r="${M_PI}" p="${M_PI/2}" y="0"/>
-      <!--finger 1-->
-      <bioloid_F2_revolute parent="dynamixel_AX12_4_link" number="1" joint_name="gripper" x_loc="0" y_loc="0" z_loc="0" ulimit="0.50" llimit="-0.60" color="${color}"/>
-      <finger_fixed parent="bioloid_F2_1_link" number="0" x_loc="0" y_loc="0" z_loc="${F2_HEIGHT}" r="0" p="0" y="0" color="${gripper_color}"/>
-      <!--finger 2-->
-      <bioloid_F3_fixed parent="dynamixel_AX12_4_link" number="4" x_loc="0" y_loc="0" z_loc="${-AX12_HEIGHT-F10_HEIGHT+0.001}" r="0" p="${M_PI}" y="0" color="${color}"/>
-      <finger_fixed parent="bioloid_F3_4_link" number="1" x_loc="0" y_loc="0" z_loc="0" r="0" p="0" y="${M_PI}" color="${gripper_color}"/>
+    <!-- fake gripper_link joint -->
+    <link name="gripper_link" />
+    <joint name="gripper_link_joint" type="fixed">
+      <origin xyz="0 0 .112" rpy="0 -${M_PI/2} 0" />
+      <parent link="bioloid_F2_0_link"/>
+      <child link="gripper_link" />
+    </joint>
+    <!-- shoulder pan joint -->
+    <dynamixel_AX12_fixed parent="arm_base_link" number="0" x_loc="0" y_loc="0" z_loc="${-AX12_WIDTH/2}" r="${M_PI/2}" p="0" y="${M_PI/2}"/>
+    <bioloid_F3_revolute parent="dynamixel_AX12_0_link" number="0" joint_name="shoulder_pan" x_loc="0" y_loc="${AX12_WIDTH/2}" z_loc="0" r="${-M_PI/2}" p="${M_PI/2}" y="${M_PI}" color="${color}"/>
+    <dynamixel_AX12_fixed parent="bioloid_F3_0_link" number="1" x_loc="0" y_loc="0" z_loc="${-AX12_HEIGHT-F10_HEIGHT+0.001}" r="0" p="${M_PI}" y="0"/>
+    <!--shoulder lift joint -->
+    <bioloid_F4_revolute parent="dynamixel_AX12_1_link" number="0" joint_name="shoulder_lift" x_loc="0" y_loc="0" z_loc="0" color="${color}"/>
+    <bioloid_F10_fixed parent="bioloid_F4_0_link" number="0" x_loc="0" y_loc="0" z_loc="${F4_HEIGHT+F10_HEIGHT/2}" color="${color}"/>
+    <bioloid_F10_fixed parent="bioloid_F10_0_link" number="1" x_loc="0" y_loc="0" z_loc="${F10_HEIGHT}" color="${color}"/>
+    <bioloid_F10_fixed parent="bioloid_F10_1_link" number="2" x_loc="0" y_loc="0" z_loc="${F10_HEIGHT}" color="${color}"/>
+    <bioloid_F3_fixed parent="bioloid_F10_2_link" number="1" x_loc="0" y_loc="0" z_loc="${F10_HEIGHT/2}" r="0" p="${M_PI}" y="0" color="${color}"/>
+    <!--elbow joint -->
+    <dynamixel_AX12_fixed parent="bioloid_F3_1_link" number="2" x_loc="0" y_loc="0" z_loc="${-AX12_HEIGHT-F10_HEIGHT+0.001}" r="0" p="${M_PI}" y="0"/>
+    <bioloid_F4_revolute parent="dynamixel_AX12_2_link" number="1" joint_name="elbow_flex" x_loc="0" y_loc="0" z_loc="0" color="${color}"/>
+    <bioloid_F10_fixed parent="bioloid_F4_1_link" number="3" x_loc="0" y_loc="0" z_loc="${F4_HEIGHT+F10_HEIGHT/2}" color="${color}"/>
+    <bioloid_F10_fixed parent="bioloid_F10_3_link" number="4" x_loc="0" y_loc="0" z_loc="${F10_HEIGHT}" color="${color}"/>
+    <bioloid_F10_fixed parent="bioloid_F10_4_link" number="5" x_loc="0" y_loc="0" z_loc="${F10_HEIGHT}" color="${color}"/>
+    <bioloid_F3_fixed parent="bioloid_F10_5_link" number="2" x_loc="0" y_loc="0" z_loc="${F10_HEIGHT/2}" r="0" p="${M_PI}" y="0" color="${color}"/>
+    <!--wrist joint-->
+    <dynamixel_AX12_fixed parent="bioloid_F3_2_link" number="3" x_loc="0" y_loc="0" z_loc="${-AX12_HEIGHT-F10_HEIGHT+0.001}" r="0" p="${M_PI}" y="0"/>
+    <bioloid_F2_revolute parent="dynamixel_AX12_3_link" number="0" joint_name="wrist_flex" x_loc="0" y_loc="0" z_loc="0" ulimit="2.0" llimit="-2.0" color="${color}"/>
+    <bioloid_F3_fixed parent="bioloid_F2_0_link" number="3" x_loc="0.000" y_loc="-0.016" z_loc="${F2_HEIGHT}" r="0" p="${M_PI}" y="${M_PI/2}" color="${color}"/>
+    <!--gripper joint -->
+    <dynamixel_AX12_fixed parent="bioloid_F3_3_link" number="4" x_loc="-0.02275" y_loc="0" z_loc="${-AX12_WIDTH/2}" r="${M_PI}" p="${M_PI/2}" y="0"/>
+    <!--finger 1-->
+    <bioloid_F2_revolute parent="dynamixel_AX12_4_link" number="1" joint_name="gripper" x_loc="0" y_loc="0" z_loc="0" ulimit="0.50" llimit="-0.60" color="${color}"/>
+    <finger_fixed parent="bioloid_F2_1_link" number="0" x_loc="0" y_loc="0" z_loc="${F2_HEIGHT}" r="0" p="0" y="0" color="${gripper_color}"/>
+    <!--finger 2-->
+    <bioloid_F3_fixed parent="dynamixel_AX12_4_link" number="4" x_loc="0" y_loc="0" z_loc="${-AX12_HEIGHT-F10_HEIGHT+0.001}" r="0" p="${M_PI}" y="0" color="${color}"/>
+    <finger_fixed parent="bioloid_F3_4_link" number="1" x_loc="0" y_loc="0" z_loc="0" r="0" p="0" y="${M_PI}" color="${gripper_color}"/>
   </macro>
 </robot>
