Commit message: Add an indigo-devel branch. More details in the readme

File: turtlebot_arm_description/urdf/arm.urdf.xacro (robot description, xacro)
@@ -1,4 +1,4 @@
 <?xml version="1.0"?>
-<robot name="turtlebot_arm"
+<robot name="turtlebot_arm" xmlns:xacro="http://ros.org/wiki/xacro"
     xmlns:sensor="http://playerstage.sourceforge.net/gazebo/xmlschema/#sensor"
     xmlns:controller="http://playerstage.sourceforge.net/gazebo/xmlschema/#controller"
@@ -6,11 +6,17 @@
     <!-- Included URDF Files -->
     <!--<include filename="$(find turtlebot_description)/urdf/turtlebot.urdf.xacro" />-->
-    <include filename="$(find turtlebot_arm_description)/urdf/arm.xacro" />
+    <xacro:include filename="$(find turtlebot_arm_description)/urdf/arm.xacro" />
     <!-- For now I have removed the turtlebot since this all moved around..
     <turtlebot />-->
-    <!-- Instead, there is a base_link -->
-    <link name="base_link"/>
-    <turtlebot_arm parent="base_link" color="white" gripper_color="green">
-      <origin xyz="0 0 0"/>
+    <!-- Instead, add a base_footprint link as turtlebot location reference -->
+    <link name="base_footprint"/>
+    <!-- Turtlebot arm macro: we can configure joints velocity limit and lower/upper limits
+         for the first joint (arm_shoulder_pan) to allow accessing to different operational
+         areas, e.g. left handed vs. right handed robot -->
+    <turtlebot_arm parent="base_footprint" color="white" gripper_color="green"
+                   joints_vlimit="1.571" pan_llimit="-2.617" pan_ulimit="2.617">
+      <!-- Place the "floating" arm at the location it should be if mounted on a turtlebot,
+           as pick and place and other demos assume this location -->
+      <origin xyz="0.1 0.03 0.435"/>
     </turtlebot_arm>
 </robot>

File: turtlebot_arm_description/urdf/arm.xacro (robot description, xacro)
@@ -1,5 +1,5 @@
 <?xml version="1.0"?>
-<robot>
-  <include filename="$(find turtlebot_arm_description)/urdf/arm_hardware.xacro" />
+<robot xmlns:xacro="http://ros.org/wiki/xacro">
+  <xacro:include filename="$(find turtlebot_arm_description)/urdf/arm_hardware.xacro"/>
   <material name="white">
     <color rgba="0.87 0.90 0.87 1.0"/>
@@ -11,5 +11,6 @@
     <color rgba="0.22 0.32 0.14 1.0"/>
   </material>
-  <macro name="turtlebot_arm" params="parent color gripper_color *origin">
+  <xacro:macro name="turtlebot_arm" params="parent color gripper_color *origin
+                                            joints_vlimit pan_llimit pan_ulimit">
     <link name="arm_base_link" />
     <joint name="arm_base_joint" type="fixed">
@@ -33,5 +34,6 @@
       <origin xyz="0 0 0" rpy="${M_PI/2} 0 ${M_PI/2}"/>
     </dynamixel_AX12_fixed>
-    <bioloid_F3_revolute parent="arm_shoulder_pan_servo_link" name="arm_shoulder_pan" color="${color}" vlimit="0.785" llimit="-2.617" ulimit="2.617">
+    <bioloid_F3_revolute parent="arm_shoulder_pan_servo_link" name="arm_shoulder_pan" color="${color}"
+                         vlimit="${joints_vlimit}" llimit="${pan_llimit}" ulimit="${pan_ulimit}">
       <origin xyz="0 ${AX12_WIDTH/2} 0" rpy="${-M_PI/2} ${M_PI/2} ${M_PI}" />
     </bioloid_F3_revolute>
@@ -40,5 +42,6 @@
       <origin xyz="0 0 ${-AX12_HEIGHT-F10_HEIGHT+0.001}" rpy="0 ${M_PI} 0" />
     </dynamixel_AX12_fixed>
-    <bioloid_F4_revolute parent="arm_shoulder_lift_servo_link" name="arm_shoulder_lift" color="${color}" vlimit="1.571" llimit="-2.617" ulimit="2.617">
+    <bioloid_F4_revolute parent="arm_shoulder_lift_servo_link" name="arm_shoulder_lift" color="${color}"
+                         vlimit="${joints_vlimit}" llimit="-2.617" ulimit="2.617">
       <origin xyz="0 0 0" rpy="0 0 0" />
     </bioloid_F4_revolute>
@@ -59,5 +62,6 @@
       <origin xyz="0 0 ${-AX12_HEIGHT-F10_HEIGHT+0.001}" rpy="0 ${M_PI} 0"/>
     </dynamixel_AX12_fixed>
-    <bioloid_F4_revolute parent="arm_elbow_flex_servo_link" name="arm_elbow_flex" color="${color}" vlimit="1.571" llimit="-2.617" ulimit="2.617">
+    <bioloid_F4_revolute parent="arm_elbow_flex_servo_link" name="arm_elbow_flex" color="${color}"
+                         vlimit="${joints_vlimit}" llimit="-2.617" ulimit="2.617">
       <origin xyz="0 0 0" rpy="0 0 0" />
     </bioloid_F4_revolute>
@@ -78,5 +82,6 @@
       <origin xyz="0 0 ${-AX12_HEIGHT-F10_HEIGHT+0.001}" rpy="0 ${M_PI} 0"/>
     </dynamixel_AX12_fixed>
-    <bioloid_F2_revolute parent="arm_wrist_flex_servo_link" name="arm_wrist_flex" color="${color}" vlimit="1.571" llimit="-1.745" ulimit="1.745">
+    <bioloid_F2_revolute parent="arm_wrist_flex_servo_link" name="arm_wrist_flex" color="${color}"
+                         vlimit="${joints_vlimit}" llimit="-1.745" ulimit="1.745">
       <origin xyz="0 0 0" rpy="0 0 0" />
     </bioloid_F2_revolute>
@@ -128,4 +133,4 @@
       <origin xyz="0 0 0" rpy="0 0 ${M_PI}" />
     </finger_fixed>
-  </macro>
+  </xacro:macro>
 </robot>
