Commit message: Add Gazebo support, including realistic weights on inertia tags. Note that I use now capitalized color names so they match [Gazebo materials](http://wiki.ros.org/simulator_gazebo/Tutorials/ListOfMaterials)

File: turtlebot_arm_description/urdf/arm.urdf.xacro (robot description, xacro)
@@ -5,5 +5,5 @@
     xmlns:interface="http://playerstage.sourceforge.net/gazebo/xmlschema/#interface">
     <!-- Included URDF Files -->
-    <xacro:include filename="$(find turtlebot_arm_description)/urdf/arm.xacro" />
+    <xacro:include filename="$(find turtlebot_arm_description)/urdf/arm.xacro"/>
     <!-- As we don't have here a turtlebot, add a base_link link as its location reference -->
     <link name="base_link"/>
@@ -11,5 +11,5 @@
          for the first joint (arm_shoulder_pan) to allow accessing to different operational
          areas, e.g. left handed vs. right handed robot -->
-    <turtlebot_arm parent="base_link" color="white" gripper_color="green"
+    <turtlebot_arm parent="base_link" color="White" gripper_color="Green"
                    joints_vlimit="1.571" pan_llimit="-2.617" pan_ulimit="2.617">
       <!-- Place the "floating" arm at the location it should be if mounted on a turtlebot,

File: turtlebot_arm_description/urdf/arm.xacro (robot description, xacro)
@@ -2,29 +2,29 @@
 <robot xmlns:xacro="http://ros.org/wiki/xacro">
   <xacro:include filename="$(find turtlebot_arm_description)/urdf/arm_hardware.xacro"/>
-  <material name="white">
+  <material name="White">
     <color rgba="0.87 0.90 0.87 1.0"/>
   </material>
-  <material name="black">
+  <material name="Black">
     <color rgba="0.0 0.0 0.0 1.0"/>
   </material>
-  <material name="green">
+  <material name="Green">
     <color rgba="0.22 0.32 0.14 1.0"/>
   </material>
   <xacro:macro name="turtlebot_arm" params="parent color gripper_color *origin
                                             joints_vlimit pan_llimit pan_ulimit">
-    <link name="arm_base_link" />
+    <link name="arm_base_link"/>
     <joint name="arm_base_joint" type="fixed">
-      <insert_block name="origin" />
+      <insert_block name="origin"/>
       <parent link="${parent}"/>
-      <child link="arm_base_link" />
+      <child link="arm_base_link"/>
     </joint>
     <!-- fake gripper_link joint gives us a free servo!
          this makes us 5DOF and saves you $44.90
          that's a lot of coin! -->
-    <link name="gripper_link" />
+    <link name="gripper_link"/>
     <joint name="gripper_link_joint" type="revolute">
-      <origin xyz="0 0 .112" rpy="0 -1.57 0" />
+      <origin xyz="0 0 .112" rpy="0 -1.57 0"/>
       <parent link="arm_wrist_flex_link"/>
-      <child link="gripper_link" />
+      <child link="gripper_link"/>
       <limit effort="30" velocity="1" lower="-3.14" upper="3.14"/>
       <axis xyz="1 0 0"/>
@@ -36,25 +36,25 @@
     <bioloid_F3_revolute parent="arm_shoulder_pan_servo_link" name="arm_shoulder_pan" color="${color}"
                          vlimit="${joints_vlimit}" llimit="${pan_llimit}" ulimit="${pan_ulimit}">
-      <origin xyz="0 ${AX12_WIDTH/2} 0" rpy="${-M_PI/2} ${M_PI/2} ${M_PI}" />
+      <origin xyz="0 ${AX12_WIDTH/2} 0" rpy="${-M_PI/2} ${M_PI/2} ${M_PI}"/>
     </bioloid_F3_revolute>
     <!-- shoulder lift joint -->
     <dynamixel_AX12_fixed parent="arm_shoulder_pan_link" name="arm_shoulder_lift_servo">
-      <origin xyz="0 0 ${-AX12_HEIGHT-F10_HEIGHT+0.001}" rpy="0 ${M_PI} 0" />
+      <origin xyz="0 0 ${-AX12_HEIGHT-F10_HEIGHT+0.001}" rpy="0 ${M_PI} 0"/>
     </dynamixel_AX12_fixed>
     <bioloid_F4_revolute parent="arm_shoulder_lift_servo_link" name="arm_shoulder_lift" color="${color}"
                          vlimit="${joints_vlimit}" llimit="-2.617" ulimit="2.617">
-      <origin xyz="0 0 0" rpy="0 0 0" />
+      <origin xyz="0 0 0" rpy="0 0 0"/>
     </bioloid_F4_revolute>
     <bioloid_F10_fixed parent="arm_shoulder_lift_link" name="arm_shoulder_F10_0" color="${color}">
-      <origin xyz="0 0 ${F4_HEIGHT+F10_HEIGHT/2}" rpy="0 0 0" />
+      <origin xyz="0 0 ${F4_HEIGHT+F10_HEIGHT/2}" rpy="0 0 0"/>
     </bioloid_F10_fixed>
     <bioloid_F10_fixed parent="arm_shoulder_F10_0_link" name="arm_shoulder_F10_1" color="${color}">
-      <origin xyz="0 0 ${F10_HEIGHT}" rpy="0 0 0" />
+      <origin xyz="0 0 ${F10_HEIGHT}" rpy="0 0 0"/>
     </bioloid_F10_fixed>
     <bioloid_F10_fixed parent="arm_shoulder_F10_1_link" name="arm_shoulder_F10_2" color="${color}">
-      <origin xyz="0 0 ${F10_HEIGHT}" rpy="0 0 0" />
+      <origin xyz="0 0 ${F10_HEIGHT}" rpy="0 0 0"/>
     </bioloid_F10_fixed>
     <bioloid_F3_fixed parent="arm_shoulder_F10_2_link" name="arm_shoulder_F3_0" color="${color}">
-      <origin xyz="0 0 ${F10_HEIGHT/2}" rpy="0 ${M_PI} 0" />
+      <origin xyz="0 0 ${F10_HEIGHT/2}" rpy="0 ${M_PI} 0"/>
     </bioloid_F3_fixed>
     <!-- elbow joint -->
@@ -64,17 +64,17 @@
     <bioloid_F4_revolute parent="arm_elbow_flex_servo_link" name="arm_elbow_flex" color="${color}"
                          vlimit="${joints_vlimit}" llimit="-2.617" ulimit="2.617">
-      <origin xyz="0 0 0" rpy="0 0 0" />
+      <origin xyz="0 0 0" rpy="0 0 0"/>
     </bioloid_F4_revolute>
     <bioloid_F10_fixed parent="arm_elbow_flex_link" name="arm_elbow_F10_0" color="${color}">
-      <origin xyz="0 0 ${F4_HEIGHT+F10_HEIGHT/2}" rpy="0 0 0" />
+      <origin xyz="0 0 ${F4_HEIGHT+F10_HEIGHT/2}" rpy="0 0 0"/>
     </bioloid_F10_fixed>
     <bioloid_F10_fixed parent="arm_elbow_F10_0_link" name="arm_elbow_F10_1" color="${color}">
-      <origin xyz="0 0 ${F10_HEIGHT}" rpy="0 0 0" />
+      <origin xyz="0 0 ${F10_HEIGHT}" rpy="0 0 0"/>
     </bioloid_F10_fixed>
     <bioloid_F10_fixed parent="arm_elbow_F10_1_link" name="arm_elbow_F10_2" color="${color}">
-      <origin xyz="0 0 ${F10_HEIGHT}" rpy="0 0 0" />
+      <origin xyz="0 0 ${F10_HEIGHT}" rpy="0 0 0"/>
     </bioloid_F10_fixed>
     <bioloid_F3_fixed parent="arm_elbow_F10_2_link" name="arm_elbow_F3_0" color="${color}">
-      <origin xyz="0 0 ${F10_HEIGHT/2}" rpy="0 ${M_PI} 0" />
+      <origin xyz="0 0 ${F10_HEIGHT/2}" rpy="0 ${M_PI} 0"/>
     </bioloid_F3_fixed>
     <!-- wrist joint -->
@@ -84,8 +84,8 @@
     <bioloid_F2_revolute parent="arm_wrist_flex_servo_link" name="arm_wrist_flex" color="${color}"
                          vlimit="${joints_vlimit}" llimit="-1.745" ulimit="1.745">
-      <origin xyz="0 0 0" rpy="0 0 0" />
+      <origin xyz="0 0 0" rpy="0 0 0"/>
     </bioloid_F2_revolute>
     <bioloid_F3_fixed parent="arm_wrist_flex_link" name="arm_wrist_F3_0" color="${color}">
-      <origin xyz="0 0.016 ${F2_HEIGHT}" rpy="0 ${M_PI} ${-M_PI/2}" />
+      <origin xyz="0 0.016 ${F2_HEIGHT}" rpy="0 ${M_PI} ${-M_PI/2}"/>
     </bioloid_F3_fixed>
     <!-- gripper joint -->
@@ -97,18 +97,18 @@
       <origin xyz="0 0 0" rpy="0 0 0"/>
       <axis xyz="0 1 0"/>
-      <limit effort="30" velocity="0.785" lower="-0.40" upper="0.46" />
+      <limit effort="30" velocity="0.785" lower="-0.40" upper="0.46"/>
       <parent link="gripper_servo_link"/>
-      <child link="gripper_active_link" />
+      <child link="gripper_active_link"/>
     </joint>
     <link name="gripper_active_link">
       <inertial>
-        <mass value="0.00001" />
-        <origin xyz="0 0 0" />
+        <mass value="0.00001"/>
+        <origin xyz="0 0 0"/>
         <inertia ixx="1.0" ixy="0.0" ixz="0.0"
           iyy="1.0" iyz="0.0"
-          izz="1.0" />
+          izz="1.0"/>
       </inertial>
       <visual>
-        <origin xyz=" 0 0 0 " rpy="0 0 0" />
+        <origin xyz=" 0 0 0 " rpy="0 0 0"/>
         <geometry>
           <mesh filename="package://turtlebot_arm_description/meshes/F2.stl" scale="${M_SCALE} ${M_SCALE} ${M_SCALE}"/>
@@ -117,5 +117,5 @@
       </visual>
       <collision>
-        <origin xyz="0.0 0.0 0.00775" rpy="0 0 0" />
+        <origin xyz="0.0 0.0 0.00775" rpy="0 0 0"/>
         <geometry>
           <box size="0.025 0.0485 0.0375"/>
@@ -124,12 +124,12 @@
     </link>
     <finger_fixed parent="gripper_active_link" name="gripper_active_finger" color="${gripper_color}">
-      <origin xyz="0 0 ${F2_HEIGHT}" rpy="0 0 0" />
+      <origin xyz="0 0 ${F2_HEIGHT}" rpy="0 0 0"/>
     </finger_fixed>
     <!-- finger 2 -->
     <bioloid_F3_fixed parent="gripper_servo_link" name="gripper_static" color="${color}">
-      <origin xyz="0 0 ${-AX12_HEIGHT-F10_HEIGHT+0.001}" rpy="0 ${M_PI} 0" />
+      <origin xyz="0 0 ${-AX12_HEIGHT-F10_HEIGHT+0.001}" rpy="0 ${M_PI} 0"/>
     </bioloid_F3_fixed>
     <finger_fixed parent="gripper_static_link" name="gripper_static_finger" color="${gripper_color}">
-      <origin xyz="0 0 0" rpy="0 0 ${M_PI}" />
+      <origin xyz="0 0 0" rpy="0 0 ${M_PI}"/>
     </finger_fixed>
   </xacro:macro>

File: turtlebot_arm_description/urdf/arm_hardware.xacro (robot description, xacro)
@@ -9,20 +9,122 @@
   <xacro:property name="AX12_WIDTH" value="0.038"/>
   <xacro:property name="F2_HEIGHT" value="0.0265"/>
+  <xacro:macro name="arm_mount" params="parent name color *origin">
+    <joint name="${name}_joint" type="fixed">
+      <insert_block name="origin"/>
+      <parent link="${parent}"/>
+      <child link="${name}_link"/>
+    </joint>
+    <link name="${name}_link">
+      <inertial>
+        <mass value="0.018"/>
+        <origin xyz="0 0 0"/>
+        <inertia ixx="1.0" ixy="0.0" ixz="0.0"
+                 iyy="1.0" iyz="0.0"
+                 izz="1.0"/>
+      </inertial>
+      <visual>
+        <origin xyz="-0.028 -0.0493 0.014" rpy="0.0 0.0 -${M_PI/2}"/>
+        <geometry>
+          <mesh filename="package://turtlebot_arm_description/meshes/mount.stl" scale="${M_SCALE} ${M_SCALE} ${M_SCALE}"/>
+        </geometry>
+        <material name="${color}"/>
+      </visual>
+      <collision>
+        <origin xyz="-0.01 0.0 0.0165" rpy="0.0 0.0 0.0"/>
+        <geometry>
+          <box size="0.074 0.074 0.004"/>
+        </geometry>
+      </collision>
+    </link>
+    <gazebo reference="${name}_link">
+      <material>Gazebo/${color}</material>
+      <selfCollide>true</selfCollide>
+      <gravity>true</gravity>
+    </gazebo>
+  </xacro:macro>
+  <xacro:macro name="finger_fixed" params="parent name color *origin">
+    <joint name="${name}_joint" type="fixed">
+      <insert_block name="origin"/>
+      <parent link="${parent}"/>
+      <child link="${name}_link"/>
+    </joint>
+    <link name="${name}_link">
+      <inertial>
+        <mass value="0.015"/>
+        <origin xyz="0 0 0"/>
+        <inertia ixx="1.0" ixy="0.0" ixz="0.0"
+                 iyy="1.0" iyz="0.0"
+                 izz="1.0"/>
+      </inertial>
+      <visual>
+        <origin xyz=" 0 0 0 " rpy="0 0 0"/>
+        <geometry>
+          <mesh filename="package://turtlebot_arm_description/meshes/finger.stl" scale="${M_SCALE} ${M_SCALE} ${M_SCALE}"/>
+        </geometry>
+        <material name="${color}"/>
+      </visual>
+      <collision>
+        <origin xyz="0.02645 0.0 -0.00655" rpy="0 0 0"/>
+        <geometry>
+          <box size="0.0783 0.03801 0.0193"/>
+        </geometry>
+      </collision>
+    </link>
+    <gazebo reference="${name}_link">
+      <material>Gazebo/${color}</material>
+      <selfCollide>true</selfCollide>
+      <gravity>true</gravity>
+    </gazebo>
+  </xacro:macro>
+  <xacro:macro name="dynamixel_AX12_fixed" params="parent name *origin">
+    <joint name="${name}_joint" type="fixed">
+      <insert_block name="origin"/>
+      <parent link="${parent}"/>
+      <child link="${name}_link"/>
+    </joint>
+    <link name="${name}_link">
+      <inertial>
+        <mass value="0.055"/>
+        <origin xyz="0 0 0"/>
+        <inertia ixx="1.0" ixy="0.0" ixz="0.0"
+                 iyy="1.0" iyz="0.0"
+                 izz="1.0"/>
+      </inertial>
+      <visual>
+        <origin xyz=" 0 0 0 " rpy="0 0 0"/>
+        <geometry>
+          <mesh filename="package://turtlebot_arm_description/meshes/ax12_box.stl" scale="${M_SCALE} ${M_SCALE} ${M_SCALE}"/>
+        </geometry>
+        <material name="black"/>
+      </visual>
+      <collision>
+        <origin xyz="0.0 0.0 -0.01241" rpy="0 0 0"/>
+        <geometry>
+          <box size="0.025 0.038 0.04762"/>
+        </geometry>
+      </collision>
+    </link>
+    <gazebo reference="${name}_link">
+      <material>Gazebo/Black</material>
+      <selfCollide>true</selfCollide>
+      <gravity>true</gravity>
+    </gazebo>
+  </xacro:macro>
   <xacro:macro name="bioloid_F10_fixed" params="parent name color *origin">
     <joint name="${name}_joint" type="fixed">
-      <insert_block name="origin" />
-      <parent link="${parent}"/>
-      <child link="${name}_link" />
-    </joint>
-    <link name="${name}_link">
-      <inertial>
-        <mass value="0.00001" />
-        <origin xyz="0 0 0" />
-        <inertia ixx="1.0" ixy="0.0" ixz="0.0"
-          iyy="1.0" iyz="0.0"
-          izz="1.0" />
-      </inertial>
-      <visual>
-        <origin xyz=" 0 0 0 " rpy="0 0 0" />
+      <insert_block name="origin"/>
+      <parent link="${parent}"/>
+      <child link="${name}_link"/>
+    </joint>
+    <link name="${name}_link">
+      <inertial>
+        <mass value="0.004"/>
+        <origin xyz="0 0 0"/>
+        <inertia ixx="1.0" ixy="0.0" ixz="0.0"
+                 iyy="1.0" iyz="0.0"
+                 izz="1.0"/>
+      </inertial>
+      <visual>
+        <origin xyz=" 0 0 0 " rpy="0 0 0"/>
         <geometry>
           <mesh filename="package://turtlebot_arm_description/meshes/F10.stl" scale="${M_SCALE} ${M_SCALE} ${M_SCALE}"/>
@@ -31,5 +133,5 @@
       </visual>
       <collision>
-        <origin xyz="0.0 0.0 0.0" rpy="0 0 0" />
+        <origin xyz="0.0 0.0 0.0" rpy="0 0 0"/>
         <geometry>
           <box size="0.025 0.038 0.004"/>
@@ -37,79 +139,26 @@
       </collision>
     </link>
-  </xacro:macro>
-  <xacro:macro name="arm_mount" params="parent name color *origin">
-    <joint name="${name}_joint" type="fixed">
-      <insert_block name="origin" />
-      <parent link="${parent}"/>
-      <child link="${name}_link" />
-    </joint>
-    <link name="${name}_link">
-      <inertial>
-        <mass value="0.00001" />
-        <origin xyz="0 0 0" />
-        <inertia ixx="1.0" ixy="0.0" ixz="0.0"
-          iyy="1.0" iyz="0.0"
-          izz="1.0" />
-      </inertial>
-      <visual>
-        <origin xyz="-0.028 -0.0493 0.014" rpy="0.0 0.0 -${M_PI/2}" />
-        <geometry>
-          <mesh filename="package://turtlebot_arm_description/meshes/mount.stl" scale="${M_SCALE} ${M_SCALE} ${M_SCALE}"/>
-        </geometry>
-        <material name="${color}"/>
-      </visual>
-      <collision>
-        <origin xyz="-0.01 0.0 0.0165" rpy="0.0 0.0 0.0" />
-        <geometry>
-          <box size="0.074 0.074 0.004"/>
-        </geometry>
-      </collision>
-    </link>
-  </xacro:macro>
-  <xacro:macro name="finger_fixed" params="parent name color *origin">
-    <joint name="${name}_joint" type="fixed">
-      <insert_block name="origin" />
-      <parent link="${parent}"/>
-      <child link="${name}_link" />
-    </joint>
-    <link name="${name}_link">
-      <inertial>
-        <mass value="0.00001" />
-        <origin xyz="0 0 0" />
-        <inertia ixx="1.0" ixy="0.0" ixz="0.0"
-          iyy="1.0" iyz="0.0"
-          izz="1.0" />
-      </inertial>
-      <visual>
-        <origin xyz=" 0 0 0 " rpy="0 0 0" />
-        <geometry>
-          <mesh filename="package://turtlebot_arm_description/meshes/finger.stl" scale="${M_SCALE} ${M_SCALE} ${M_SCALE}"/>
-        </geometry>
-        <material name="${color}"/>
-      </visual>
-      <collision>
-        <origin xyz="0.02645 0.0 -0.00655" rpy="0 0 0" />
-        <geometry>
-          <box size="0.0783 0.03801 0.0193"/>
-        </geometry>
-      </collision>
-    </link>
+    <gazebo reference="${name}_link">
+      <material>Gazebo/${color}</material>
+      <selfCollide>true</selfCollide>
+      <gravity>true</gravity>
+    </gazebo>
   </xacro:macro>
   <xacro:macro name="bioloid_F3_fixed" params="parent name color *origin">
     <joint name="${name}_joint" type="fixed">
-      <insert_block name="origin" />
-      <parent link="${parent}"/>
-      <child link="${name}_link" />
-    </joint>
-    <link name="${name}_link">
-      <inertial>
-        <mass value="0.00001" />
-        <origin xyz="0 0 0" />
-        <inertia ixx="1.0" ixy="0.0" ixz="0.0"
-          iyy="1.0" iyz="0.0"
-          izz="1.0" />
-      </inertial>
-      <visual>
-        <origin xyz=" 0 0 0 " rpy="0 0 0" />
+      <insert_block name="origin"/>
+      <parent link="${parent}"/>
+      <child link="${name}_link"/>
+    </joint>
+    <link name="${name}_link">
+      <inertial>
+        <mass value="0.005"/>
+        <origin xyz="0 0 0"/>
+        <inertia ixx="1.0" ixy="0.0" ixz="0.0"
+                 iyy="1.0" iyz="0.0"
+                 izz="1.0"/>
+      </inertial>
+      <visual>
+        <origin xyz=" 0 0 0 " rpy="0 0 0"/>
         <geometry>
           <mesh filename="package://turtlebot_arm_description/meshes/F3.stl" scale="${M_SCALE} ${M_SCALE} ${M_SCALE}"/>
@@ -118,5 +167,5 @@
       </visual>
       <collision>
-        <origin xyz="0.0 0.0 -0.0045" rpy="0 0 0" />
+        <origin xyz="0.0 0.0 -0.0045" rpy="0 0 0"/>
         <geometry>
           <box size="0.025 0.038 0.009"/>
@@ -124,52 +173,28 @@
       </collision>
     </link>
-  </xacro:macro>
-  <xacro:macro name="dynamixel_AX12_fixed" params="parent name *origin">
-    <joint name="${name}_joint" type="fixed">
-      <insert_block name="origin" />
-      <parent link="${parent}"/>
-      <child link="${name}_link" />
-    </joint>
-    <link name="${name}_link">
-      <inertial>
-        <mass value="0.00001" />
-        <origin xyz="0 0 0" />
-        <inertia ixx="1.0" ixy="0.0" ixz="0.0"
-          iyy="1.0" iyz="0.0"
-          izz="1.0" />
-      </inertial>
-      <visual>
-        <origin xyz=" 0 0 0 " rpy="0 0 0" />
-        <geometry>
-          <mesh filename="package://turtlebot_arm_description/meshes/ax12_box.stl" scale="${M_SCALE} ${M_SCALE} ${M_SCALE}"/>
-        </geometry>
-        <material name="black"/>
-      </visual>
-      <collision>
-        <origin xyz="0.0 0.0 -0.01241" rpy="0 0 0" />
-        <geometry>
-          <box size="0.025 0.038 0.04762"/>
-        </geometry>
-      </collision>
-    </link>
+    <gazebo reference="${name}_link">
+      <material>Gazebo/${color}</material>
+      <selfCollide>true</selfCollide>
+      <gravity>true</gravity>
+    </gazebo>
   </xacro:macro>
   <xacro:macro name="bioloid_F3_revolute" params="parent name color llimit ulimit vlimit *origin">
     <joint name="${name}_joint" type="revolute">
-      <insert_block name="origin" />
+      <insert_block name="origin"/>
       <axis xyz="0 0 -1"/>
-      <limit effort="30" velocity="${vlimit}" lower="${llimit}" upper="${ulimit}" />
-      <parent link="${parent}"/>
-      <child link="${name}_link" />
-    </joint>
-    <link name="${name}_link">
-      <inertial>
-        <mass value="0.00001" />
-        <origin xyz="0 0 0" />
-        <inertia ixx="1.0" ixy="0.0" ixz="0.0"
-          iyy="1.0" iyz="0.0"
-          izz="1.0" />
-      </inertial>
-      <visual>
-        <origin xyz=" 0 0 0 " rpy="0 0 0" />
+      <limit effort="30" velocity="${vlimit}" lower="${llimit}" upper="${ulimit}"/>
+      <parent link="${parent}"/>
+      <child link="${name}_link"/>
+    </joint>
+    <link name="${name}_link">
+      <inertial>
+        <mass value="0.008"/>
+        <origin xyz="0 0 0"/>
+        <inertia ixx="1.0" ixy="0.0" ixz="0.0"
+                 iyy="1.0" iyz="0.0"
+                 izz="1.0"/>
+      </inertial>
+      <visual>
+        <origin xyz=" 0 0 0 " rpy="0 0 0"/>
         <geometry>
           <mesh filename="package://turtlebot_arm_description/meshes/F3.stl" scale="${M_SCALE} ${M_SCALE} ${M_SCALE}"/>
@@ -178,5 +203,5 @@
       </visual>
       <collision>
-        <origin xyz="0.0 0.0 -0.0045" rpy="0 0 0" />
+        <origin xyz="0.0 0.0 -0.0045" rpy="0 0 0"/>
         <geometry>
           <box size="0.025 0.038 0.009"/>
@@ -184,23 +209,28 @@
       </collision>
     </link>
+    <gazebo reference="${name}_link">
+      <material>Gazebo/${color}</material>
+      <selfCollide>true</selfCollide>
+      <gravity>true</gravity>
+    </gazebo>
   </xacro:macro>
   <xacro:macro name="bioloid_F2_revolute" params="parent name color llimit ulimit vlimit *origin">
     <joint name="${name}_joint" type="revolute">
-      <insert_block name="origin" />
+      <insert_block name="origin"/>
       <axis xyz="0 1 0"/>
-      <limit effort="30" velocity="${vlimit}" lower="${llimit}" upper="${ulimit}" />
-      <parent link="${parent}"/>
-      <child link="${name}_link" />
-    </joint>
-    <link name="${name}_link">
-      <inertial>
-        <mass value="0.00001" />
-        <origin xyz="0 0 0" />
-        <inertia ixx="1.0" ixy="0.0" ixz="0.0"
-          iyy="1.0" iyz="0.0"
-          izz="1.0" />
-      </inertial>
-      <visual>
-        <origin xyz=" 0 0 0 " rpy="0 0 0" />
+      <limit effort="30" velocity="${vlimit}" lower="${llimit}" upper="${ulimit}"/>
+      <parent link="${parent}"/>
+      <child link="${name}_link"/>
+    </joint>
+    <link name="${name}_link">
+      <inertial>
+        <mass value="0.010"/>
+        <origin xyz="0 0 0"/>
+        <inertia ixx="1.0" ixy="0.0" ixz="0.0"
+                 iyy="1.0" iyz="0.0"
+                 izz="1.0"/>
+      </inertial>
+      <visual>
+        <origin xyz=" 0 0 0 " rpy="0 0 0"/>
         <geometry>
           <mesh filename="package://turtlebot_arm_description/meshes/F2.stl" scale="${M_SCALE} ${M_SCALE} ${M_SCALE}"/>
@@ -209,5 +239,5 @@
       </visual>
       <collision>
-        <origin xyz="0.0 0.0 0.00775" rpy="0 0 0" />
+        <origin xyz="0.0 0.0 0.00775" rpy="0 0 0"/>
         <geometry>
           <box size="0.025 0.0485 0.0375"/>
@@ -215,23 +245,28 @@
       </collision>
     </link>
+    <gazebo reference="${name}_link">
+      <material>Gazebo/${color}</material>
+      <selfCollide>true</selfCollide>
+      <gravity>true</gravity>
+    </gazebo>
   </xacro:macro>
   <xacro:macro name="bioloid_F4_revolute" params="parent name color llimit ulimit vlimit *origin">
     <joint name="${name}_joint" type="revolute">
-      <insert_block name="origin" />
+      <insert_block name="origin"/>
       <axis xyz="0 1 0"/>
-      <limit effort="30" velocity="${vlimit}" lower="${llimit}" upper="${ulimit}" />
-      <parent link="${parent}"/>
-      <child link="${name}_link" />
-    </joint>
-    <link name="${name}_link">
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