Commit message: added two dynamixels and parts, looking good

File: turtlebot_arm_description/urdf/arm.xacro (robot description, xacro)
@@ -4,9 +4,16 @@
     <macro name="turtlebot_arm">
       <!--link name="base_link" /-->
-      <bioloid_F4_revolute parent="base_link" number="0" x_loc="0" y_loc="0" z_loc="0.5"/>
+      <dynamixel_AX12_fixed parent="base_link" number="0" x_loc="0" y_loc="0" z_loc="0.5" r="0" p="0" y="0"/>
+      <bioloid_F4_revolute parent="dynamixel_AX12_0_link" number="0" x_loc="0" y_loc="0" z_loc="0"/>
       <bioloid_F10_fixed parent="bioloid_F4_0_link" number="0" x_loc="0" y_loc="0" z_loc="${F4_HEIGHT+F10_HEIGHT/2}"/>
       <bioloid_F10_fixed parent="bioloid_F10_0_link" number="1" x_loc="0" y_loc="0" z_loc="${F10_HEIGHT}"/>
       <bioloid_F10_fixed parent="bioloid_F10_1_link" number="2" x_loc="0" y_loc="0" z_loc="${F10_HEIGHT}" />
       <bioloid_F3_fixed parent="bioloid_F10_2_link" number="0" x_loc="0" y_loc="0" z_loc="${F10_HEIGHT/2}" r="0" p="${M_PI}" y="0" />
+      <dynamixel_AX12_fixed parent="bioloid_F3_0_link" number="1" x_loc="0" y_loc="0" z_loc="${-AX12_HEIGHT-F10_HEIGHT}" r="0" p="${M_PI}" y="0"/>
+      <bioloid_F4_revolute parent="dynamixel_AX12_1_link" number="1" x_loc="0" y_loc="0" z_loc="0"/>
+      <bioloid_F10_fixed parent="bioloid_F4_1_link" number="3" x_loc="0" y_loc="0" z_loc="${F4_HEIGHT+F10_HEIGHT/2}"/>
+      <bioloid_F10_fixed parent="bioloid_F10_3_link" number="4" x_loc="0" y_loc="0" z_loc="${F10_HEIGHT}"/>
+      <bioloid_F10_fixed parent="bioloid_F10_4_link" number="5" x_loc="0" y_loc="0" z_loc="${F10_HEIGHT}" />
+      <bioloid_F3_fixed parent="bioloid_F10_5_link" number="1" x_loc="0" y_loc="0" z_loc="${F10_HEIGHT/2}" r="0" p="${M_PI}" y="0" />
   </macro>
 </robot>

File: turtlebot_arm_description/urdf/arm_hardware.xacro (robot description, xacro)
@@ -6,9 +6,10 @@
   <property name="F4_HEIGHT" value="0.0525"/>
   <property name="F3_HEIGHT" value="0.009"/>
+  <property name="AX12_HEIGHT" value="0.0385"/>
   <material name="green">
     <color rgba="0.22 0.32 0.14 1.0"/>
   </material>
-  <material name="blue">
-    <color rgba="0.0 0.0 0.8 1.0"/>
+  <material name="black">
+    <color rgba="0.0 0.0 0.0 1.0"/>
   </material>
  <macro name="bioloid_F10_fixed" params="parent number x_loc y_loc z_loc">
@@ -61,4 +62,33 @@
         </geometry>
         <material name="green"/>
+      </visual>
+      <collision>
+        <origin xyz="0.0 0.0 -0.0045" rpy="0 0 0" />
+        <geometry>
+          <box size="0.025 0.038 0.009"/>
+        </geometry>
+      </collision>
+    </link>
+  </macro>
+ <macro name="dynamixel_AX12_fixed" params="parent number x_loc y_loc z_loc r p y">
+    <joint name="dynamixel_AX12_${number}_joint" type="fixed">
+      <origin xyz="${x_loc} ${y_loc} ${z_loc}" rpy="${r} ${p} ${y}" />
+      <parent link="${parent}"/>
+      <child link="dynamixel_AX12_${number}_link" />
+    </joint>
+    <link name="dynamixel_AX12_${number}_link">
+      <inertial>
+        <mass value="0.00001" />
+        <origin xyz="0 0 0" />
+        <inertia ixx="1.0" ixy="0.0" ixz="0.0"
+          iyy="1.0" iyz="0.0"
+          izz="1.0" />
+      </inertial>
+      <visual>
+        <origin xyz=" 0 0 0 " rpy="0 0 0" />
+        <geometry>
+          <mesh filename="package://turtlebot_arm_description/meshes/ax12_box.stl" scale="${M_SCALE} ${M_SCALE} ${M_SCALE}"/>
+        </geometry>
+        <material name="black"/>
       </visual>
       <collision>

Commit message: adding more links

File: turtlebot_arm_description/urdf/arm.xacro (robot description, xacro)
@@ -3,17 +3,23 @@
   <include filename="$(find turtlebot_arm_description)/urdf/arm_hardware.xacro" />
     <macro name="turtlebot_arm">
-      <!--link name="base_link" /-->
-      <dynamixel_AX12_fixed parent="base_link" number="0" x_loc="0" y_loc="0" z_loc="0.5" r="0" p="0" y="0"/>
-      <bioloid_F4_revolute parent="dynamixel_AX12_0_link" number="0" x_loc="0" y_loc="0" z_loc="0"/>
+      <dynamixel_AX12_fixed parent="base_link" number="0" x_loc="0" y_loc="0" z_loc="0.5" r="${M_PI/2}" p="0" y="${M_PI/2}"/>
+      <bioloid_F3_revolute parent="dynamixel_AX12_0_link" number="0" joint_number="0" x_loc="0" y_loc="${AX12_WIDTH/2}" z_loc="0.0" r="${M_PI}" p="${M_PI/2}" y="${M_PI/2}" />
+      <dynamixel_AX12_fixed parent="bioloid_F3_0_link" number="1" x_loc="0" y_loc="0" z_loc="${-AX12_HEIGHT-F10_HEIGHT}" r="0" p="${M_PI}" y="0"/>
+      <bioloid_F4_revolute parent="dynamixel_AX12_1_link" number="0" joint_number="1" x_loc="0" y_loc="0" z_loc="0"/>
       <bioloid_F10_fixed parent="bioloid_F4_0_link" number="0" x_loc="0" y_loc="0" z_loc="${F4_HEIGHT+F10_HEIGHT/2}"/>
       <bioloid_F10_fixed parent="bioloid_F10_0_link" number="1" x_loc="0" y_loc="0" z_loc="${F10_HEIGHT}"/>
       <bioloid_F10_fixed parent="bioloid_F10_1_link" number="2" x_loc="0" y_loc="0" z_loc="${F10_HEIGHT}" />
-      <bioloid_F3_fixed parent="bioloid_F10_2_link" number="0" x_loc="0" y_loc="0" z_loc="${F10_HEIGHT/2}" r="0" p="${M_PI}" y="0" />
-      <dynamixel_AX12_fixed parent="bioloid_F3_0_link" number="1" x_loc="0" y_loc="0" z_loc="${-AX12_HEIGHT-F10_HEIGHT}" r="0" p="${M_PI}" y="0"/>
-      <bioloid_F4_revolute parent="dynamixel_AX12_1_link" number="1" x_loc="0" y_loc="0" z_loc="0"/>
+      <bioloid_F3_fixed parent="bioloid_F10_2_link" number="1" x_loc="0" y_loc="0" z_loc="${F10_HEIGHT/2}" r="0" p="${M_PI}" y="0" />
+      <dynamixel_AX12_fixed parent="bioloid_F3_1_link" number="2" x_loc="0" y_loc="0" z_loc="${-AX12_HEIGHT-F10_HEIGHT}" r="0" p="${M_PI}" y="0"/>
+      <bioloid_F4_revolute parent="dynamixel_AX12_2_link" number="1" joint_number="2" x_loc="0" y_loc="0" z_loc="0"/>
       <bioloid_F10_fixed parent="bioloid_F4_1_link" number="3" x_loc="0" y_loc="0" z_loc="${F4_HEIGHT+F10_HEIGHT/2}"/>
       <bioloid_F10_fixed parent="bioloid_F10_3_link" number="4" x_loc="0" y_loc="0" z_loc="${F10_HEIGHT}"/>
       <bioloid_F10_fixed parent="bioloid_F10_4_link" number="5" x_loc="0" y_loc="0" z_loc="${F10_HEIGHT}" />
-      <bioloid_F3_fixed parent="bioloid_F10_5_link" number="1" x_loc="0" y_loc="0" z_loc="${F10_HEIGHT/2}" r="0" p="${M_PI}" y="0" />
+      <bioloid_F3_fixed parent="bioloid_F10_5_link" number="2" x_loc="0" y_loc="0" z_loc="${F10_HEIGHT/2}" r="0" p="${M_PI}" y="0" />
+      <dynamixel_AX12_fixed parent="bioloid_F3_2_link" number="3" x_loc="0" y_loc="0" z_loc="${-AX12_HEIGHT-F10_HEIGHT}" r="0" p="${M_PI}" y="0"/>
+      <bioloid_F2_revolute parent="dynamixel_AX12_3_link" number="0" joint_number="3" x_loc="0" y_loc="0" z_loc="0"/>
+      <bioloid_F3_fixed parent="bioloid_F2_0_link" number="3" x_loc="0" y_loc="-0.008" z_loc="${F2_HEIGHT}" r="0" p="${M_PI}" y="${M_PI/2}" />
+      <dynamixel_AX12_fixed parent="bioloid_F3_3_link" number="4" x_loc="-0.02275" y_loc="0" z_loc="${-AX12_WIDTH/2}" r="${M_PI}" p="${M_PI/2}" y="0"/>
+      <bioloid_F2_revolute parent="dynamixel_AX12_4_link" number="1" joint_number="4" x_loc="0" y_loc="0" z_loc="0"/>
   </macro>
 </robot>

File: turtlebot_arm_description/urdf/arm_hardware.xacro (robot description, xacro)
@@ -7,4 +7,6 @@
   <property name="F3_HEIGHT" value="0.009"/>
   <property name="AX12_HEIGHT" value="0.0385"/>
+  <property name="AX12_WIDTH" value="0.038"/>
+  <property name="F2_HEIGHT" value="0.0265"/>
   <material name="green">
     <color rgba="0.22 0.32 0.14 1.0"/>
@@ -100,6 +102,37 @@
     </link>
   </macro>
- <macro name="bioloid_F2_revoute" params="parent number x_loc y_loc z_loc">
-    <joint name="bioloid_F2_${number}_joint" type="revolute">
+ <macro name="bioloid_F3_revolute" params="parent number joint_number x_loc y_loc z_loc r p y">
+    <joint name="joint_${joint_number}" type="revolute">
+      <origin xyz="${x_loc} ${y_loc} ${z_loc}" rpy="${r} ${p} ${y}" />
+      <parent link="${parent}"/>
+       <axis xyz="0 0 1"/>
+      <limit effort="30" velocity="1.0" lower="-1.57" upper="1.57" />
+      <child link="bioloid_F3_${number}_link" />
+    </joint>
+    <link name="bioloid_F3_${number}_link">
+      <inertial>
+        <mass value="0.00001" />
+        <origin xyz="0 0 0" />
+        <inertia ixx="1.0" ixy="0.0" ixz="0.0"
+          iyy="1.0" iyz="0.0"
+          izz="1.0" />
+      </inertial>
+      <visual>
+        <origin xyz=" 0 0 0 " rpy="0 0 0" />
+        <geometry>
+          <mesh filename="package://turtlebot_arm_description/meshes/F3.stl" scale="${M_SCALE} ${M_SCALE} ${M_SCALE}"/>
+        </geometry>
+        <material name="green"/>
+      </visual>
+      <collision>
+        <origin xyz="0.0 0.0 -0.0045" rpy="0 0 0" />
+        <geometry>
+          <box size="0.025 0.038 0.009"/>
+        </geometry>
+      </collision>
+    </link>
+  </macro>
+ <macro name="bioloid_F2_revolute" params="parent number joint_number x_loc y_loc z_loc">
+    <joint name="joint_${joint_number}" type="revolute">
       <origin xyz="${x_loc} ${y_loc} ${z_loc}" rpy="0 0 0" />
       <parent link="${parent}"/>
@@ -131,6 +164,6 @@
     </link>
   </macro>
- <macro name="bioloid_F4_revolute" params="parent number x_loc y_loc z_loc">
-    <joint name="bioloid_F4_${number}_joint" type="revolute">
+ <macro name="bioloid_F4_revolute" params="parent number joint_number x_loc y_loc z_loc">
+    <joint name="joint_${joint_number}" type="revolute">
       <origin xyz="${x_loc} ${y_loc} ${z_loc}" rpy="0 0 0" />
       <parent link="${parent}"/>

Commit message: full arm plus fingers

File: turtlebot_arm_description/urdf/arm.xacro (robot description, xacro)
@@ -3,7 +3,9 @@
   <include filename="$(find turtlebot_arm_description)/urdf/arm_hardware.xacro" />
     <macro name="turtlebot_arm">
-      <dynamixel_AX12_fixed parent="base_link" number="0" x_loc="0" y_loc="0" z_loc="0.5" r="${M_PI/2}" p="0" y="${M_PI/2}"/>
+      <!-- shoulder pan joint -->
+      <dynamixel_AX12_fixed parent="plate_3_link" number="0" x_loc="0.1143" y_loc="0" z_loc="${0.0508-AX12_WIDTH/2}" r="${M_PI/2}" p="0" y="${M_PI/2}"/>
       <bioloid_F3_revolute parent="dynamixel_AX12_0_link" number="0" joint_number="0" x_loc="0" y_loc="${AX12_WIDTH/2}" z_loc="0.0" r="${M_PI}" p="${M_PI/2}" y="${M_PI/2}" />
-      <dynamixel_AX12_fixed parent="bioloid_F3_0_link" number="1" x_loc="0" y_loc="0" z_loc="${-AX12_HEIGHT-F10_HEIGHT}" r="0" p="${M_PI}" y="0"/>
+      <dynamixel_AX12_fixed parent="bioloid_F3_0_link" number="1" x_loc="0" y_loc="0" z_loc="${-AX12_HEIGHT-F10_HEIGHT+0.001}" r="0" p="${M_PI}" y="0"/>
+      <!--shoulder lift joint -->
       <bioloid_F4_revolute parent="dynamixel_AX12_1_link" number="0" joint_number="1" x_loc="0" y_loc="0" z_loc="0"/>
       <bioloid_F10_fixed parent="bioloid_F4_0_link" number="0" x_loc="0" y_loc="0" z_loc="${F4_HEIGHT+F10_HEIGHT/2}"/>
@@ -11,5 +13,6 @@
       <bioloid_F10_fixed parent="bioloid_F10_1_link" number="2" x_loc="0" y_loc="0" z_loc="${F10_HEIGHT}" />
       <bioloid_F3_fixed parent="bioloid_F10_2_link" number="1" x_loc="0" y_loc="0" z_loc="${F10_HEIGHT/2}" r="0" p="${M_PI}" y="0" />
-      <dynamixel_AX12_fixed parent="bioloid_F3_1_link" number="2" x_loc="0" y_loc="0" z_loc="${-AX12_HEIGHT-F10_HEIGHT}" r="0" p="${M_PI}" y="0"/>
+      <!--elbow joint -->
+      <dynamixel_AX12_fixed parent="bioloid_F3_1_link" number="2" x_loc="0" y_loc="0" z_loc="${-AX12_HEIGHT-F10_HEIGHT+0.001}" r="0" p="${M_PI}" y="0"/>
       <bioloid_F4_revolute parent="dynamixel_AX12_2_link" number="1" joint_number="2" x_loc="0" y_loc="0" z_loc="0"/>
       <bioloid_F10_fixed parent="bioloid_F4_1_link" number="3" x_loc="0" y_loc="0" z_loc="${F4_HEIGHT+F10_HEIGHT/2}"/>
@@ -17,9 +20,16 @@
       <bioloid_F10_fixed parent="bioloid_F10_4_link" number="5" x_loc="0" y_loc="0" z_loc="${F10_HEIGHT}" />
       <bioloid_F3_fixed parent="bioloid_F10_5_link" number="2" x_loc="0" y_loc="0" z_loc="${F10_HEIGHT/2}" r="0" p="${M_PI}" y="0" />
-      <dynamixel_AX12_fixed parent="bioloid_F3_2_link" number="3" x_loc="0" y_loc="0" z_loc="${-AX12_HEIGHT-F10_HEIGHT}" r="0" p="${M_PI}" y="0"/>
-      <bioloid_F2_revolute parent="dynamixel_AX12_3_link" number="0" joint_number="3" x_loc="0" y_loc="0" z_loc="0"/>
+      <!--wrist joint-->
+      <dynamixel_AX12_fixed parent="bioloid_F3_2_link" number="3" x_loc="0" y_loc="0" z_loc="${-AX12_HEIGHT-F10_HEIGHT+0.001}" r="0" p="${M_PI}" y="0"/>
+      <bioloid_F2_revolute parent="dynamixel_AX12_3_link" number="0" joint_number="3" x_loc="0" y_loc="0" z_loc="0" ulimit="1.57" llimit="-1.57"/>
       <bioloid_F3_fixed parent="bioloid_F2_0_link" number="3" x_loc="0" y_loc="-0.008" z_loc="${F2_HEIGHT}" r="0" p="${M_PI}" y="${M_PI/2}" />
+      <!--gripper joint -->
       <dynamixel_AX12_fixed parent="bioloid_F3_3_link" number="4" x_loc="-0.02275" y_loc="0" z_loc="${-AX12_WIDTH/2}" r="${M_PI}" p="${M_PI/2}" y="0"/>
-      <bioloid_F2_revolute parent="dynamixel_AX12_4_link" number="1" joint_number="4" x_loc="0" y_loc="0" z_loc="0"/>
+      <!--finger 1-->
+      <bioloid_F2_revolute parent="dynamixel_AX12_4_link" number="1" joint_number="4" x_loc="0" y_loc="0" z_loc="0" ulimit="0.50" llimit="-0.60"/>
+      <finger_fixed parent="bioloid_F2_1_link" number="0" x_loc="0" y_loc="0" z_loc="${F2_HEIGHT}" r="0" p="0" y="0"/>
+      <!--finger 2-->
+      <bioloid_F3_fixed parent="dynamixel_AX12_4_link" number="4" x_loc="0" y_loc="0" z_loc="${-AX12_HEIGHT-F10_HEIGHT+0.001}" r="0" p="${M_PI}" y="0" />
+      <finger_fixed parent="bioloid_F3_4_link" number="1" x_loc="0" y_loc="0" z_loc="0" r="0" p="0" y="${M_PI}"/>
   </macro>
 </robot>

File: turtlebot_arm_description/urdf/arm_hardware.xacro (robot description, xacro)
@@ -15,4 +15,7 @@
     <color rgba="0.0 0.0 0.0 1.0"/>
   </material>
+  <material name="orange">
+    <color rgba="1.0 0.54 0.0 1.0"/>
+  </material>
  <macro name="bioloid_F10_fixed" params="parent number x_loc y_loc z_loc">
     <joint name="bioloid_F10_${number}_joint" type="fixed">
@@ -44,4 +47,33 @@
     </link>
   </macro>
+ <macro name="finger_fixed" params="parent number x_loc y_loc z_loc r p y">
+    <joint name="finger_${number}_joint" type="fixed">
+      <origin xyz="${x_loc} ${y_loc} ${z_loc}" rpy="${r} ${p} ${y}" />
+      <parent link="${parent}"/>
+      <child link="finger_${number}_link" />
+    </joint>
+    <link name="finger_${number}_link">
+      <inertial>
+        <mass value="0.00001" />
+        <origin xyz="0 0 0" />
+        <inertia ixx="1.0" ixy="0.0" ixz="0.0"
+          iyy="1.0" iyz="0.0"
+          izz="1.0" />
+      </inertial>
+      <visual>
+        <origin xyz=" 0 0 0 " rpy="0 0 0" />
+        <geometry>
+          <mesh filename="package://turtlebot_arm_description/meshes/finger.stl" scale="${M_SCALE} ${M_SCALE} ${M_SCALE}"/>
+        </geometry>
+        <material name="orange"/>
+      </visual>
+      <collision>
+        <origin xyz="0.02645 0.0 0.00655" rpy="0 0 0" />
+        <geometry>
+          <box size="0.0783 0.03801 0.0193"/>
+        </geometry>
+      </collision>
+    </link>
+  </macro>
  <macro name="bioloid_F3_fixed" params="parent number x_loc y_loc z_loc r p y">
     <joint name="bioloid_F3_${number}_joint" type="fixed">
@@ -133,10 +165,10 @@
     </link>
   </macro>
- <macro name="bioloid_F2_revolute" params="parent number joint_number x_loc y_loc z_loc">
+ <macro name="bioloid_F2_revolute" params="parent number joint_number x_loc y_loc z_loc ulimit llimit">
     <joint name="joint_${joint_number}" type="revolute">
       <origin xyz="${x_loc} ${y_loc} ${z_loc}" rpy="0 0 0" />
       <parent link="${parent}"/>
        <axis xyz="0 1 0"/>
-      <limit effort="30" velocity="1.0" lower="-1.57" upper="1.57" />
+      <limit effort="30" velocity="1.0" lower="${llimit}" upper="${ulimit}" />
       <child link="bioloid_F2_${number}_link" />
     </joint>

Commit message: changing angle limits

File: turtlebot_arm_description/urdf/arm.xacro (robot description, xacro)
@@ -22,5 +22,5 @@
       <!--wrist joint-->
       <dynamixel_AX12_fixed parent="bioloid_F3_2_link" number="3" x_loc="0" y_loc="0" z_loc="${-AX12_HEIGHT-F10_HEIGHT+0.001}" r="0" p="${M_PI}" y="0"/>
-      <bioloid_F2_revolute parent="dynamixel_AX12_3_link" number="0" joint_number="3" x_loc="0" y_loc="0" z_loc="0" ulimit="1.57" llimit="-1.57"/>
+      <bioloid_F2_revolute parent="dynamixel_AX12_3_link" number="0" joint_number="3" x_loc="0" y_loc="0" z_loc="0" ulimit="2.61" llimit="-2.61"/>
       <bioloid_F3_fixed parent="bioloid_F2_0_link" number="3" x_loc="0" y_loc="-0.008" z_loc="${F2_HEIGHT}" r="0" p="${M_PI}" y="${M_PI/2}" />
       <!--gripper joint -->

File: turtlebot_arm_description/urdf/arm_hardware.xacro (robot description, xacro)
@@ -1,5 +1,5 @@
 <?xml version="1.0"?>
 <robot>
-  <property name="M_PI" value="3.14159"/>
+x  <property name="M_PI" value="3.14159"/>
   <property name="M_SCALE" value="0.001"/>
   <property name="F10_HEIGHT" value="0.004"/>
@@ -139,5 +139,5 @@
       <parent link="${parent}"/>
        <axis xyz="0 0 1"/>
-      <limit effort="30" velocity="1.0" lower="-1.57" upper="1.57" />
+      <limit effort="30" velocity="1.0" lower="-2.61" upper="2.61" />
       <child link="bioloid_F3_${number}_link" />
     </joint>
@@ -201,5 +201,5 @@
       <parent link="${parent}"/>
        <axis xyz="0 1 0"/>
-      <limit effort="30" velocity="1.0" lower="-1.57" upper="1.57" />
+      <limit effort="30" velocity="1.0" lower="-2.61" upper="2.61" />
       <child link="bioloid_F4_${number}_link" />
     </joint>

Commit message: changing limits

File: turtlebot_arm_description/urdf/arm.xacro (robot description, xacro)
@@ -5,8 +5,8 @@
       <!-- shoulder pan joint -->
       <dynamixel_AX12_fixed parent="plate_3_link" number="0" x_loc="0.1143" y_loc="0" z_loc="${0.0508-AX12_WIDTH/2}" r="${M_PI/2}" p="0" y="${M_PI/2}"/>
-      <bioloid_F3_revolute parent="dynamixel_AX12_0_link" number="0" joint_number="0" x_loc="0" y_loc="${AX12_WIDTH/2}" z_loc="0.0" r="${M_PI}" p="${M_PI/2}" y="${M_PI/2}" />
+      <bioloid_F3_revolute parent="dynamixel_AX12_0_link" number="0" joint_name="shoulder_pan" x_loc="0" y_loc="${AX12_WIDTH/2}" z_loc="0.0" r="${M_PI}" p="${M_PI/2}" y="${M_PI/2}" />
       <dynamixel_AX12_fixed parent="bioloid_F3_0_link" number="1" x_loc="0" y_loc="0" z_loc="${-AX12_HEIGHT-F10_HEIGHT+0.001}" r="0" p="${M_PI}" y="0"/>
       <!--shoulder lift joint -->
-      <bioloid_F4_revolute parent="dynamixel_AX12_1_link" number="0" joint_number="1" x_loc="0" y_loc="0" z_loc="0"/>
+      <bioloid_F4_revolute parent="dynamixel_AX12_1_link" number="0" joint_name="shoulder_lift" x_loc="0" y_loc="0" z_loc="0"/>
       <bioloid_F10_fixed parent="bioloid_F4_0_link" number="0" x_loc="0" y_loc="0" z_loc="${F4_HEIGHT+F10_HEIGHT/2}"/>
       <bioloid_F10_fixed parent="bioloid_F10_0_link" number="1" x_loc="0" y_loc="0" z_loc="${F10_HEIGHT}"/>
@@ -15,5 +15,5 @@
       <!--elbow joint -->
       <dynamixel_AX12_fixed parent="bioloid_F3_1_link" number="2" x_loc="0" y_loc="0" z_loc="${-AX12_HEIGHT-F10_HEIGHT+0.001}" r="0" p="${M_PI}" y="0"/>
-      <bioloid_F4_revolute parent="dynamixel_AX12_2_link" number="1" joint_number="2" x_loc="0" y_loc="0" z_loc="0"/>
+      <bioloid_F4_revolute parent="dynamixel_AX12_2_link" number="1" joint_name="elbow_flex" x_loc="0" y_loc="0" z_loc="0"/>
       <bioloid_F10_fixed parent="bioloid_F4_1_link" number="3" x_loc="0" y_loc="0" z_loc="${F4_HEIGHT+F10_HEIGHT/2}"/>
       <bioloid_F10_fixed parent="bioloid_F10_3_link" number="4" x_loc="0" y_loc="0" z_loc="${F10_HEIGHT}"/>
@@ -22,10 +22,10 @@
       <!--wrist joint-->
       <dynamixel_AX12_fixed parent="bioloid_F3_2_link" number="3" x_loc="0" y_loc="0" z_loc="${-AX12_HEIGHT-F10_HEIGHT+0.001}" r="0" p="${M_PI}" y="0"/>
-      <bioloid_F2_revolute parent="dynamixel_AX12_3_link" number="0" joint_number="3" x_loc="0" y_loc="0" z_loc="0" ulimit="2.61" llimit="-2.61"/>
+      <bioloid_F2_revolute parent="dynamixel_AX12_3_link" number="0" joint_name="wrist_flex" x_loc="0" y_loc="0" z_loc="0" ulimit="2.0" llimit="-2.0"/>
       <bioloid_F3_fixed parent="bioloid_F2_0_link" number="3" x_loc="0" y_loc="-0.008" z_loc="${F2_HEIGHT}" r="0" p="${M_PI}" y="${M_PI/2}" />
       <!--gripper joint -->
       <dynamixel_AX12_fixed parent="bioloid_F3_3_link" number="4" x_loc="-0.02275" y_loc="0" z_loc="${-AX12_WIDTH/2}" r="${M_PI}" p="${M_PI/2}" y="0"/>
       <!--finger 1-->
-      <bioloid_F2_revolute parent="dynamixel_AX12_4_link" number="1" joint_number="4" x_loc="0" y_loc="0" z_loc="0" ulimit="0.50" llimit="-0.60"/>
+      <bioloid_F2_revolute parent="dynamixel_AX12_4_link" number="1" joint_name="gripper" x_loc="0" y_loc="0" z_loc="0" ulimit="0.50" llimit="-0.60"/>
       <finger_fixed parent="bioloid_F2_1_link" number="0" x_loc="0" y_loc="0" z_loc="${F2_HEIGHT}" r="0" p="0" y="0"/>
       <!--finger 2-->

File: turtlebot_arm_description/urdf/arm_hardware.xacro (robot description, xacro)
@@ -1,5 +1,5 @@
 <?xml version="1.0"?>
 <robot>
-x  <property name="M_PI" value="3.14159"/>
+  <property name="M_PI" value="3.14159"/>
   <property name="M_SCALE" value="0.001"/>
   <property name="F10_HEIGHT" value="0.004"/>
@@ -134,10 +134,10 @@
     </link>
   </macro>
- <macro name="bioloid_F3_revolute" params="parent number joint_number x_loc y_loc z_loc r p y">
-    <joint name="joint_${joint_number}" type="revolute">
+ <macro name="bioloid_F3_revolute" params="parent number joint_name x_loc y_loc z_loc r p y">
+    <joint name="${joint_name}_joint" type="revolute">
       <origin xyz="${x_loc} ${y_loc} ${z_loc}" rpy="${r} ${p} ${y}" />
       <parent link="${parent}"/>
        <axis xyz="0 0 1"/>
-      <limit effort="30" velocity="1.0" lower="-2.61" upper="2.61" />
+      <limit effort="30" velocity="1.0" lower="-2.0" upper="2.0" />
       <child link="bioloid_F3_${number}_link" />
     </joint>
@@ -165,6 +165,6 @@
     </link>
   </macro>
- <macro name="bioloid_F2_revolute" params="parent number joint_number x_loc y_loc z_loc ulimit llimit">
-    <joint name="joint_${joint_number}" type="revolute">
+ <macro name="bioloid_F2_revolute" params="parent number joint_name x_loc y_loc z_loc ulimit llimit">
+    <joint name="${joint_name}_joint" type="revolute">
       <origin xyz="${x_loc} ${y_loc} ${z_loc}" rpy="0 0 0" />
       <parent link="${parent}"/>
@@ -196,10 +196,10 @@
     </link>
   </macro>
- <macro name="bioloid_F4_revolute" params="parent number joint_number x_loc y_loc z_loc">
-    <joint name="joint_${joint_number}" type="revolute">
+ <macro name="bioloid_F4_revolute" params="parent number joint_name x_loc y_loc z_loc">
+    <joint name="${joint_name}_joint" type="revolute">
       <origin xyz="${x_loc} ${y_loc} ${z_loc}" rpy="0 0 0" />
       <parent link="${parent}"/>
        <axis xyz="0 1 0"/>
-      <limit effort="30" velocity="1.0" lower="-2.61" upper="2.61" />
+      <limit effort="30" velocity="1.0" lower="-2.0" upper="2.0" />
       <child link="bioloid_F4_${number}_link" />
     </joint>
