Commit message: Screwing up the URDF

File: turtlebot_arm_description/urdf/arm.xacro (robot description, xacro)
@@ -3,4 +3,11 @@
   <include filename="$(find turtlebot_arm_description)/urdf/arm_hardware.xacro" />
     <macro name="turtlebot_arm">
+      <!-- fake arm_base_link joint -->
+      <link name="arm_base_link" />
+      <joint name="arm_base_joint" type="fixed">
+        <origin xyz="0 0 0 " rpy="-${M_PI/2} 0 -${M_PI/2}" />
+        <parent link="dynamixel_AX12_0_link"/>
+        <child link="arm_base_link" />
+      </joint>
       <!-- shoulder pan joint -->
       <dynamixel_AX12_fixed parent="plate_3_link" number="0" x_loc="0.1143" y_loc="0" z_loc="${0.0508-AX12_WIDTH/2}" r="${M_PI/2}" p="0" y="${M_PI/2}"/>

Commit message: Pretty pretty arm base

File: turtlebot_arm_description/urdf/arm.xacro (robot description, xacro)
@@ -6,5 +6,5 @@
       <link name="arm_base_link" />
       <joint name="arm_base_joint" type="fixed">
-        <origin xyz="0 0 0 " rpy="-${M_PI/2} 0 -${M_PI/2}" />
+        <origin xyz="0 0 0 " rpy="-${M_PI/2} -${M_PI/2} 0" />
         <parent link="dynamixel_AX12_0_link"/>
         <child link="arm_base_link" />

Commit message: Now with more gripper_link

File: turtlebot_arm_description/urdf/arm.xacro (robot description, xacro)
@@ -9,4 +9,11 @@
         <parent link="dynamixel_AX12_0_link"/>
         <child link="arm_base_link" />
+      </joint>
+      <!-- fake gripper_link joint -->
+      <link name="gripper_ink" />
+      <joint name="gripper_link_joint" type="fixed">
+        <origin xyz="0 0 0 " rpy="0 0 0" />
+        <parent link="bioloid_F2_0_link"/>
+        <child link="gripper_link" />
       </joint>
       <!-- shoulder pan joint -->

Commit message: Late night URDF party (excitement)

File: turtlebot_arm_description/urdf/arm.xacro (robot description, xacro)
@@ -11,7 +11,7 @@
       </joint>
       <!-- fake gripper_link joint -->
-      <link name="gripper_ink" />
+      <link name="gripper_link" />
       <joint name="gripper_link_joint" type="fixed">
-        <origin xyz="0 0 0 " rpy="0 0 0" />
+        <origin xyz="0 0 .07" rpy="0 -${M_PI/2} 0" />
         <parent link="bioloid_F2_0_link"/>
         <child link="gripper_link" />

Commit message: Moved gripper_link up to line up with the gripper

File: turtlebot_arm_description/urdf/arm.xacro (robot description, xacro)
@@ -13,5 +13,5 @@
       <link name="gripper_link" />
       <joint name="gripper_link_joint" type="fixed">
-        <origin xyz="0 0 .07" rpy="0 -${M_PI/2} 0" />
+        <origin xyz="0 0 .112" rpy="0 -${M_PI/2} 0" />
         <parent link="bioloid_F2_0_link"/>
         <child link="gripper_link" />

Commit message: Set proper gripper_joint limits

File: turtlebot_arm_description/urdf/arm.xacro (robot description, xacro)
@@ -97,5 +97,5 @@
       <origin xyz="0 0 0" rpy="0 0 0"/>
       <axis xyz="0 1 0"/>
-      <limit effort="30" velocity="0.785" lower="-0.060" upper="0.50" />
+      <limit effort="30" velocity="0.785" lower="-0.40" upper="0.46" />
       <parent link="gripper_servo_link"/>
       <child link="gripper_active_link" />

Commit message: Provide meaningful values for links' moment of inertia. All excepf for the AX-12 servos are just epsilon values, as they are small plastic parts, very light. For the servos I used the formulas for solid cuboids explained here: http://en.wikipedia.org/wiki/List_of_moments_of_inertia

File: turtlebot_arm_description/urdf/arm.xacro (robot description, xacro)
@@ -24,5 +24,5 @@
     <link name="gripper_link"/>
     <joint name="gripper_link_joint" type="revolute">
-      <origin xyz="0 0 .112" rpy="0 -1.57 0"/>
+      <origin xyz="0 0 0.112" rpy="0 -1.57 0"/>
       <parent link="arm_wrist_flex_link"/>
       <child link="gripper_link"/>
@@ -103,9 +103,9 @@
     <link name="gripper_active_link">
       <inertial>
-        <mass value="0.00001"/>
+        <mass value="0.010"/>
         <origin xyz="0 0 0"/>
-        <inertia ixx="1.0" ixy="0.0" ixz="0.0"
-          iyy="1.0" iyz="0.0"
-          izz="1.0"/>
+        <inertia ixx="0.000001" ixy="0.0" ixz="0.0"
+                 iyy="0.000001" iyz="0.0"
+                 izz="0.000001"/>
       </inertial>
       <visual>

File: turtlebot_arm_description/urdf/arm_hardware.xacro (robot description, xacro)
@@ -19,7 +19,7 @@
         <mass value="0.018"/>
         <origin xyz="0 0 0"/>
-        <inertia ixx="1.0" ixy="0.0" ixz="0.0"
-                 iyy="1.0" iyz="0.0"
-                 izz="1.0"/>
+        <inertia ixx="0.000001" ixy="0.0" ixz="0.0"
+                 iyy="0.000001" iyz="0.0"
+                 izz="0.000001"/>
       </inertial>
       <visual>
@@ -53,7 +53,7 @@
         <mass value="0.015"/>
         <origin xyz="0 0 0"/>
-        <inertia ixx="1.0" ixy="0.0" ixz="0.0"
-                 iyy="1.0" iyz="0.0"
-                 izz="1.0"/>
+        <inertia ixx="0.000001" ixy="0.0" ixz="0.0"
+                 iyy="0.000001" iyz="0.0"
+                 izz="0.000001"/>
       </inertial>
       <visual>
@@ -87,7 +87,7 @@
         <mass value="0.055"/>
         <origin xyz="0 0 0"/>
-        <inertia ixx="1.0" ixy="0.0" ixz="0.0"
-                 iyy="1.0" iyz="0.0"
-                 izz="1.0"/>
+        <inertia ixx="0.000017012" ixy="0.0" ixz="0.0"
+                 iyy="0.000013258" iyz="0.0"
+                 izz="0.000009483"/>
       </inertial>
       <visual>
@@ -121,7 +121,7 @@
         <mass value="0.004"/>
         <origin xyz="0 0 0"/>
-        <inertia ixx="1.0" ixy="0.0" ixz="0.0"
-                 iyy="1.0" iyz="0.0"
-                 izz="1.0"/>
+        <inertia ixx="0.000001" ixy="0.0" ixz="0.0"
+                 iyy="0.000001" iyz="0.0"
+                 izz="0.000001"/>
       </inertial>
       <visual>
@@ -155,7 +155,7 @@
         <mass value="0.005"/>
         <origin xyz="0 0 0"/>
-        <inertia ixx="1.0" ixy="0.0" ixz="0.0"
-                 iyy="1.0" iyz="0.0"
-                 izz="1.0"/>
+        <inertia ixx="0.000001" ixy="0.0" ixz="0.0"
+                 iyy="0.000001" iyz="0.0"
+                 izz="0.000001"/>
       </inertial>
       <visual>
@@ -184,4 +184,5 @@
       <axis xyz="0 0 -1"/>
       <limit effort="30" velocity="${vlimit}" lower="${llimit}" upper="${ulimit}"/>
+      <dynamics friction="0.13"/>
       <parent link="${parent}"/>
       <child link="${name}_link"/>
@@ -191,7 +192,7 @@
         <mass value="0.008"/>
         <origin xyz="0 0 0"/>
-        <inertia ixx="1.0" ixy="0.0" ixz="0.0"
-                 iyy="1.0" iyz="0.0"
-                 izz="1.0"/>
+        <inertia ixx="0.000001" ixy="0.0" ixz="0.0"
+                 iyy="0.000001" iyz="0.0"
+                 izz="0.000001"/>
       </inertial>
       <visual>
@@ -220,4 +221,5 @@
       <axis xyz="0 1 0"/>
       <limit effort="30" velocity="${vlimit}" lower="${llimit}" upper="${ulimit}"/>
+      <dynamics friction="0.13"/>
       <parent link="${parent}"/>
       <child link="${name}_link"/>
@@ -227,7 +229,7 @@
         <mass value="0.010"/>
         <origin xyz="0 0 0"/>
-        <inertia ixx="1.0" ixy="0.0" ixz="0.0"
-                 iyy="1.0" iyz="0.0"
-                 izz="1.0"/>
+        <inertia ixx="0.000001" ixy="0.0" ixz="0.0"
+                 iyy="0.000001" iyz="0.0"
+                 izz="0.000001"/>
       </inertial>
       <visual>
@@ -256,4 +258,5 @@
       <axis xyz="0 1 0"/>
       <limit effort="30" velocity="${vlimit}" lower="${llimit}" upper="${ulimit}"/>
+      <dynamics friction="0.13"/>
       <parent link="${parent}"/>
       <child link="${name}_link"/>
@@ -263,7 +266,7 @@
         <mass value="0.016"/>
         <origin xyz="0 0 0"/>
-        <inertia ixx="1.0" ixy="0.0" ixz="0.0"
-                 iyy="1.0" iyz="0.0"
-                 izz="1.0"/>
+        <inertia ixx="0.000001" ixy="0.0" ixz="0.0"
+                 iyy="0.000001" iyz="0.0"
+                 izz="0.000001"/>
       </inertial>
       <visual>
