Commit message: Simplification of turtlebot arm config for multiple arms 	- removed need for separate pincher_arm.xacro file         - note: the combined file has new joint limits that <should> work for either         - some modifications to YAML files based on update to ArbotixROS

File: turtlebot_arm_description/urdf/pincher_arm.urdf (robot description, URDF)
Before this commit: robot turtlebot_arm, 24 links, 23 joints
Joints:
- joint arm_elbow_flex_joint: limit lower=-2.617 upper=2.617 effort=30 velocity=1.571 -> lower=-2.42 upper=2.38 effort=30 velocity=1.571
- joint arm_shoulder_lift_joint: limit lower=-2.617 upper=2.617 effort=30 velocity=1.571 -> lower=-2.21 upper=2.16 effort=30 velocity=1.571
- joint arm_shoulder_pan_joint: limit lower=-2.617 upper=2.617 effort=30 velocity=1.571 -> lower=-2.62 upper=2.62 effort=30 velocity=1.571
- joint arm_wrist_flex_joint: limit lower=-1.745 upper=1.745 effort=30 velocity=1.571 -> lower=-1.72 upper=1.68 effort=30 velocity=1.571

File: turtlebot_arm_description/urdf/pincher_arm.urdf.xacro (robot description, xacro)
@@ -2,5 +2,5 @@
 <robot name="turtlebot_arm" xmlns:xacro="http://ros.org/wiki/xacro">
     <!-- Included URDF Files -->
-    <xacro:include filename="$(find turtlebot_arm_description)/urdf/pincher_arm.xacro"/>
+    <xacro:include filename="$(find turtlebot_arm_description)/urdf/turtlebot_arm.xacro"/>
     <!-- As we don't have here a turtlebot, add a base_link link as its location reference -->
     <link name="base_link"/>
@@ -8,6 +8,5 @@
          for the first joint (arm_shoulder_pan) to allow accessing to different operational
          areas, e.g. left handed vs. right handed robot -->
-    <turtlebot_arm parent="base_link" color="Gray" gripper_color="Gray"
-                   joints_vlimit="1.571" pan_llimit="-2.617" pan_ulimit="2.617">
+    <turtlebot_arm parent="base_link" color="Gray" gripper_color="Gray" joints_vlimit="1.571" pan_llimit="-2.617" pan_ulimit="2.617" pincher_gripper="true">
       <!-- Place the "floating" arm at the location it should be if mounted on a turtlebot,
            as pick and place and other demos assume this location -->

File: turtlebot_arm_description/urdf/turtlebot_arm.urdf (robot description, URDF)
Before this commit: robot turtlebot_arm, 25 links, 24 joints
Joints:
- joint arm_elbow_flex_joint: limit lower=-2.617 upper=2.617 effort=30 velocity=1.571 -> lower=-2.42 upper=2.38 effort=30 velocity=1.571
- joint arm_shoulder_lift_joint: limit lower=-2.617 upper=2.617 effort=30 velocity=1.571 -> lower=-2.21 upper=2.16 effort=30 velocity=1.571
- joint arm_shoulder_pan_joint: limit lower=-2.617 upper=2.617 effort=30 velocity=1.571 -> lower=-2.62 upper=2.62 effort=30 velocity=1.571
- joint arm_wrist_flex_joint: limit lower=-1.745 upper=1.745 effort=30 velocity=1.571 -> lower=-1.72 upper=1.68 effort=30 velocity=1.571

File: turtlebot_arm_description/urdf/turtlebot_arm.urdf.xacro (robot description, xacro)
@@ -9,5 +9,5 @@
          areas, e.g. left handed vs. right handed robot -->
     <turtlebot_arm parent="base_link" color="White" gripper_color="Green"
-                   joints_vlimit="1.571" pan_llimit="-2.617" pan_ulimit="2.617">
+                   joints_vlimit="1.571" pan_llimit="-2.617" pan_ulimit="2.617" pincher_gripper="false">
       <!-- Place the "floating" arm at the location it should be if mounted on a turtlebot,
            as pick and place and other demos assume this location -->

File: turtlebot_arm_description/urdf/turtlebot_arm.xacro (robot description, xacro)
@@ -6,10 +6,13 @@
   </material>
   <material name="Black">
-    <color rgba="0.0 0.0 0.0 1.0"/>
+    <color rgba="0.08 0.08 0.08 1.0"/>
+  </material>
+  <material name="Gray">
+    <color rgba="0.2 0.2 0.21 1.0"/>
   </material>
   <material name="Green">
     <color rgba="0.22 0.32 0.14 1.0"/>
   </material>
-  <xacro:macro name="turtlebot_arm" params="parent color gripper_color *origin
+  <xacro:macro name="turtlebot_arm" params="parent color pincher_gripper gripper_color *origin
                                             joints_vlimit pan_llimit pan_ulimit">
     <link name="arm_base_link"/>
@@ -35,5 +38,5 @@
     </dynamixel_AX12_fixed>
     <bioloid_F3_revolute parent="arm_shoulder_pan_servo_link" name="arm_shoulder_pan" color="${color}"
-                         vlimit="${joints_vlimit}" llimit="${pan_llimit}" ulimit="${pan_ulimit}">
+                         vlimit="${joints_vlimit}" llimit="-2.62" ulimit="2.62">
       <origin xyz="0 ${AX12_WIDTH/2} 0" rpy="${-M_PI/2} ${M_PI/2} ${M_PI}"/>
     </bioloid_F3_revolute>
@@ -43,5 +46,5 @@
     </dynamixel_AX12_fixed>
     <bioloid_F4_revolute parent="arm_shoulder_lift_servo_link" name="arm_shoulder_lift" color="${color}"
-                         vlimit="${joints_vlimit}" llimit="-2.617" ulimit="2.617">
+                         vlimit="${joints_vlimit}" llimit="-2.21" ulimit="2.16">
       <origin xyz="0 0 0" rpy="0 0 0"/>
     </bioloid_F4_revolute>
@@ -63,5 +66,5 @@
     </dynamixel_AX12_fixed>
     <bioloid_F4_revolute parent="arm_elbow_flex_servo_link" name="arm_elbow_flex" color="${color}"
-                         vlimit="${joints_vlimit}" llimit="-2.617" ulimit="2.617">
+                         vlimit="${joints_vlimit}" llimit="-2.42" ulimit="2.38">
       <origin xyz="0 0 0" rpy="0 0 0"/>
     </bioloid_F4_revolute>
@@ -83,5 +86,5 @@
     </dynamixel_AX12_fixed>
     <bioloid_F2_revolute parent="arm_wrist_flex_servo_link" name="arm_wrist_flex" color="${color}"
-                         vlimit="${joints_vlimit}" llimit="-1.745" ulimit="1.745">
+                         vlimit="${joints_vlimit}" llimit="-1.72" ulimit="1.68">
       <origin xyz="0 0 0" rpy="0 0 0"/>
     </bioloid_F2_revolute>
@@ -90,5 +93,10 @@
     </bioloid_F3_fixed>
   <!-- Gripper -->
+  <xacro:if value="${pincher_gripper}">
+  <xacro:include filename="$(find turtlebot_arm_description)/urdf/pincher_gripper.xacro"/>
+  </xacro:if>
+  <xacro:unless value="${pincher_gripper}">
   <xacro:include filename="$(find turtlebot_arm_description)/urdf/turtlebot_gripper.xacro"/>
+  </xacro:unless>
   </xacro:macro>
 </robot>
