Commit message: support for multiple arm types

File: turtlebot_arm_description/urdf/pincher_arm.urdf.xacro (robot description, xacro)
@@ -19,5 +19,5 @@
     <link name="base_link"/>
     <!-- Turtlebot arm macro -->
-    <turtlebot_arm parent="base_link" color="Gray" gripper_color="Gray"   pincher_gripper="true">
+    <turtlebot_arm parent="base_link" color="Gray" gripper_color="Gray"   pincher_gripper="true" turtlebot_gripper="false">
       <!-- Place the "floating" arm at the location it should be if mounted on a turtlebot,
            as pick and place and other demos assume this location -->

File: turtlebot_arm_description/urdf/turtlebot_arm.urdf.xacro (robot description, xacro)
@@ -19,5 +19,5 @@
     <!-- Turtlebot arm macro -->
     <turtlebot_arm parent="base_link" color="White" gripper_color="Green"
-                   pincher_gripper="false">
+                    pincher_gripper="false" turtlebot_gripper="true">
       <!-- Place the "floating" arm at the location it should be if mounted on a turtlebot,
            as pick and place and other demos assume this location -->

File: turtlebot_arm_description/urdf/turtlebot_arm.xacro (robot description, xacro)
@@ -15,5 +15,5 @@
     <color rgba="0.22 0.32 0.14 1.0"/>
   </material>
-  <xacro:macro name="turtlebot_arm" params="parent color pincher_gripper gripper_color *origin">
+  <xacro:macro name="turtlebot_arm" params="parent color pincher_gripper turtlebot_gripper gripper_color *origin">
     <link name="arm_base_link"/>
     <joint name="arm_base_joint" type="fixed">
@@ -93,7 +93,7 @@
   <xacro:include filename="$(find turtlebot_arm_description)/urdf/pincher_gripper.xacro"/>
   </xacro:if>
-  <xacro:unless value="${pincher_gripper}">
+  <xacro:if value="${turtlebot_gripper}">
   <xacro:include filename="$(find turtlebot_arm_description)/urdf/turtlebot_gripper.xacro"/>
-  </xacro:unless>
+  </xacro:if>
   </xacro:macro>
 </robot>
