Commit message: Swapped arm colors to be consistent with newer arm.

File: turtlebot_arm_description/urdf/arm_hardware.xacro (robot description, xacro)
@@ -9,12 +9,12 @@
   <property name="AX12_WIDTH" value="0.038"/>
   <property name="F2_HEIGHT" value="0.0265"/>
-  <material name="green">
-    <color rgba="0.22 0.32 0.14 1.0"/>
+  <material name="white">
+    <color rgba="0.87 0.90 0.87 1.0"/>
   </material>
   <material name="black">
     <color rgba="0.0 0.0 0.0 1.0"/>
   </material>
-  <material name="orange">
-    <color rgba="1.0 0.54 0.0 1.0"/>
+  <material name="green">
+    <color rgba="0.22 0.32 0.14 1.0"/>
   </material>
  <macro name="bioloid_F10_fixed" params="parent number x_loc y_loc z_loc">
@@ -37,5 +37,5 @@
           <mesh filename="package://turtlebot_arm_description/meshes/F10.stl" scale="${M_SCALE} ${M_SCALE} ${M_SCALE}"/>
         </geometry>
-        <material name="green"/>
+        <material name="white"/>
       </visual>
       <collision>
@@ -66,5 +66,5 @@
           <mesh filename="package://turtlebot_arm_description/meshes/finger.stl" scale="${M_SCALE} ${M_SCALE} ${M_SCALE}"/>
         </geometry>
-        <material name="orange"/>
+        <material name="green"/>
       </visual>
       <collision>
@@ -95,5 +95,5 @@
           <mesh filename="package://turtlebot_arm_description/meshes/F3.stl" scale="${M_SCALE} ${M_SCALE} ${M_SCALE}"/>
         </geometry>
-        <material name="green"/>
+        <material name="white"/>
       </visual>
       <collision>
@@ -155,5 +155,5 @@
           <mesh filename="package://turtlebot_arm_description/meshes/F3.stl" scale="${M_SCALE} ${M_SCALE} ${M_SCALE}"/>
         </geometry>
-        <material name="green"/>
+        <material name="white"/>
       </visual>
       <collision>
@@ -186,5 +186,5 @@
           <mesh filename="package://turtlebot_arm_description/meshes/F2.stl" scale="${M_SCALE} ${M_SCALE} ${M_SCALE}"/>
         </geometry>
-        <material name="green"/>
+        <material name="white"/>
       </visual>
       <collision>
@@ -217,5 +217,5 @@
           <mesh filename="package://turtlebot_arm_description/meshes/F4.stl" scale="${M_SCALE} ${M_SCALE} ${M_SCALE}"/>
         </geometry>
-        <material name="green"/>
+        <material name="white"/>
       </visual>
       <collision>

Commit message: Fix orientation issues, Close #64

File: turtlebot_arm_description/urdf/arm_hardware.xacro (robot description, xacro)
@@ -129,5 +129,5 @@
       <origin xyz="${x_loc} ${y_loc} ${z_loc}" rpy="${r} ${p} ${y}" />
       <parent link="${parent}"/>
-       <axis xyz="0 0 1"/>
+       <axis xyz="0 0 -1"/>
       <limit effort="30" velocity="1.0" lower="-2.0" upper="2.0" />
       <child link="bioloid_F3_${number}_link" />

Commit message: Add arm mount macro and mesh (downloaded here: http://www.thingiverse.com/thing:11193/#files)

File: turtlebot_arm_description/urdf/arm_hardware.xacro (robot description, xacro)
@@ -38,4 +38,33 @@
     </link>
   </macro>
+  <macro name="arm_mount" params="parent name color *origin">
+    <joint name="${name}_joint" type="fixed">
+      <insert_block name="origin" />
+      <parent link="${parent}"/>
+      <child link="${name}_link" />
+    </joint>
+    <link name="${name}_link">
+      <inertial>
+        <mass value="0.00001" />
+        <origin xyz="0 0 0" />
+        <inertia ixx="1.0" ixy="0.0" ixz="0.0"
+          iyy="1.0" iyz="0.0"
+          izz="1.0" />
+      </inertial>
+      <visual>
+        <origin xyz="-0.028 -0.0493 0.014" rpy="0.0 0.0 -${M_PI/2}" />
+        <geometry>
+          <mesh filename="package://turtlebot_arm_description/meshes/mount.stl" scale="${M_SCALE} ${M_SCALE} ${M_SCALE}"/>
+        </geometry>
+        <material name="${color}"/>
+      </visual>
+      <collision>
+        <origin xyz="-0.01 0.0 0.0165" rpy="0.0 0.0 0.0" />
+        <geometry>
+          <box size="0.074 0.074 0.004"/>
+        </geometry>
+      </collision>
+    </link>
+  </macro>
   <macro name="finger_fixed" params="parent name color *origin">
     <joint name="${name}_joint" type="fixed">

Commit message: Added triangular gripper finger mesh to PhantomX gripper URDF

File: turtlebot_arm_description/urdf/arm_hardware.xacro (robot description, xacro)
@@ -96,5 +96,5 @@
           <mesh filename="package://turtlebot_arm_description/meshes/ax12_box.stl" scale="${M_SCALE} ${M_SCALE} ${M_SCALE}"/>
         </geometry>
-        <material name="black"/>
+        <material name="${color}"/>
       </visual>
       <collision>
@@ -290,3 +290,37 @@
     </gazebo>
   </xacro:macro>
+  <xacro:macro name="gripper_finger_base" params="parent name color *origin">
+    <joint name="${name}_joint" type="fixed">
+      <insert_block name="origin"/>
+      <parent link="${parent}"/>
+      <child link="${name}_link"/>
+    </joint>
+    <link name="${name}_link">
+      <inertial>
+        <mass value="0.00001"/>
+        <origin xyz="0 0 0"/>
+        <inertia ixx="1.0" ixy="0.0" ixz="0.0"
+          iyy="1.0" iyz="0.0"
+          izz="1.0"/>
+      </inertial>
+      <visual>
+        <origin xyz="0.016 0 -.015 " rpy="${M_PI} ${-M_PI/2} ${M_PI/2}"/>
+        <geometry>
+          <mesh filename="package://turtlebot_arm_description/meshes/finger_base_px.stl" scale=".01 .01 .01"/>
+        </geometry>
+        <material name="${color}"/>
+      </visual>
+      <collision>
+        <origin xyz="0.015 0 -0.0135" rpy="0 0 0"/>
+        <geometry>
+          <box size="0.002 0.040 0.075"/>
+        </geometry>
+      </collision>
+    </link >
+    <gazebo reference="${name}_link">
+      <material>Gazebo/${color}</material>
+      <selfCollide>true</selfCollide>
+      <gravity>true</gravity>
+    </gazebo>
+  </xacro:macro>
 </robot>

File: turtlebot_arm_description/urdf/pincher_arm.urdf (robot description, URDF)
Before this commit: robot turtlebot_arm, 23 links, 22 joints
Links:
- removed link gripper_static_link
- added link gripper_active2_link, mass 0.00001; collision box size=0.036 0.028 0.004; visual mesh filename=package://turtlebot_arm_description/meshes/finger_px.stl scale=.01 .01 .01
- added link gripper_finger_base_link, mass 0.00001; collision box size=0.002 0.040 0.075; visual mesh filename=package://turtlebot_arm_description/meshes/finger_base_px.s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 scale=.01 .01 .01
- link gripper_active_link: geometry collision box size=0.036 0.028 0.004; visual mesh filename=package://turtlebot_arm_description/meshes/finger_px.stl scale=.01 .01 .01
Joints:
- removed joint gripper_static_joint
- added joint gripper2_joint: type fixed, parent gripper_servo_link, child gripper_active2_link
- added joint gripper_finger_base_joint: type fixed, parent arm_wrist_F3_0_link, child gripper_finger_base_link, origin xyz=-0.025 0 -.05  rpy=3.14159 -1.570795 3.14159

File: turtlebot_arm_description/urdf/pincher_arm.urdf.xacro (robot description, xacro)
@@ -8,5 +8,5 @@
          for the first joint (arm_shoulder_pan) to allow accessing to different operational
          areas, e.g. left handed vs. right handed robot -->
-    <turtlebot_arm parent="base_link" color="White" gripper_color="White"
+    <turtlebot_arm parent="base_link" color="Gray" gripper_color="Gray"
                    joints_vlimit="1.571" pan_llimit="-2.617" pan_ulimit="2.617">
       <!-- Place the "floating" arm at the location it should be if mounted on a turtlebot,

File: turtlebot_arm_description/urdf/pincher_arm.xacro (robot description, xacro)
@@ -3,8 +3,11 @@
   <xacro:include filename="$(find turtlebot_arm_description)/urdf/arm_hardware.xacro"/>
   <material name="White">
-    <color rgba="0.87 0.90 0.87 1.0"/>
+    <color rgba="0.8 0.8 0.78 1.0"/>
   </material>
   <material name="Black">
-    <color rgba="0.0 0.0 0.0 1.0"/>
+    <color rgba="0.08 0.08 0.08 1.0"/>
+  </material>
+  <material name="Gray">
+    <color rgba="0.2 0.2 0.21 1.0"/>
   </material>
   <material name="Green">

File: turtlebot_arm_description/urdf/pincher_gripper.xacro (robot description, xacro)
@@ -1,9 +1,14 @@
 <?xml version="1.0"?>
 <robot xmlns:xacro="http://ros.org/wiki/xacro">
+    <!-- finger base -->
+     <gripper_finger_base parent="arm_wrist_F3_0_link" name="gripper_finger_base" color="${color}">
+      <origin xyz="-0.025 0 -.05 " rpy="${M_PI} ${-M_PI/2} ${M_PI}"/>
+    </gripper_finger_base>
+    <!-- finger 1 -->
+    <dynamixel_AX12_fixed parent="arm_wrist_F3_0_link" name="gripper_servo" >
+      <origin xyz="-0.02275 0 ${-AX12_WIDTH/2}" rpy="${M_PI} ${M_PI/2} 0"/>
+      <!--origin xyz="-0.02275 0 ${-AX12_WIDTH/2}" rpy="${-M_PI/2} ${M_PI/2} ${M_PI}"/-->
+    </dynamixel_AX12_fixed>
     <!-- gripper joint -->
-    <dynamixel_AX12_fixed parent="arm_wrist_F3_0_link" name="gripper_servo">
-      <origin xyz="-0.02275 0 ${-AX12_WIDTH/2}" rpy="${M_PI} ${M_PI/2} 0"/>
-    </dynamixel_AX12_fixed>
-    <!-- finger 1 -->
     <joint name="gripper_joint" type="prismatic">
       <origin xyz="0 0 0" rpy="0 0 0"/>
@@ -22,20 +27,58 @@
       </inertial>
       <visual>
-        <origin xyz="0.035 0 -0.03 " rpy="0 0 0"/>
+        <origin xyz="0.016 0 -.015 " rpy="${M_PI} ${-M_PI/2} ${M_PI/2}"/>
         <geometry>
-          <mesh filename="package://turtlebot_arm_description/meshes/F10.stl" scale="${M_SCALE} ${M_SCALE} ${M_SCALE}"/>
+          <mesh filename="package://turtlebot_arm_description/meshes/finger_px.stl" scale=".01 .01 .01"/>
         </geometry>
-        <material name="${color}"/>
+        <material name="${gripper_color}"/>
       </visual>
       <collision>
-        <origin xyz="0.035 0 -0.03" rpy="0 0 0"/>
+        <origin xyz="0.035 0 -0.0135" rpy="0 0 0"/>
         <geometry>
-          <box size="0.025 0.038 0.004"/>
+          <box size="0.036 0.028 0.004"/>
         </geometry>
       </collision>
     </link>
-    <!-- finger 2 -->
+    <!-- finger2 -->
+    <!-- gripper joint -->
+    <!--  Mimic Causes Missing Joint error in Moveit
+      <joint name="gripper_joint2" type="prismatic">
+      <origin xyz="0 0 0" rpy="0 0 0"/>
+      <axis xyz="0 0 1"/>
+      <limit effort="30" velocity="0.5" lower="0.002" upper="0.031"/>
+      <parent link="gripper_servo_link"/>
+      <child link="gripper_active2_link"/>
+      <mimic joint="gripper_joint" multiplier="-.5"  offset = "0"/>
+    </joint-->
+      <!-- gripper joint -->
+    <joint name="gripper2_joint" type="fixed">
+      <parent link="gripper_servo_link"/>
+      <child link="gripper_active2_link"/>
+    </joint>
+       <link name="gripper_active2_link">
+      <inertial>
+        <mass value="0.00001"/>
+        <origin xyz="0 0 0"/>
+        <inertia ixx="1.0" ixy="0.0" ixz="0.0"
+          iyy="1.0" iyz="0.0"
+          izz="1.0"/>
+      </inertial>
+      <visual>
+        <origin xyz="0.016 0 -.015 " rpy="${M_PI} ${M_PI/2} ${M_PI/2}"/>
+        <geometry>
+          <mesh filename="package://turtlebot_arm_description/meshes/finger_px.stl" scale=".01 .01 .01"/>
+        </geometry>
+        <material name="${gripper_color}"/>
+      </visual>
+      <collision>
+        <origin xyz="0.035 0 -0.018" rpy="0 0 0"/>
+        <geometry>
+          <box size="0.036 0.028 0.004"/>
+        </geometry>
+      </collision>
+    </link>
+    <!-- finger 2 >
     <bioloid_F10_fixed parent="gripper_servo_link" name="gripper_static" color="${gripper_color}">
-      <origin xyz="0.035 0 ${-AX12_HEIGHT-F10_HEIGHT+0.01}" rpy="0 ${M_PI} 0"/>
-    </bioloid_F10_fixed>
+      <origin xyz="0.035 0 ${-AX12_HEIGHT-F10_HEIGHT+0.01}" rpy="0 ${M_PI} ${M_PI/2}"/>
+    </bioloid_F10_fixed -->
 </robot>
