Commit message: Simplifying multiple arm support   -  Adding section in turtlebot_arm.urdf.xacro for joint limits   -  Renaming finger mesh files to be model specific

File: turtlebot_arm_description/urdf/arm_hardware.xacro (robot description, xacro)
@@ -1,3 +1,4 @@
 <?xml version="1.0"?>
+<!-- Basic URDF components for Turtlebot Arm and PhantomX Pincher Arm-->
 <robot xmlns:xacro="http://ros.org/wiki/xacro">
   <xacro:property name="M_PI" value="3.14159"/>
@@ -8,4 +9,5 @@
   <xacro:property name="AX12_HEIGHT" value="0.0385"/>
   <xacro:property name="AX12_WIDTH" value="0.038"/>
+  <xacro:property name="AX12_LENGTH" value="0.050"/>
   <xacro:property name="F2_HEIGHT" value="0.0265"/>
   <xacro:macro name="arm_mount" params="parent name color *origin">
@@ -60,5 +62,5 @@
         <origin xyz=" 0 0 0 " rpy="0 0 0"/>
         <geometry>
-          <mesh filename="package://turtlebot_arm_description/meshes/finger.stl" scale="${M_SCALE} ${M_SCALE} ${M_SCALE}"/>
+          <mesh filename="package://turtlebot_arm_description/meshes/turtlebot_finger.stl" scale="${M_SCALE} ${M_SCALE} ${M_SCALE}"/>
         </geometry>
         <material name="${color}"/>
@@ -96,5 +98,5 @@
           <mesh filename="package://turtlebot_arm_description/meshes/ax12_box.stl" scale="${M_SCALE} ${M_SCALE} ${M_SCALE}"/>
         </geometry>
-        <material name="${color}"/>
+        <material name="Black"/>
       </visual>
       <collision>
@@ -307,5 +309,5 @@
         <origin xyz="0.016 0 -.015 " rpy="${M_PI} ${-M_PI/2} ${M_PI/2}"/>
         <geometry>
-          <mesh filename="package://turtlebot_arm_description/meshes/finger_base_px.stl" scale=".01 .01 .01"/>
+          <mesh filename="package://turtlebot_arm_description/meshes/pincher_finger_base.stl" scale=".01 .01 .01"/>
         </geometry>
         <material name="${color}"/>
@@ -324,3 +326,32 @@
     </gazebo>
   </xacro:macro>
+    <xacro:macro name="pincher_gripper" params="name color *origin">
+      <link name="${name}_link">
+      <inertial>
+        <mass value="0.00001"/>
+        <origin xyz="0 0 0"/>
+        <inertia ixx="1.0" ixy="0.0" ixz="0.0"
+          iyy="1.0" iyz="0.0"
+          izz="1.0"/>
+      </inertial>
+      <visual>
+        <insert_block name="origin"/>
+        <geometry>
+          <mesh filename="package://turtlebot_arm_description/meshes/pincher_finger.stl" scale=".01 .01 .01"/>
+        </geometry>
+        <material name="${color}"/>
+      </visual>
+      <collision>
+        <insert_block name="origin"/>
+        <geometry>
+          <box size="0.036 0.028 0.004"/>
+        </geometry>
+      </collision>
+    </link>
+      <gazebo reference="${name}_link">
+      <material>Gazebo/${color}</material>
+      <selfCollide>true</selfCollide>
+      <gravity>true</gravity>
+    </gazebo>
+  </xacro:macro>
 </robot>

File: turtlebot_arm_description/urdf/pincher_arm.urdf (robot description, URDF)
Before this commit: robot turtlebot_arm, 24 links, 23 joints
Links:
- link gripper_active2_link: geometry collision box size=0.036 0.028 0.004; visual mesh filename=package://turtlebot_arm_description/meshes/pincher_finger.s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 scale=.01 .01 .01
- link gripper_active_link: geometry collision box size=0.036 0.028 0.004; visual mesh filename=package://turtlebot_arm_description/meshes/pincher_finger.s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 scale=.01 .01 .01
- link gripper_finger_base_link: geometry collision box size=0.002 0.040 0.075; visual mesh filename=package://turtlebot_arm_description/meshes/pincher_finger_b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 scale=.01 .01 .01
Joints:
- joint arm_elbow_flex_joint: limit lower=-2.42 upper=2.38 effort=30 velocity=1.571 -> lower=-2.617 upper=2.617 effort=30 velocity=1.571
- joint arm_shoulder_lift_joint: limit lower=-2.21 upper=2.16 effort=30 velocity=1.571 -> lower=-2.617 upper=2.617 effort=30 velocity=1.571
- joint arm_shoulder_pan_joint: limit lower=-2.62 upper=2.62 effort=30 velocity=1.571 -> lower=-2.617 upper=2.617 effort=30 velocity=1.571
- joint arm_wrist_F3_0_joint: origin xyz=0 0.016 0.0265 rpy=0 3.14159 -1.570795 -> xyz=0 0 0.0265 rpy=0 3.14159 -3.14159
- joint arm_wrist_flex_joint: limit lower=-1.72 upper=1.68 effort=30 velocity=1.571 -> lower=-1.745 upper=1.745 effort=30 velocity=1.571
- joint gripper_finger_base_joint: origin xyz=-0.025 0 -.05  rpy=3.14159 -1.570795 3.14159 -> xyz=0.01  0.038 0 rpy=1.570795 -3.14159 1.570795; parent arm_wrist_F3_0_link -> gripper_servo_link
- joint gripper_joint: axis 0 0 1 -> 1 0 0
- joint gripper_servo_joint: origin xyz=-0.02275 0 -0.019 rpy=3.14159 1.570795 0 -> xyz=0 0 -0.019 rpy=1.570795 3.14159 1.570795

File: turtlebot_arm_description/urdf/pincher_arm.urdf.xacro (robot description, xacro)
@@ -1,12 +1,23 @@
 <?xml version="1.0"?>
+<!-- Describe URDF for PhantomX Pincher Arm -->
 <robot name="turtlebot_arm" xmlns:xacro="http://ros.org/wiki/xacro">
+    <!-- We can configure joints velocity limit and lower/upper limits
+          to allow access to different operational areas, e.g. left handed vs. right handed robot -->
+    <xacro:property name="joints_vlimit" value="1.571"/>
+    <xacro:property name="pan_llimit" value="-2.617"/>
+    <xacro:property name="pan_ulimit" value="2.617"/>
+    <xacro:property name="shoulder_llimit" value="-2.2"/>
+    <xacro:property name="shoulder_ulimit" value="2.16"/>
+    <xacro:property name="elbow_llimit" value="-2.42"/>
+    <xacro:property name="elbow_ulimit" value="2.38"/>
+    <xacro:property name="wrist_llimit" value="-1.72"/>
+    <xacro:property name="wrist_ulimit" value="1.68"/>
     <!-- Included URDF Files -->
+     <!-- Pincher arm is same as Turtlebot -->
     <xacro:include filename="$(find turtlebot_arm_description)/urdf/turtlebot_arm.xacro"/>
-    <!-- As we don't have here a turtlebot, add a base_link link as its location reference -->
+    <!-- As we don't have here a turtlebot base, add a base_link link as its location reference -->
     <link name="base_link"/>
-    <!-- Turtlebot arm macro: we can configure joints velocity limit and lower/upper limits
-         for the first joint (arm_shoulder_pan) to allow accessing to different operational
-         areas, e.g. left handed vs. right handed robot -->
-    <turtlebot_arm parent="base_link" color="Gray" gripper_color="Gray" joints_vlimit="1.571" pan_llimit="-2.617" pan_ulimit="2.617" pincher_gripper="true">
+    <!-- Turtlebot arm macro -->
+    <turtlebot_arm parent="base_link" color="Gray" gripper_color="Gray"   pincher_gripper="true">
       <!-- Place the "floating" arm at the location it should be if mounted on a turtlebot,
            as pick and place and other demos assume this location -->

File: turtlebot_arm_description/urdf/pincher_gripper.xacro (robot description, xacro)
@@ -1,47 +1,39 @@
 <?xml version="1.0"?>
+<!-- PhantomX Pincher Arm gripper URDF-->
 <robot xmlns:xacro="http://ros.org/wiki/xacro">
-    <!-- finger base -->
-     <gripper_finger_base parent="arm_wrist_F3_0_link" name="gripper_finger_base" color="${color}">
-      <origin xyz="-0.025 0 -.05 " rpy="${M_PI} ${-M_PI/2} ${M_PI}"/>
+    <bioloid_F3_fixed parent="arm_wrist_flex_link" name="arm_wrist_F3_0" color="${color}">
+      <origin xyz="0 0 ${F2_HEIGHT}" rpy="0 ${M_PI} ${-M_PI}"/>
+    </bioloid_F3_fixed>
+    <!-- gripper joint -->
+    <dynamixel_AX12_fixed parent="arm_wrist_F3_0_link" name="gripper_servo" >
+      <origin xyz="0 0 ${-AX12_WIDTH/2}" rpy="${M_PI/2} ${M_PI} ${M_PI/2}"/>
+    </dynamixel_AX12_fixed>
+     <gripper_finger_base parent="gripper_servo_link" name="gripper_finger_base" color="${color}">
+      <origin xyz="0.01  ${AX12_WIDTH} 0" rpy="${M_PI/2} ${-M_PI} ${M_PI/2}"/>
     </gripper_finger_base>
-    <!-- finger 1 -->
-    <dynamixel_AX12_fixed parent="arm_wrist_F3_0_link" name="gripper_servo" >
-      <origin xyz="-0.02275 0 ${-AX12_WIDTH/2}" rpy="${M_PI} ${M_PI/2} 0"/>
-      <!--origin xyz="-0.02275 0 ${-AX12_WIDTH/2}" rpy="${-M_PI/2} ${M_PI/2} ${M_PI}"/-->
-    </dynamixel_AX12_fixed>
-    <!-- gripper joint -->
+     <!-- Finger 1 -->
     <joint name="gripper_joint" type="prismatic">
       <origin xyz="0 0 0" rpy="0 0 0"/>
-      <axis xyz="0 0 1"/>
+      <axis xyz="1 0 0"/>
       <limit effort="30" velocity="0.5" lower="0.002" upper="0.031"/>
       <parent link="gripper_servo_link"/>
       <child link="gripper_active_link"/>
     </joint>
-    <link name="gripper_active_link">
-      <inertial>
-        <mass value="0.00001"/>
-        <origin xyz="0 0 0"/>
-        <inertia ixx="1.0" ixy="0.0" ixz="0.0"
-          iyy="1.0" iyz="0.0"
-          izz="1.0"/>
-      </inertial>
-      <visual>
-        <origin xyz="0.016 0 -.015 " rpy="${M_PI} ${-M_PI/2} ${M_PI/2}"/>
-        <geometry>
-          <mesh filename="package://turtlebot_arm_description/meshes/finger_px.stl" scale=".01 .01 .01"/>
-        </geometry>
-        <material name="${gripper_color}"/>
-      </visual>
-      <collision>
-        <origin xyz="0.035 0 -0.0135" rpy="0 0 0"/>
-        <geometry>
-          <box size="0.036 0.028 0.004"/>
-        </geometry>
-      </collision>
-    </link>
-    <!-- finger2 -->
-    <!-- gripper joint -->
-    <!--  Mimic Causes Missing Joint error in Moveit
-      <joint name="gripper_joint2" type="prismatic">
+    <pincher_gripper name="gripper_active" color="${color}" >
+      <origin xyz="-0.02 0.023 0" rpy="${-M_PI/2} 0 0"/>
+    </pincher_gripper>
+    <!-- Finger 2 -->
+    <!-- Note: currently static but should be a Mimic of Finger 1 -->
+    <joint name="gripper2_joint" type="fixed">
+      <parent link="gripper_servo_link"/>
+      <child link="gripper_active2_link"/>
+    </joint>
+    <pincher_gripper name="gripper_active2" color="${color}" >
+      <origin xyz="-0.02 0.023 0" rpy="${-M_PI/2} ${M_PI} 0"/>
+    </pincher_gripper>
+    <!-- Using Mimic -->
+    <!-- gripper 2 joint -->
+    <!--  ### Mimic would be better but causes Missing Joint error in Moveit
+      <joint name="gripper2_joint" type="prismatic">
       <origin xyz="0 0 0" rpy="0 0 0"/>
       <axis xyz="0 0 1"/>
@@ -51,34 +43,3 @@
       <mimic joint="gripper_joint" multiplier="-.5"  offset = "0"/>
     </joint-->
-      <!-- gripper joint -->
-    <joint name="gripper2_joint" type="fixed">
-      <parent link="gripper_servo_link"/>
-      <child link="gripper_active2_link"/>
-    </joint>
-       <link name="gripper_active2_link">
-      <inertial>
-        <mass value="0.00001"/>
-        <origin xyz="0 0 0"/>
-        <inertia ixx="1.0" ixy="0.0" ixz="0.0"
-          iyy="1.0" iyz="0.0"
-          izz="1.0"/>
-      </inertial>
-      <visual>
-        <origin xyz="0.016 0 -.015 " rpy="${M_PI} ${M_PI/2} ${M_PI/2}"/>
-        <geometry>
-          <mesh filename="package://turtlebot_arm_description/meshes/finger_px.stl" scale=".01 .01 .01"/>
-        </geometry>
-        <material name="${gripper_color}"/>
-      </visual>
-      <collision>
-        <origin xyz="0.035 0 -0.018" rpy="0 0 0"/>
-        <geometry>
-          <box size="0.036 0.028 0.004"/>
-        </geometry>
-      </collision>
-    </link>
-    <!-- finger 2 >
-    <bioloid_F10_fixed parent="gripper_servo_link" name="gripper_static" color="${gripper_color}">
-      <origin xyz="0.035 0 ${-AX12_HEIGHT-F10_HEIGHT+0.01}" rpy="0 ${M_PI} ${M_PI/2}"/>
-    </bioloid_F10_fixed -->
 </robot>

File: turtlebot_arm_description/urdf/turtlebot_arm.urdf (robot description, URDF)
Before this commit: robot turtlebot_arm, 25 links, 24 joints
Links:
- link gripper_active_finger_link: geometry collision box size=0.0783 0.03801 0.0193; visual mesh filename=package://turtlebot_arm_description/meshes/turtlebot_finger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 scale=0.001 0.001 0.001
- link gripper_static_finger_link: geometry collision box size=0.0783 0.03801 0.0193; visual mesh filename=package://turtlebot_arm_description/meshes/turtlebot_finger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 scale=0.001 0.001 0.001
Joints:
- joint arm_elbow_flex_joint: limit lower=-2.42 upper=2.38 effort=30 velocity=1.571 -> lower=-2.617 upper=2.617 effort=30 velocity=1.571
- joint arm_shoulder_lift_joint: limit lower=-2.21 upper=2.16 effort=30 velocity=1.571 -> lower=-2.617 upper=2.617 effort=30 velocity=1.571
- joint arm_shoulder_pan_joint: limit lower=-2.62 upper=2.62 effort=30 velocity=1.571 -> lower=-2.617 upper=2.617 effort=30 velocity=1.571
- joint arm_wrist_flex_joint: limit lower=-1.72 upper=1.68 effort=30 velocity=1.571 -> lower=-1.745 upper=1.745 effort=30 velocity=1.571

File: turtlebot_arm_description/urdf/turtlebot_arm.urdf.xacro (robot description, xacro)
@@ -1,13 +1,23 @@
 <?xml version="1.0"?>
+<!-- Describe URDF for Turtlebot Arm -->
 <robot name="turtlebot_arm" xmlns:xacro="http://ros.org/wiki/xacro">
+    <!-- We can configure joints velocity limit and lower/upper limits
+          to allow access to different operational areas, e.g. left handed vs. right handed robot -->
+    <xacro:property name="joints_vlimit" value="1.571"/>
+    <xacro:property name="pan_llimit" value="-2.617"/>
+    <xacro:property name="pan_ulimit" value="2.617"/>
+    <xacro:property name="shoulder_llimit" value="-2.617"/>
+    <xacro:property name="shoulder_ulimit" value="2.617"/>
+    <xacro:property name="elbow_llimit" value="-2.617"/>
+    <xacro:property name="elbow_ulimit" value="2.617"/>
+    <xacro:property name="wrist_llimit" value="-2.617"/>
+    <xacro:property name="wrist_ulimit" value="2.617"/>
     <!-- Included URDF Files -->
     <xacro:include filename="$(find turtlebot_arm_description)/urdf/turtlebot_arm.xacro"/>
-    <!-- As we don't have here a turtlebot, add a base_link link as its location reference -->
+    <!-- As we don't have here a turtlebot base, add a base_link link as its location reference -->
     <link name="base_link"/>
-    <!-- Turtlebot arm macro: we can configure joints velocity limit and lower/upper limits
-         for the first joint (arm_shoulder_pan) to allow accessing to different operational
-         areas, e.g. left handed vs. right handed robot -->
+    <!-- Turtlebot arm macro -->
     <turtlebot_arm parent="base_link" color="White" gripper_color="Green"
-                   joints_vlimit="1.571" pan_llimit="-2.617" pan_ulimit="2.617" pincher_gripper="false">
+                   pincher_gripper="false">
       <!-- Place the "floating" arm at the location it should be if mounted on a turtlebot,
            as pick and place and other demos assume this location -->

File: turtlebot_arm_description/urdf/turtlebot_arm.xacro (robot description, xacro)
@@ -1,3 +1,4 @@
 <?xml version="1.0"?>
+<!-- Arm description for Turtlebot Arm and PhantomX Pincher arm -->
 <robot xmlns:xacro="http://ros.org/wiki/xacro">
   <xacro:include filename="$(find turtlebot_arm_description)/urdf/arm_hardware.xacro"/>
@@ -14,6 +15,5 @@
     <color rgba="0.22 0.32 0.14 1.0"/>
   </material>
-  <xacro:macro name="turtlebot_arm" params="parent color pincher_gripper gripper_color *origin
-                                            joints_vlimit pan_llimit pan_ulimit">
+  <xacro:macro name="turtlebot_arm" params="parent color pincher_gripper gripper_color *origin">
     <link name="arm_base_link"/>
     <joint name="arm_base_joint" type="fixed">
@@ -38,5 +38,5 @@
     </dynamixel_AX12_fixed>
     <bioloid_F3_revolute parent="arm_shoulder_pan_servo_link" name="arm_shoulder_pan" color="${color}"
-                         vlimit="${joints_vlimit}" llimit="-2.62" ulimit="2.62">
+                         vlimit="${joints_vlimit}" llimit="${pan_llimit}" ulimit="${pan_ulimit}">
       <origin xyz="0 ${AX12_WIDTH/2} 0" rpy="${-M_PI/2} ${M_PI/2} ${M_PI}"/>
     </bioloid_F3_revolute>
@@ -46,5 +46,5 @@
     </dynamixel_AX12_fixed>
     <bioloid_F4_revolute parent="arm_shoulder_lift_servo_link" name="arm_shoulder_lift" color="${color}"
-                         vlimit="${joints_vlimit}" llimit="-2.21" ulimit="2.16">
+                         vlimit="${joints_vlimit}" llimit="${shoulder_llimit}" ulimit="${shoulder_ulimit}">
       <origin xyz="0 0 0" rpy="0 0 0"/>
     </bioloid_F4_revolute>
@@ -66,5 +66,5 @@
     </dynamixel_AX12_fixed>
     <bioloid_F4_revolute parent="arm_elbow_flex_servo_link" name="arm_elbow_flex" color="${color}"
-                         vlimit="${joints_vlimit}" llimit="-2.42" ulimit="2.38">
+                         vlimit="${joints_vlimit}" llimit="${elbow_llimit}" ulimit="${elbow_ulimit}">
       <origin xyz="0 0 0" rpy="0 0 0"/>
     </bioloid_F4_revolute>
@@ -86,11 +86,8 @@
     </dynamixel_AX12_fixed>
     <bioloid_F2_revolute parent="arm_wrist_flex_servo_link" name="arm_wrist_flex" color="${color}"
-                         vlimit="${joints_vlimit}" llimit="-1.72" ulimit="1.68">
+                         vlimit="${joints_vlimit}" llimit="${wrist_llimit}" ulimit="${wrist_ulimit}">
       <origin xyz="0 0 0" rpy="0 0 0"/>
     </bioloid_F2_revolute>
-    <bioloid_F3_fixed parent="arm_wrist_flex_link" name="arm_wrist_F3_0" color="${color}">
-      <origin xyz="0 0.016 ${F2_HEIGHT}" rpy="0 ${M_PI} ${-M_PI/2}"/>
-    </bioloid_F3_fixed>
-  <!-- Gripper -->
+  <!-- gripper - Load either Turtlebot gripper or Pincher Gripper -->
   <xacro:if value="${pincher_gripper}">
   <xacro:include filename="$(find turtlebot_arm_description)/urdf/pincher_gripper.xacro"/>

File: turtlebot_arm_description/urdf/turtlebot_gripper.xacro (robot description, xacro)
@@ -1,4 +1,8 @@
 <?xml version="1.0"?>
+<!-- Turtlebot Arm gripper URDF-->
 <robot xmlns:xacro="http://ros.org/wiki/xacro">
+    <bioloid_F3_fixed parent="arm_wrist_flex_link" name="arm_wrist_F3_0" color="${color}">
+      <origin xyz="0 0.016 ${F2_HEIGHT}" rpy="0 ${M_PI} ${-M_PI/2}"/>
+    </bioloid_F3_fixed>
     <!-- gripper joint -->
     <dynamixel_AX12_fixed parent="arm_wrist_F3_0_link" name="gripper_servo">
