Commit message: Corrected inertial tensor estimates in udrf
Many of the inertial values in turtlebot_arm_description were incorrect.
Added a macro to produce more true to reality inertial values and
regenerated urdfs.

File: turtlebot_arm_description/urdf/arm_hardware.xacro (robot description, xacro)
@@ -11,4 +11,15 @@
   <xacro:property name="AX12_LENGTH" value="0.050"/>
   <xacro:property name="F2_HEIGHT" value="0.0265"/>
+  <!-- Calculates the inertial properties of a bounding box. From
+       https://en.wikipedia.org/wiki/List_of_moments_of_inertia#List_of_3D_inertia_tensors-->
+  <xacro:macro name="box_inertia" params="length width height mass">
+    <inertial>
+      <mass value="${mass}"/>
+      <origin xyz="0 0 0"/>
+      <inertia ixx="${mass/12*(height**2+length**2)}" ixy="0" ixz = "0"
+               iyy="${mass/12*(width**2+length**2)}" iyz="0"
+               izz="${mass/12*(width**2+height**2)}"/>
+    </inertial>
+  </xacro:macro>
   <xacro:macro name="arm_mount" params="parent name color *origin">
     <joint name="${name}_joint" type="fixed">
@@ -18,11 +29,5 @@
     </joint>
     <link name="${name}_link">
-      <inertial>
-        <mass value="0.018"/>
-        <origin xyz="0 0 0"/>
-        <inertia ixx="0.000001" ixy="0.0" ixz="0.0"
-                 iyy="0.000001" iyz="0.0"
-                 izz="0.000001"/>
-      </inertial>
+      <xacro:box_inertia length="0.074" width="0.074" height="0.004" mass="0.018"/>
       <visual>
         <origin xyz="-0.028 -0.0493 0.014" rpy="0.0 0.0 -${M_PI/2}"/>
@@ -52,11 +57,5 @@
     </joint>
     <link name="${name}_link">
-      <inertial>
-        <mass value="0.015"/>
-        <origin xyz="0 0 0"/>
-        <inertia ixx="0.000001" ixy="0.0" ixz="0.0"
-                 iyy="0.000001" iyz="0.0"
-                 izz="0.000001"/>
-      </inertial>
+      <xacro:box_inertia length="0.0783" width="0.03801" height="0.0193" mass="0.015"/>
       <visual>
         <origin xyz=" 0 0 0 " rpy="0 0 0"/>
@@ -120,11 +119,5 @@
     </joint>
     <link name="${name}_link">
-      <inertial>
-        <mass value="0.004"/>
-        <origin xyz="0 0 0"/>
-        <inertia ixx="0.000001" ixy="0.0" ixz="0.0"
-                 iyy="0.000001" iyz="0.0"
-                 izz="0.000001"/>
-      </inertial>
+      <xacro:box_inertia length="0.025" width="0.038" height="0.004" mass="0.004"/>
       <visual>
         <origin xyz=" 0 0 0 " rpy="0 0 0"/>
@@ -154,11 +147,5 @@
     </joint>
     <link name="${name}_link">
-      <inertial>
-        <mass value="0.005"/>
-        <origin xyz="0 0 0"/>
-        <inertia ixx="0.000001" ixy="0.0" ixz="0.0"
-                 iyy="0.000001" iyz="0.0"
-                 izz="0.000001"/>
-      </inertial>
+      <xacro:box_inertia length="0.025" width="0.038" height="0.009" mass="0.005"/>
       <visual>
         <origin xyz=" 0 0 0 " rpy="0 0 0"/>
@@ -191,11 +178,5 @@
     </joint>
     <link name="${name}_link">
-      <inertial>
-        <mass value="0.008"/>
-        <origin xyz="0 0 0"/>
-        <inertia ixx="0.000001" ixy="0.0" ixz="0.0"
-                 iyy="0.000001" iyz="0.0"
-                 izz="0.000001"/>
-      </inertial>
+      <xacro:box_inertia length="0.025" width="0.038" height="0.009" mass="0.008"/>
       <visual>
         <origin xyz=" 0 0 0 " rpy="0 0 0"/>
@@ -228,11 +209,5 @@
     </joint>
     <link name="${name}_link">
-      <inertial>
-        <mass value="0.010"/>
-        <origin xyz="0 0 0"/>
-        <inertia ixx="0.000001" ixy="0.0" ixz="0.0"
-                 iyy="0.000001" iyz="0.0"
-                 izz="0.000001"/>
-      </inertial>
+      <xacro:box_inertia length="0.025" width="0.0485" height="0.0375" mass="0.010"/>
       <visual>
         <origin xyz=" 0 0 0 " rpy="0 0 0"/>
@@ -265,11 +240,5 @@
     </joint>
     <link name="${name}_link">
-      <inertial>
-        <mass value="0.016"/>
-        <origin xyz="0 0 0"/>
-        <inertia ixx="0.000001" ixy="0.0" ixz="0.0"
-                 iyy="0.000001" iyz="0.0"
-                 izz="0.000001"/>
-      </inertial>
+      <xacro:box_inertia length="0.028" width="0.0485" height="0.065" mass="0.016"/>
       <visual>
         <origin xyz=" 0 0 0 " rpy="0 0 0"/>
@@ -299,11 +268,5 @@
     </joint>
     <link name="${name}_link">
-      <inertial>
-        <mass value="0.00001"/>
-        <origin xyz="0 0 0"/>
-        <inertia ixx="1.0" ixy="0.0" ixz="0.0"
-          iyy="1.0" iyz="0.0"
-          izz="1.0"/>
-      </inertial>
+      <xacro:box_inertia length="0.002" width="0.040" height="0.075" mass="0.00001"/>
       <visual>
         <origin xyz="0.016 0 -.015 " rpy="${M_PI} ${-M_PI/2} ${M_PI/2}"/>
@@ -328,11 +291,5 @@
     <xacro:macro name="pincher_gripper" params="name color *origin">
       <link name="${name}_link">
-      <inertial>
-        <mass value="0.00001"/>
-        <origin xyz="0 0 0"/>
-        <inertia ixx="1.0" ixy="0.0" ixz="0.0"
-          iyy="1.0" iyz="0.0"
-          izz="1.0"/>
-      </inertial>
+      <xacro:box_inertia length="0.036" width="0.028" height="0.004" mass="0.00001"/>
       <visual>
         <xacro:insert_block name="origin"/>

File: turtlebot_arm_description/urdf/pincher_arm.urdf (robot description, URDF)
Before this commit: robot turtlebot_arm, 24 links, 23 joints
Links:
- link arm_wrist_flex_link: mass 0.010 -> 0.01
- link gripper_active2_link: mass 0.00001 -> 1e-05
- link gripper_active_link: mass 0.00001 -> 1e-05
- link gripper_finger_base_link: mass 0.00001 -> 1e-05
Joints:
- joint arm_elbow_flex_joint: limit lower=-2.617 upper=2.617 effort=30 velocity=1.571 -> lower=-2.42 upper=2.38 effort=30 velocity=1.571
- joint arm_shoulder_lift_joint: limit lower=-2.617 upper=2.617 effort=30 velocity=1.571 -> lower=-2.2 upper=2.16 effort=30 velocity=1.571
- joint arm_wrist_flex_joint: limit lower=-1.745 upper=1.745 effort=30 velocity=1.571 -> lower=-1.72 upper=1.68 effort=30 velocity=1.571

File: turtlebot_arm_description/urdf/turtlebot_arm.urdf (robot description, URDF)
Before this commit: robot turtlebot_arm, 25 links, 24 joints
Links:
- link arm_wrist_flex_link: mass 0.010 -> 0.01

Commit message: Issue #21: fix pincher gripper collision boxes

File: turtlebot_arm_description/urdf/arm_hardware.xacro (robot description, xacro)
@@ -277,5 +277,5 @@
       </visual>
       <collision>
-        <origin xyz="0.015 0 -0.0135" rpy="0 0 0"/>
+        <origin xyz="0.016 0.0 -0.015" rpy="0 0 0"/>
         <geometry>
           <box size="0.002 0.040 0.075"/>
@@ -302,9 +302,9 @@
         <xacro:insert_block name="origin"/>
         <geometry>
-          <box size="0.036 0.028 0.004"/>
-        </geometry>
-      </collision>
-    </link>
-      <gazebo reference="${name}_link">
+          <box size="0.023 0.028 0.038"/>
+        </geometry>
+      </collision>
+    </link>
+    <gazebo reference="${name}_link">
       <material>Gazebo/${color}</material>
       <selfCollide>true</selfCollide>

File: turtlebot_arm_description/urdf/pincher_gripper.xacro (robot description, xacro)
@@ -21,5 +21,5 @@
     </joint>
     <pincher_gripper name="gripper_active" color="${color}" >
-      <origin xyz="-0.02 0.023 0" rpy="${-M_PI/2} 0 0"/>
+      <origin xyz="-0.0086 0.0414 0" rpy="${-M_PI/2} 0 0"/>
     </pincher_gripper>
     <!-- Finger 2 -->
@@ -30,5 +30,5 @@
     </joint>
     <pincher_gripper name="gripper_active2" color="${color}" >
-      <origin xyz="-0.02 0.023 0" rpy="${-M_PI/2} ${M_PI} 0"/>
+      <origin xyz="-0.0314 0.0414 0" rpy="${-M_PI/2} ${M_PI} 0"/>
     </pincher_gripper>
     <!-- Using Mimic -->

Commit message: Cleaned up pincher gripper description
Slightly restructured the TF tree of the pincher gripper to make more
sense compared to the physical construction of the gripper.

File: turtlebot_arm_description/urdf/arm_hardware.xacro (robot description, xacro)
@@ -11,4 +11,5 @@
   <xacro:property name="AX12_LENGTH" value="0.050"/>
   <xacro:property name="F2_HEIGHT" value="0.0265"/>
+  <xacro:property name="FINGER_HEIGHT" value="0.038"/>
   <!-- Calculates the inertial properties of a bounding box. From
        https://en.wikipedia.org/wiki/List_of_moments_of_inertia#List_of_3D_inertia_tensors-->
@@ -50,32 +51,4 @@
     </gazebo>
   </xacro:macro>
-  <xacro:macro name="finger_fixed" params="parent name color *origin">
-    <joint name="${name}_joint" type="fixed">
-      <xacro:insert_block name="origin"/>
-      <parent link="${parent}"/>
-      <child link="${name}_link"/>
-    </joint>
-    <link name="${name}_link">
-      <xacro:box_inertia length="0.0783" width="0.03801" height="0.0193" mass="0.015"/>
-      <visual>
-        <origin xyz=" 0 0 0 " rpy="0 0 0"/>
-        <geometry>
-          <mesh filename="package://turtlebot_arm_description/meshes/turtlebot_finger.stl" scale="${M_SCALE} ${M_SCALE} ${M_SCALE}"/>
-        </geometry>
-        <material name="${color}"/>
-      </visual>
-      <collision>
-        <origin xyz="0.02645 0.0 -0.00655" rpy="0 0 0"/>
-        <geometry>
-          <box size="0.0783 0.03801 0.0193"/>
-        </geometry>
-      </collision>
-    </link>
-    <gazebo reference="${name}_link">
-      <material>Gazebo/${color}</material>
-      <selfCollide>true</selfCollide>
-      <gravity>true</gravity>
-    </gazebo>
-  </xacro:macro>
   <xacro:macro name="dynamixel_AX12_fixed" params="parent name *origin">
     <joint name="${name}_joint" type="fixed">
@@ -268,19 +241,18 @@
     </joint>
     <link name="${name}_link">
-      <xacro:box_inertia length="0.002" width="0.040" height="0.075" mass="0.00001"/>
-      <visual>
-        <origin xyz="0.016 0 -.015 " rpy="${M_PI} ${-M_PI/2} ${M_PI/2}"/>
-        <geometry>
-          <mesh filename="package://turtlebot_arm_description/meshes/pincher_finger_base.stl" scale=".01 .01 .01"/>
-        </geometry>
-        <material name="${color}"/>
-      </visual>
-      <collision>
-        <origin xyz="0.016 0.0 -0.015" rpy="0 0 0"/>
-        <geometry>
-          <box size="0.002 0.040 0.075"/>
-        </geometry>
-      </collision>
-    </link >
+      <xacro:box_inertia length="0.002" width="0.075" height="0.040" mass="0.00001"/>
+      <visual>
+        <origin xyz="0 0 0" rpy="0 0 0"/>
+        <geometry>
+          <box size="0.002 0.075 0.040"/>
+        </geometry>
+        <material name="${color}"/>
+      </visual>
+      <collision>
+        <geometry>
+          <box size="0.002 0.075 0.040"/>
+        </geometry>
+      </collision>
+    </link>
     <gazebo reference="${name}_link">
       <material>Gazebo/${color}</material>

File: turtlebot_arm_description/urdf/pincher_gripper.xacro (robot description, xacro)
@@ -2,4 +2,5 @@
 <!-- PhantomX Pincher Arm gripper URDF-->
 <robot xmlns:xacro="http://ros.org/wiki/xacro">
+    <xacro:property name="GRIPPER_MAX" value="0.035"/>
     <bioloid_F3_fixed parent="arm_wrist_flex_link" name="arm_wrist_F3_0" color="${color}">
       <origin xyz="0 0 ${F2_HEIGHT}" rpy="0 ${M_PI} ${-M_PI}"/>
@@ -9,37 +10,31 @@
       <origin xyz="0 0 ${-AX12_WIDTH/2}" rpy="${M_PI/2} ${M_PI} ${M_PI/2}"/>
     </dynamixel_AX12_fixed>
-     <gripper_finger_base parent="gripper_servo_link" name="gripper_finger_base" color="${color}">
-      <origin xyz="0.01  ${AX12_WIDTH} 0" rpy="${M_PI/2} ${-M_PI} ${M_PI/2}"/>
+    <gripper_finger_base parent="gripper_servo_link" name="gripper_finger_base" color="${color}">
+        <origin xyz="0 ${AX12_WIDTH/2} 0" rpy="${M_PI} 0 ${M_PI/2}"/>
     </gripper_finger_base>
-     <!-- Finger 1 -->
+    <!-- Master finger -->
+    <!-- NOTE: The transmission for gripper_joint MUST specify a mechnaical reduction of two for
+         the gripper seperation to be calculated correctly -->
     <joint name="gripper_joint" type="prismatic">
-      <origin xyz="0 0 0" rpy="0 0 0"/>
-      <axis xyz="1 0 0"/>
-      <limit effort="30" velocity="0.5" lower="0.002" upper="0.031"/>
-      <parent link="gripper_servo_link"/>
+      <origin xyz="${FINGER_HEIGHT/2} 0 0" rpy="0 0 0"/>
+      <axis xyz="0 1 0"/>
+      <limit effort="30" velocity="0.05" lower="0.001" upper="${GRIPPER_MAX/2}"/>
+      <parent link="gripper_finger_base_link"/>
       <child link="gripper_active_link"/>
     </joint>
     <pincher_gripper name="gripper_active" color="${color}" >
-      <origin xyz="-0.0086 0.0414 0" rpy="${-M_PI/2} 0 0"/>
+      <origin xyz="0 0.01 0" rpy="${M_PI/2} 0 ${M_PI/2}"/>
     </pincher_gripper>
-    <!-- Finger 2 -->
-    <!-- Note: currently static but should be a Mimic of Finger 1 -->
-    <joint name="gripper2_joint" type="fixed">
-      <parent link="gripper_servo_link"/>
+    <!-- Slave finger -->
+    <joint name="gripper2_joint" type="prismatic">
+      <origin xyz="${FINGER_HEIGHT/2} 0 0" rpy="${M_PI} 0 0"/>
+      <axis xyz="0 1 0"/>
+      <limit effort="30" velocity="0.05" lower="0.001" upper="${GRIPPER_MAX/2}"/>
+      <parent link="gripper_finger_base_link"/>
       <child link="gripper_active2_link"/>
+      <mimic joint="gripper_joint"/>
     </joint>
     <pincher_gripper name="gripper_active2" color="${color}" >
-      <origin xyz="-0.0314 0.0414 0" rpy="${-M_PI/2} ${M_PI} 0"/>
+      <origin xyz="0 0.01 0" rpy="${M_PI/2} 0 ${M_PI/2}"/>
     </pincher_gripper>
-    <!-- Using Mimic -->
-    <!-- gripper 2 joint -->
-    <!--  ### Mimic would be better but causes Missing Joint error in Moveit
-      <joint name="gripper2_joint" type="prismatic">
-      <origin xyz="0 0 0" rpy="0 0 0"/>
-      <axis xyz="0 0 1"/>
-      <limit effort="30" velocity="0.5" lower="0.002" upper="0.031"/>
-      <parent link="gripper_servo_link"/>
-      <child link="gripper_active2_link"/>
-      <mimic joint="gripper_joint" multiplier="-.5"  offset = "0"/>
-    </joint-->
 </robot>

File: turtlebot_arm_description/urdf/turtlebot_arm.xacro (robot description, xacro)
@@ -27,5 +27,10 @@
     <link name="gripper_link"/>
     <joint name="gripper_link_joint" type="revolute">
-      <origin xyz="0 0 0.112" rpy="0 -1.57 0"/>
+      <xacro:if value="${turtlebot_gripper}">
+        <origin xyz="0 0 0.112" rpy="0 -1.57 0"/>
+      </xacro:if>
+      <xacro:if value="${pincher_gripper}">
+        <origin xyz="0 0 0.085" rpy="0 -1.57 0"/>
+      </xacro:if>
       <parent link="arm_wrist_flex_link"/>
       <child link="gripper_link"/>
